File: HARDWARE/Ethernet.kicad_sch (KiCad schematic)
At the start: 22 parts, among them J1 RJ45_Wuerth_7499151120, U4 KSZ8463FRL, Y1 25Mhz

Commit message: schematic capture
Parts:
- removed C4, C5: 0.1u, symbol Device:C_Small
- removed J1: RJ45_Wuerth_7499151120, Connector_RJ:RJ45_Wuerth_7499151120_Horizontal, symbol Connector:RJ45_Wuerth_7499151120
- added C12, C13, C14, C15: 0.1u, symbol Device:C_Small
- added J1, J2: KLS12-TL051, symbol meshium_duo:KLS12-TL051
- renumbered C7 to C10, C6 to C11, C3 to C5, C2 to C6, C8 to C7, C9 to C8, C10 to C9, R2 to R1, R1 to R2, R6 to R3, R7 to R4, R3 to R5, R5 to R6, R4 to R7
Connections:
- net +3V3: now also J1.12 (LEDY_A), J1.9 (LEDG_A), J2.12 (LEDY_A), J2.9 (LEDG_A)
- net Earth: now also J1.4 (SHIELD), J1.5 (SHIELD), J2.4 (SHIELD), J2.5 (SHIELD)
- net GND: now also C12.1, C13.1, C14.1, C15.1
- net at R8.2: now also J2.10 (LEDG_C)
- net at R9.2: now also J2.11 (LEDY_C)
- net at U4.10 (RXM2): now also J2.1 (TD+)
- net at U4.11 (RXP2): now also J2.2 (TD-)
- net at U4.13 (TXM2): now also J2.7 (RD+)
- net at U4.14 (TXP2): now also J2.8 (RD-)
- net at U4.1 (RXM1): now also J1.1 (TD+)
- net at U4.2 (RXP1): now also J1.2 (TD-)
- net at U4.4 (TXM1): now also J1.7 (RD+)
- net at U4.5 (TXP1): now also J1.8 (RD-)
- net at R6.2: now also J1.10 (LEDG_C)
- net at R7.2: now also J1.11 (LEDY_C)
- new net: C15.2, J2.6 (CT)
- new net: C12.2, J1.3 (CT)
- new net: C14.2, J1.6 (CT)
- new net: C13.2, J2.3 (CT)

Commit message: schematic capture
Parts:
- added U8, U9: USBLC6-4SC6, Package_TO_SOT_SMD:SOT-23-6, symbol Power_Protection:USBLC6-4SC6
- C10, C11, C12, C13, C14, C15, C5, C6, C7, C8, C9: footprint (none) -> Capacitor_SMD:C_0603_1608Metric
- R1, R2, R3, R4, R5, R6, R7, R8, R9: footprint Resistor_SMD:R_0402_1005Metric -> Resistor_SMD:R_0603_1608Metric
Changed lines of the file:
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@@
       (effects (font (size 0.8 0.8)))
     )
-    (property "Footprint" "Resistor_SMD:R_0402_1005Metric" (at 104.14 109.22 0)
+    (property "Footprint" "Resistor_SMD:R_0603_1608Metric" (at 104.14 109.22 0)
       (effects (font (size 1.27 1.27)) hide)
     )
@@
       (effects (font (size 1.27 1.27)))
     )
-    (property "Footprint" "" (at 242.57 149.86 0)
+    (property "Footprint" "Capacitor_SMD:C_0603_1608Metric" (at 242.57 149.86 0)
       (effects (font (size 1.27 1.27)) hide)
     )
@@
     )
   )
+  (symbol (lib_id "Power_Protection:USBLC6-4SC6") (at 201.93 46.99 0) (unit 1)
+    (in_bom yes) (on_board yes) (dnp no) (fields_autoplaced)
+    (property "Reference" "U8" (at 203.5811 34.29 0)
+      (effects (font (size 1.27 1.27)) (justify left))
+    )
+    (property "Value" "USBLC6-4SC6" (at 203.5811 36.83 0)
+      (effects (font (size 1.27 1.27)) (justify left))
+    )
+    (property "Footprint" "Package_TO_SOT_SMD:SOT-23-6" (at 201.93 59.69 0)
+      (effects (font (size 1.27 1.27)) hide)
+    )
+    (property "Datasheet" "https://www.st.com/resource/en/datasheet/usblc6-4.pdf" (at 207.01 38.1 0)
+      (effects (font (size 1.27 1.27)) hide)
+    )
+    (pin "1")
+    (pin "2")
+    (pin "3")
+    (pin "4")
+    (pin "5")
+    (pin "6")
+    (instances
+      (project "meshium_duo"
+        (path "/2783b917-8d7b-4d69-a31c-61fb9333015c/48aab9f2-2fa4-4160-b2c2-696df96194f5"
+          (reference "U8") (unit 1)
+        )
+      )
+    )
+  )
   (symbol (lib_id "power:GND") (at 102.87 57.15 180) (unit 1)
     (in_bom yes) (on_board yes) (dnp no) (fields_autoplaced)
@@
       (effects (font (size 1.27 1.27)) (justify right))
     )
-    (property "Footprint" "" (at 147.32 54.61 0)
+    (property "Footprint" "Capacitor_SMD:C_0603_1608Metric" (at 147.32 54.61 0)
       (effects (font (size 1.27 1.27)) hide)
     )
@@
       (effects (font (size 0.8 0.8)))
     )
-    (property "Footprint" "Resistor_SMD:R_0402_1005Metric" (at 193.04 140.97 0)
+    (property "Footprint" "Resistor_SMD:R_0603_1608Metric" (at 193.04 140.97 0)
       (effects (font (size 1.27 1.27)) hide)
     )
@@
       (effects (font (size 0.8 0.8)))
     )
-    (property "Footprint" "Resistor_SMD:R_0402_1005Metric" (at 243.84 106.68 0)
+    (property "Footprint" "Resistor_SMD:R_0603_1608Metric" (at 243.84 106.68 0)
       (effects (font (size 1.27 1.27)) hide)
     )
@@
       (effects (font (size 1.27 1.27)) (justify right))
     )
-    (property "Footprint" "" (at 121.92 35.56 0)
+    (property "Footprint" "Capacitor_SMD:C_0603_1608Metric" (at 121.92 35.56 0)
       (effects (font (size 1.27 1.27)) hide)
     )
@@
       (effects (font (size 1.27 1.27)))
     )
-    (property "Footprint" "" (at 237.49 73.66 0)
+    (property "Footprint" "Capacitor_SMD:C_0603_1608Metric" (at 237.49 73.66 0)
       (effects (font (size 1.27 1.27)) hide)
     )
@@
       (effects (font (size 0.8 0.8)))
     )
-    (property "Footprint" "Resistor_SMD:R_0402_1005Metric" (at 193.04 80.01 0)
+    (property "Footprint" "Resistor_SMD:R_0603_1608Metric" (at 193.04 80.01 0)
       (effects (font (size 1.27 1.27)) hide)
     )
@@
       (effects (font (size 1.27 1.27)) (justify left))
     )
-    (property "Footprint" "" (at 107.95 60.96 0)
+    (property "Footprint" "Capacitor_SMD:C_0603_1608Metric" (at 107.95 60.96 0)
       (effects (font (size 1.27 1.27)) hide)
     )
@@
       (effects (font (size 1.27 1.27)) (justify right))
     )
-    (property "Footprint" "" (at 162.56 54.61 0)
+    (property "Footprint" "Capacitor_SMD:C_0603_1608Metric" (at 162.56 54.61 0)
       (effects (font (size 1.27 1.27)) hide)
     )
@@
       (effects (font (size 1.27 1.27)))
     )
-    (property "Footprint" "" (at 242.57 73.66 0)
+    (property "Footprint" "Capacitor_SMD:C_0603_1608Metric" (at 242.57 73.66 0)
       (effects (font (size 1.27 1.27)) hide)
     )
@@
       (effects (font (size 0.8 0.8)))
     )
-    (property "Footprint" "Resistor_SMD:R_0402_1005Metric" (at 104.14 88.9 0)
+    (property "Footprint" "Resistor_SMD:R_0603_1608Metric" (at 104.14 88.9 0)
       (effects (font (size 1.27 1.27)) hide)
     )
@@
       (effects (font (size 1.27 1.27)) (justify left))
     )
-    (property "Footprint" "" (at 97.79 60.96 0)
+    (property "Footprint" "Capacitor_SMD:C_0603_1608Metric" (at 97.79 60.96 0)
       (effects (font (size 1.27 1.27)) hide)
     )
@@
       (effects (font (size 1.27 1.27)))
     )
-    (property "Footprint" "" (at 237.49 149.86 0)
+    (property "Footprint" "Capacitor_SMD:C_0603_1608Metric" (at 237.49 149.86 0)
       (effects (font (size 1.27 1.27)) hide)
     )
@@
       (effects (font (size 0.8 0.8)))
     )
-    (property "Footprint" "Resistor_SMD:R_0402_1005Metric" (at 243.84 109.22 0)
+    (property "Footprint" "Resistor_SMD:R_0603_1608Metric" (at 243.84 109.22 0)
       (effects (font (size 1.27 1.27)) hide)
     )
@@
       (effects (font (size 0.8 0.8)))
     )
-    (property "Footprint" "Resistor_SMD:R_0402_1005Metric" (at 243.84 33.02 0)
+    (property "Footprint" "Resistor_SMD:R_0603_1608Metric" (at 243.84 33.02 0)
       (effects (font (size 1.27 1.27)) hide)
     )
@@
       (effects (font (size 1.27 1.27)) (justify right))
     )
-    (property "Footprint" "" (at 139.7 35.56 0)
+    (property "Footprint" "Capacitor_SMD:C_0603_1608Metric" (at 139.7 35.56 0)
       (effects (font (size 1.27 1.27)) hide)
     )
@@
       (effects (font (size 0.8 0.8)))
     )
-    (property "Footprint" "Resistor_SMD:R_0402_1005Metric" (at 243.84 30.48 0)
+    (property "Footprint" "Resistor_SMD:R_0603_1608Metric" (at 243.84 30.48 0)
       (effects (font (size 1.27 1.27)) hide)
     )
@@
       (effects (font (size 1.27 1.27)) (justify right))
     )
-    (property "Footprint" "" (at 130.81 35.56 0)
+    (property "Footprint" "Capacitor_SMD:C_0603_1608Metric" (at 130.81 35.56 0)
       (effects (font (size 1.27 1.27)) hide)
     )
@@
       (effects (font (size 0.8 0.8)))
     )
-    (property "Footprint" "Resistor_SMD:R_0402_1005Metric" (at 193.04 102.87 0)
+    (property "Footprint" "Resistor_SMD:R_0603_1608Metric" (at 193.04 102.87 0)
       (effects (font (size 1.27 1.27)) hide)
     )
@@
         )
       )
+    )
+  )
+  (symbol (lib_id "Power_Protection:USBLC6-4SC6") (at 212.09 157.48 0) (unit 1)
+    (in_bom yes) (on_board yes) (dnp no) (fields_autoplaced)
+    (property "Reference" "U9" (at 213.7411 144.78 0)
+      (effects (font (size 1.27 1.27)) (justify left))
+    )
+    (property "Value" "USBLC6-4SC6" (at 213.7411 147.32 0)
+      (effects (font (size 1.27 1.27)) (justify left))
+    )
+    (property "Footprint" "Package_TO_SOT_SMD:SOT-23-6" (at 212.09 170.18 0)
+      (effects (font (size 1.27 1.27)) hide)
+    )
+    (property "Datasheet" "https://www.st.com/resource/en/datasheet/usblc6-4.pdf" (at 217.17 148.59 0)
+      (effects (font (size 1.27 1.27)) hide)
+    )
+    (pin "1")
+    (pin "2")
+    (pin "3")
+    (pin "4")
+    (pin "5")
+    (pin "6")
+    (instances
+      (project "meshium_duo"
+        (path "/2783b917-8d7b-4d69-a31c-61fb9333015c/48aab9f2-2fa4-4160-b2c2-696df96194f5"
+          (reference "U9") (unit 1)
+        )
+      )

Commit message: schematic capture
Parts:
- FB1: footprint (none) -> Capacitor_SMD:C_0603_1608Metric
- Y1: footprint (none) -> Crystal:Crystal_SMD_3225-4Pin_3.2x2.5mm
Changed lines of the file:
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@@
       (effects (font (size 1.27 1.27)))
     )
-    (property "Footprint" "" (at 102.87 64.77 0)
+    (property "Footprint" "Crystal:Crystal_SMD_3225-4Pin_3.2x2.5mm" (at 102.87 64.77 0)
       (effects (font (size 1.27 1.27)) hide)
     )
@@
       (effects (font (size 1.27 1.27)) hide)
     )
-    (property "Footprint" "" (at 153.67 60.198 90)
-      (effects (font (size 1.27 1.27)) hide)
-    )
+    (property "Footprint" "Capacitor_SMD:C_0603_1608Metric" (at 153.67 60.198 90)
+      (effects (font (size 1.27 1.27)) hide)
+    )

Commit message: schematic capture
Parts:
- J1, J2: footprint (none) -> Footpint:KLS12-TL051
Changed lines of the file:
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@@
       (effects (font (size 1.27 1.27)) (justify right))
     )
-    (property "Footprint" "" (at 259.08 135.89 0)
+    (property "Footprint" "Footpint:KLS12-TL051" (at 259.08 135.89 0)
       (effects (font (size 1.27 1.27)) hide)
     )
@@
       (effects (font (size 1.27 1.27)) (justify right))
     )
-    (property "Footprint" "" (at 259.08 59.69 0)
+    (property "Footprint" "Footpint:KLS12-TL051" (at 259.08 59.69 0)
       (effects (font (size 1.27 1.27)) hide)
     )

Commit message: schematic capture
Connections:
- net +3V3: now also U8.5 (VBUS), U9.5 (VBUS)
- net GND: now also U8.2 (GND), U9.2 (GND)
- net at U8.1 (I/O1): now also J1.8 (RD-), U4.5 (TXP1)
- net at U8.3 (I/O2): now also J1.7 (RD+), U4.4 (TXM1)
- net at U8.4 (I/O3): now also J1.1 (TD+), U4.1 (RXM1)
- net at U8.6 (I/O4): now also J1.2 (TD-), U4.2 (RXP1)
- net at J2.1 (TD+), U4.10 (RXM2): now also U9.4 (I/O3)
- net at J2.2 (TD-), U4.11 (RXP2): now also U9.6 (I/O4)
- net at J2.7 (RD+), U4.13 (TXM2): now also U9.1 (I/O1)
- net at J2.8 (RD-), U4.14 (TXP2): now also U9.3 (I/O2)
Other:
- moved on the sheet: R5, U8, U9
