File: HARDWARE/Ethernet.kicad_sch (KiCad schematic)
At the start: 27 parts, among them J1 KLS12-TL051, J2 KLS12-TL051, U4 KSZ8463FRL, U8 USBLC6-4SC6, U9 USBLC6-4SC6, Y1 25Mhz

Commit message: schematic capture
Parts:
- renumbered C5 to C35, C6 to C36, C7 to C37, C8 to C38, C9 to C39, C10 to C40, C11 to C41, C12 to C42, C13 to C43, C14 to C44, C15 to C45, FB1 to FB2, J1 to J4, J2 to J5, R1 to R14, R2 to R15, R5 to R16, R3 to R17, R4 to R18, R6 to R19, R7 to R20, R8 to R21, R9 to R22, U4 to U7, Y1 to Y3

Commit message: tracerouting
Parts:
- removed J4, J5: KLS12-TL051, Footpint:KLS12-TL051, symbol meshium_duo:KLS12-TL051
- removed Y3: 25Mhz, Crystal:Crystal_SMD_3225-4Pin_3.2x2.5mm, symbol Device:Crystal_Small
- added J20: TRJ26404AENL, symbol meshium_duo:TRJ26404AENL
- added Y1: 25MHz, Crystal:Crystal_SMD_3225-4Pin_3.2x2.5mm, symbol Device:Crystal_GND24_Small
Connections:
- net +3V3: now also J20.A11 (LEDY_A), J20.A9 (LEDG_A), J20.B11 (LEDY_A), J20.B9 (LEDG_A)
- net Earth: now also J20.A8 (TERM), J20.B8 (TERM), J20.SH (SHIELD), J20.SH (SHIELD)
- net GND: now also Y1.2, Y1.4
- net at C35.2, U7.18 (XI): now also Y1.3
- net at C36.2, U7.19 (XO): now also Y1.1
- net at C45.2: now also J20.B4 (CT)
- net RXM1: now reaches U8.1 (I/O1)
- net RXM1: now also U7.1 (RXM1), J20.A1 (RD+); no longer U7.5 (TXP1)
- net RXP1: now reaches U8.3 (I/O2)
- net RXP1: now also U7.2 (RXP1), J20.A2 (RD-); no longer U7.4 (TXM1)
- net TXM1: now reaches U8.4 (I/O3)
- net TXM1: now also U7.4 (TXM1), J20.A3 (TD+); no longer U7.1 (RXM1)
- net TXP1: now reaches U8.6 (I/O4)
- net TXP1: now also U7.5 (TXP1), J20.A6 (TD-); no longer U7.2 (RXP1)
- net RXM2: now reaches U7.10 (RXM2)
- net RXM2: now also U9.1 (I/O1), J20.B1 (RD+); no longer U9.4 (I/O3)
- net RXP2: now reaches U7.11 (RXP2)
- net RXP2: now also U9.3 (I/O2), J20.B2 (RD-); no longer U9.6 (I/O4)
- net TXM2: now reaches U7.13 (TXM2)
- net TXM2: now also U9.4 (I/O3), J20.B3 (TD+); no longer U9.1 (I/O1)
- net TXP2: now reaches U7.14 (TXP2)
- net TXP2: now also U9.6 (I/O4), J20.B6 (TD-); no longer U9.3 (I/O2)
- net at R21.2: now also J20.B10 (LEDG_C)
- net at C42.2: now also J20.A5 (CT)
- net at C44.2: now also J20.A4 (CT)
- net at C43.2: now also J20.B5 (CT)
- net at R22.2: now also J20.B12 (LEDY_C)
- net at R20.2: now also J20.A12 (LEDY_C)
- net at R19.2: now also J20.A10 (LEDG_C)
Other:
- moved on the sheet: C35, C36, C37, C38, C39, C40, C41, C42, C43, C44, C45, FB2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

Commit message: tracerouting
Parts:
- renumbered Y1 to Y3
Changed lines of the file:
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@@
   (symbol (lib_id "Device:Crystal_GND24_Small") (at 86.36 62.23 180) (unit 1)
     (in_bom yes) (on_board yes) (dnp no)
-    (property "Reference" "Y1" (at 83.82 58.42 0)
+    (property "Reference" "Y3" (at 83.82 58.42 0)
       (effects (font (size 1.27 1.27)))
     )
@@
     (instances
       (project "meshium_duo"
-        (path "/2783b917-8d7b-4d69-a31c-61fb9333015c/b5f76ac1-5f31-46a3-a641-c3c4fe73e10b"
-          (reference "Y1") (unit 1)
-        )
         (path "/2783b917-8d7b-4d69-a31c-61fb9333015c/48aab9f2-2fa4-4160-b2c2-696df96194f5"
           (reference "Y3") (unit 1)
