File: HARDWARE/Memory.kicad_sch (KiCad schematic)
At the start: 3 parts, among them U2 MX25L3233FZN, U3 MT48LC16M16A2P

Commit message: pcb creation
Parts:
- added C18: 1u, symbol Device:C_Small
- added C19, C20: 0.1u, symbol Device:C_Small
Connections:
- net +3V3: now also C18.1, C19.1, C20.1
- net GND: now also C18.2, C19.2, C20.2
Changed lines of the file:
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@@
   (junction (at 153.67 33.02) (diameter 0) (color 0 0 0 0)
   )
+  (junction (at 222.25 101.6) (diameter 0) (color 0 0 0 0)
+  )
   (junction (at 82.55 90.17) (diameter 0) (color 0 0 0 0)
   )
   (junction (at 182.88 118.11) (diameter 0) (color 0 0 0 0)
   )
+  (junction (at 213.36 111.76) (diameter 0) (color 0 0 0 0)
+  )
   (junction (at 182.88 44.45) (diameter 0) (color 0 0 0 0)
   )
   (junction (at 82.55 62.23) (diameter 0) (color 0 0 0 0)
   )
+  (junction (at 231.14 101.6) (diameter 0) (color 0 0 0 0)
+  )
+  (junction (at 222.25 111.76) (diameter 0) (color 0 0 0 0)
+  )
   (bus_entry (at 214.63 83.82) (size 2.54 -2.54)
     (stroke (width 0) (type default))
@@
     (stroke (width 0) (type default))
   )
-  (bus_entry (at 214.63 53.34) (size 2.54 -2.54)
-    (stroke (width 0) (type default))
-  )
   (bus_entry (at 214.63 81.28) (size 2.54 -2.54)
     (stroke (width 0) (type default))
@@
     (stroke (width 0) (type default))
   )
-  (bus_entry (at 214.63 50.8) (size 2.54 -2.54)
-    (stroke (width 0) (type default))
-  )
   (bus_entry (at 153.67 66.04) (size 2.54 2.54)
     (stroke (width 0) (type default))
@@
     (stroke (width 0) (type default))
   )
+  (wire (pts (xy 231.14 109.22) (xy 231.14 111.76))
+    (stroke (width 0) (type default))
+  )
   (bus (pts (xy 153.67 86.36) (xy 153.67 83.82))
     (stroke (width 0) (type default))
@@
     (stroke (width 0) (type default))
   )
+  (wire (pts (xy 231.14 100.33) (xy 231.14 101.6))
+    (stroke (width 0) (type default))
+  )
   (wire (pts (xy 198.12 71.12) (xy 214.63 71.12))
     (stroke (width 0) (type default))
@@
     (stroke (width 0) (type default))
   )
+  (wire (pts (xy 213.36 111.76) (xy 213.36 109.22))
+    (stroke (width 0) (type default))
+  )
   (wire (pts (xy 185.42 45.72) (xy 185.42 44.45))
     (stroke (width 0) (type default))
@@
     (stroke (width 0) (type default))
   )
+  (wire (pts (xy 222.25 109.22) (xy 222.25 111.76))
+    (stroke (width 0) (type default))
+  )
   (bus (pts (xy 153.67 81.28) (xy 153.67 78.74))
     (stroke (width 0) (type default))
@@
     (stroke (width 0) (type default))
   )
+  (wire (pts (xy 213.36 101.6) (xy 222.25 101.6))
+    (stroke (width 0) (type default))
+  )
   (bus (pts (xy 153.67 66.04) (xy 153.67 63.5))
     (stroke (width 0) (type default))
@@
     (stroke (width 0) (type default))
   )
+  (wire (pts (xy 213.36 104.14) (xy 213.36 101.6))
+    (stroke (width 0) (type default))
+  )
   (wire (pts (xy 182.88 43.18) (xy 182.88 44.45))
     (stroke (width 0) (type default))
@@
     (stroke (width 0) (type default))
   )
+  (wire (pts (xy 231.14 111.76) (xy 222.25 111.76))
+    (stroke (width 0) (type default))
+  )
   (wire (pts (xy 198.12 50.8) (xy 214.63 50.8))
     (stroke (width 0) (type default))
@@
     (stroke (width 0) (type default))
   )
+  (wire (pts (xy 222.25 101.6) (xy 222.25 104.14))
+    (stroke (width 0) (type default))
+  )
   (wire (pts (xy 182.88 119.38) (xy 182.88 118.11))
     (stroke (width 0) (type default))
@@
     (stroke (width 0) (type default))
   )
+  (wire (pts (xy 222.25 101.6) (xy 231.14 101.6))
+    (stroke (width 0) (type default))
+  )
   (bus (pts (xy 153.67 96.52) (xy 153.67 93.98))
     (stroke (width 0) (type default))
   )
+  (wire (pts (xy 222.25 111.76) (xy 213.36 111.76))
+    (stroke (width 0) (type default))
+  )
   (wire (pts (xy 198.12 53.34) (xy 214.63 53.34))
     (stroke (width 0) (type default))
@@
     (stroke (width 0) (type default))
   )
+  (wire (pts (xy 231.14 101.6) (xy 231.14 104.14))
+    (stroke (width 0) (type default))
+  )
   (bus (pts (xy 153.67 55.88) (xy 153.67 58.42))
     (stroke (width 0) (type default))
@@
     (stroke (width 0) (type default))
   )
+  (wire (pts (xy 213.36 111.76) (xy 213.36 113.03))
+    (stroke (width 0) (type default))
+  )
   (wire (pts (xy 54.61 78.74) (xy 72.39 78.74))
     (stroke (width 0) (type default))
@@
   (label "FMC_D12" (at 212.09 81.28 180) (fields_autoplaced)
     (effects (font (size 1.27 1.27)) (justify right bottom))
+  )
+  (global_label "FMC_D0" (shape input) (at 214.63 50.8 0) (fields_autoplaced)
+    (effects (font (size 1.27 1.27)) (justify left))
+    (property "Intersheetrefs" "${INTERSHEET_REFS}" (at 224.8723 50.8 0)
+      (effects (font (size 1.27 1.27)) (justify left) hide)
+    )
   )
   (hierarchical_label "FMC_SDRAM" (shape bidirectional) (at 151.13 33.02 180) (fields_autoplaced)
@@
     )
   )
+  (symbol (lib_id "Device:C_Small") (at 231.14 106.68 0) (unit 1)
+    (in_bom yes) (on_board yes) (dnp no) (fields_autoplaced)
+    (property "Reference" "C20" (at 233.68 105.4163 0)
+      (effects (font (size 1.27 1.27)) (justify left))
+    )
+    (property "Value" "0.1u" (at 233.68 107.9563 0)
+      (effects (font (size 1.27 1.27)) (justify left))
+    )
+    (property "Footprint" "" (at 231.14 106.68 0)
+      (effects (font (size 1.27 1.27)) hide)
+    )
+    (property "Datasheet" "~" (at 231.14 106.68 0)
+      (effects (font (size 1.27 1.27)) hide)
+    )
+    (pin "1")
+    (pin "2")
+    (instances
+      (project "meshium_duo"
+        (path "/2783b917-8d7b-4d69-a31c-61fb9333015c/4650415e-d772-4f66-8f38-5713f833944e"
+          (reference "C20") (unit 1)
+        )
+      )
+    )
+  )
   (symbol (lib_id "power:+3V3") (at 182.88 43.18 0) (unit 1)
     (in_bom yes) (on_board yes) (dnp no) (fields_autoplaced)
@@
     )
   )
+  (symbol (lib_id "power:GND") (at 213.36 113.03 0) (unit 1)
+    (in_bom yes) (on_board yes) (dnp no) (fields_autoplaced)
+    (property "Reference" "#PWR033" (at 213.36 119.38 0)
+      (effects (font (size 1.27 1.27)) hide)
+    )
+    (property "Value" "GND" (at 213.36 118.11 0)
+      (effects (font (size 1.27 1.27)))
+    )
+    (property "Footprint" "" (at 213.36 113.03 0)
+      (effects (font (size 1.27 1.27)) hide)
+    )
+    (property "Datasheet" "" (at 213.36 113.03 0)
+      (effects (font (size 1.27 1.27)) hide)
+    )
+    (pin "1")
+    (instances
+      (project "meshium_duo"
+        (path "/2783b917-8d7b-4d69-a31c-61fb9333015c/4650415e-d772-4f66-8f38-5713f833944e"
+          (reference "#PWR033") (unit 1)
+        )
+      )
+    )
+  )
+  (symbol (lib_id "power:+3V3") (at 231.14 100.33 0) (unit 1)
+    (in_bom yes) (on_board yes) (dnp no) (fields_autoplaced)
+    (property "Reference" "#PWR034" (at 231.14 104.14 0)
+      (effects (font (size 1.27 1.27)) hide)
+    )
+    (property "Value" "+3V3" (at 231.14 95.25 0)
+      (effects (font (size 1.27 1.27)))
+    )
+    (property "Footprint" "" (at 231.14 100.33 0)
+      (effects (font (size 1.27 1.27)) hide)
+    )
+    (property "Datasheet" "" (at 231.14 100.33 0)
+      (effects (font (size 1.27 1.27)) hide)
+    )
+    (pin "1")
+    (instances
+      (project "meshium_duo"
+        (path "/2783b917-8d7b-4d69-a31c-61fb9333015c/4650415e-d772-4f66-8f38-5713f833944e"
+          (reference "#PWR034") (unit 1)
+        )
+      )
+    )
+  )
+  (symbol (lib_id "Device:C_Small") (at 222.25 106.68 0) (unit 1)
+    (in_bom yes) (on_board yes) (dnp no) (fields_autoplaced)
+    (property "Reference" "C19" (at 224.79 105.4163 0)
+      (effects (font (size 1.27 1.27)) (justify left))
+    )
+    (property "Value" "0.1u" (at 224.79 107.9563 0)
+      (effects (font (size 1.27 1.27)) (justify left))
+    )
+    (property "Footprint" "" (at 222.25 106.68 0)
+      (effects (font (size 1.27 1.27)) hide)
+    )
+    (property "Datasheet" "~" (at 222.25 106.68 0)
+      (effects (font (size 1.27 1.27)) hide)
+    )
+    (pin "1")
+    (pin "2")
+    (instances
+      (project "meshium_duo"
+        (path "/2783b917-8d7b-4d69-a31c-61fb9333015c/4650415e-d772-4f66-8f38-5713f833944e"
+          (reference "C19") (unit 1)
+        )
+      )
+    )
+  )
   (symbol (lib_id "power:GND") (at 91.44 62.23 90) (unit 1)
     (in_bom yes) (on_board yes) (dnp no) (fields_autoplaced)
@@
         )
       )
+    )
+  )
+  (symbol (lib_id "Device:C_Small") (at 213.36 106.68 0) (unit 1)
+    (in_bom yes) (on_board yes) (dnp no) (fields_autoplaced)
+    (property "Reference" "C18" (at 215.9 105.4163 0)
+      (effects (font (size 1.27 1.27)) (justify left))
+    )
+    (property "Value" "1u" (at 215.9 107.9563 0)
+      (effects (font (size 1.27 1.27)) (justify left))
+    )
+    (property "Footprint" "" (at 213.36 106.68 0)
+      (effects (font (size 1.27 1.27)) hide)
+    )
+    (property "Datasheet" "~" (at 213.36 106.68 0)
+      (effects (font (size 1.27 1.27)) hide)
+    )
+    (pin "1")
+    (pin "2")
+    (instances
+      (project "meshium_duo"
+        (path "/2783b917-8d7b-4d69-a31c-61fb9333015c/4650415e-d772-4f66-8f38-5713f833944e"
+          (reference "C18") (unit 1)
+        )
+      )

Commit message: schematic capture
Parts:
- removed U2: MX25L3233FZN, Package_SON:WSON-8-1EP_6x5mm_P1.27mm_EP3.4x4mm, symbol Memory_Flash:MX25L3233FZN
- added U2: MX25L25635F, Package_SON:WSON-8-1EP_8x6mm_P1.27mm_EP3.4x4.3mm, symbol meshium_duo:MX25R3235FM1xx0
- renumbered C18 to C2, C19 to C3, C20 to C4
Connections:
- net +3V3: now also U2.8 (VCC)
- net GND: now also U2.4 (GND)
- net QSPI_BK1_CLK: now also U2.6 (SCLK)
- net QSPI_BK1_IO0: now also U2.5 (SI/SIO0)
- net QSPI_BK1_IO1: now also U2.2 (SO/SIO1)
- net QSPI_BK1_IO2: now also U2.3 (~{WP}/SIO2)
- net QSPI_BK1_IO3: now also U2.7 (~{RESET}/SIO3)
- net QSPI_BK1_NCS: now also U2.1 (~{CS})

Commit message: schematic capture
Parts:
- C1, C2, C3, C4: footprint (none) -> Capacitor_SMD:C_0603_1608Metric
Changed lines of the file:
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@@
       (effects (font (size 1.27 1.27)) (justify left))
     )
-    (property "Footprint" "" (at 231.14 106.68 0)
+    (property "Footprint" "Capacitor_SMD:C_0603_1608Metric" (at 231.14 106.68 0)
       (effects (font (size 1.27 1.27)) hide)
     )
@@
       (effects (font (size 1.27 1.27)))
     )
-    (property "Footprint" "" (at 87.63 62.23 0)
+    (property "Footprint" "Capacitor_SMD:C_0603_1608Metric" (at 87.63 62.23 0)
       (effects (font (size 1.27 1.27)) hide)
     )
@@
       (effects (font (size 1.27 1.27)) (justify left))
     )
-    (property "Footprint" "" (at 222.25 106.68 0)
+    (property "Footprint" "Capacitor_SMD:C_0603_1608Metric" (at 222.25 106.68 0)
       (effects (font (size 1.27 1.27)) hide)
     )
@@
       (effects (font (size 1.27 1.27)) (justify left))
     )
-    (property "Footprint" "" (at 213.36 106.68 0)
+    (property "Footprint" "Capacitor_SMD:C_0603_1608Metric" (at 213.36 106.68 0)
       (effects (font (size 1.27 1.27)) hide)
     )

Commit message: schematic capture
Parts:
- renumbered C1 to C31, C2 to C32, C3 to C33, C4 to C34, U2 to U5, U3 to U6
Changed lines of the file:
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@@
   (symbol (lib_id "Memory_RAM:MT48LC16M16A2P") (at 185.42 81.28 0) (unit 1)
     (in_bom yes) (on_board yes) (dnp no) (fields_autoplaced)
-    (property "Reference" "U3" (at 187.6141 43.18 0)
+    (property "Reference" "U6" (at 187.6141 43.18 0)
       (effects (font (size 1.27 1.27)) (justify left))
     )
@@
       (project "meshium_duo"
         (path "/2783b917-8d7b-4d69-a31c-61fb9333015c/4650415e-d772-4f66-8f38-5713f833944e"
-          (reference "U3") (unit 1)
+          (reference "U6") (unit 1)
         )
       )
@@
   (symbol (lib_id "power:GND") (at 182.88 119.38 0) (unit 1)
     (in_bom yes) (on_board yes) (dnp no) (fields_autoplaced)
-    (property "Reference" "#PWR06" (at 182.88 125.73 0)
+    (property "Reference" "#PWR053" (at 182.88 125.73 0)
       (effects (font (size 1.27 1.27)) hide)
     )
@@
       (project "meshium_duo"
         (path "/2783b917-8d7b-4d69-a31c-61fb9333015c/4650415e-d772-4f66-8f38-5713f833944e"
-          (reference "#PWR06") (unit 1)
+          (reference "#PWR053") (unit 1)
         )
       )
@@
   (symbol (lib_id "power:GND") (at 82.55 91.44 0) (unit 1)
     (in_bom yes) (on_board yes) (dnp no) (fields_autoplaced)
-    (property "Reference" "#PWR03" (at 82.55 97.79 0)
+    (property "Reference" "#PWR050" (at 82.55 97.79 0)
       (effects (font (size 1.27 1.27)) hide)
     )
@@
       (project "meshium_duo"
         (path "/2783b917-8d7b-4d69-a31c-61fb9333015c/4650415e-d772-4f66-8f38-5713f833944e"
-          (reference "#PWR03") (unit 1)
+          (reference "#PWR050") (unit 1)
         )
       )
@@
   (symbol (lib_id "power:+3V3") (at 82.55 59.69 0) (unit 1)
     (in_bom yes) (on_board yes) (dnp no) (fields_autoplaced)
-    (property "Reference" "#PWR02" (at 82.55 63.5 0)
+    (property "Reference" "#PWR049" (at 82.55 63.5 0)
       (effects (font (size 1.27 1.27)) hide)
     )
@@
       (project "meshium_duo"
         (path "/2783b917-8d7b-4d69-a31c-61fb9333015c/4650415e-d772-4f66-8f38-5713f833944e"
-          (reference "#PWR02") (unit 1)
+          (reference "#PWR049") (unit 1)
         )
       )
@@
   (symbol (lib_id "Device:C_Small") (at 231.14 106.68 0) (unit 1)
     (in_bom yes) (on_board yes) (dnp no) (fields_autoplaced)
-    (property "Reference" "C4" (at 233.68 105.4163 0)
+    (property "Reference" "C34" (at 233.68 105.4163 0)
       (effects (font (size 1.27 1.27)) (justify left))
     )
@@
       (project "meshium_duo"
         (path "/2783b917-8d7b-4d69-a31c-61fb9333015c/4650415e-d772-4f66-8f38-5713f833944e"
-          (reference "C4") (unit 1)
+          (reference "C34") (unit 1)
         )
       )
@@
   (symbol (lib_id "power:+3V3") (at 182.88 43.18 0) (unit 1)
     (in_bom yes) (on_board yes) (dnp no) (fields_autoplaced)
-    (property "Reference" "#PWR05" (at 182.88 46.99 0)
+    (property "Reference" "#PWR052" (at 182.88 46.99 0)
       (effects (font (size 1.27 1.27)) hide)
     )
@@
       (project "meshium_duo"
         (path "/2783b917-8d7b-4d69-a31c-61fb9333015c/4650415e-d772-4f66-8f38-5713f833944e"
-          (reference "#PWR05") (unit 1)
+          (reference "#PWR052") (unit 1)
         )
       )
@@
   (symbol (lib_id "Device:C_Small") (at 87.63 62.23 90) (unit 1)
     (in_bom yes) (on_board yes) (dnp no)
-    (property "Reference" "C1" (at 87.63 57.15 90)
+    (property "Reference" "C31" (at 87.63 57.15 90)
       (effects (font (size 1.27 1.27)))
     )
@@
       (project "meshium_duo"
         (path "/2783b917-8d7b-4d69-a31c-61fb9333015c/4650415e-d772-4f66-8f38-5713f833944e"
-          (reference "C1") (unit 1)
+          (reference "C31") (unit 1)
         )
       )
@@
   (symbol (lib_id "power:GND") (at 213.36 113.03 0) (unit 1)
     (in_bom yes) (on_board yes) (dnp no) (fields_autoplaced)
-    (property "Reference" "#PWR07" (at 213.36 119.38 0)
+    (property "Reference" "#PWR054" (at 213.36 119.38 0)
       (effects (font (size 1.27 1.27)) hide)
     )
@@
       (project "meshium_duo"
         (path "/2783b917-8d7b-4d69-a31c-61fb9333015c/4650415e-d772-4f66-8f38-5713f833944e"
-          (reference "#PWR07") (unit 1)
+          (reference "#PWR054") (unit 1)
         )
       )
@@
   (symbol (lib_id "power:+3V3") (at 231.14 100.33 0) (unit 1)
     (in_bom yes) (on_board yes) (dnp no) (fields_autoplaced)
-    (property "Reference" "#PWR08" (at 231.14 104.14 0)
+    (property "Reference" "#PWR055" (at 231.14 104.14 0)
       (effects (font (size 1.27 1.27)) hide)
     )
@@
       (project "meshium_duo"
         (path "/2783b917-8d7b-4d69-a31c-61fb9333015c/4650415e-d772-4f66-8f38-5713f833944e"
-          (reference "#PWR08") (unit 1)
+          (reference "#PWR055") (unit 1)
         )
       )
@@
   (symbol (lib_id "Device:C_Small") (at 222.25 106.68 0) (unit 1)
     (in_bom yes) (on_board yes) (dnp no) (fields_autoplaced)
-    (property "Reference" "C3" (at 224.79 105.4163 0)
+    (property "Reference" "C33" (at 224.79 105.4163 0)
       (effects (font (size 1.27 1.27)) (justify left))
     )
@@
       (project "meshium_duo"
         (path "/2783b917-8d7b-4d69-a31c-61fb9333015c/4650415e-d772-4f66-8f38-5713f833944e"
-          (reference "C3") (unit 1)
+          (reference "C33") (unit 1)
         )
       )
@@
   (symbol (lib_id "meshium_duo:MX25R3235FM1xx0") (at 82.55 76.2 0) (unit 1)
     (in_bom yes) (on_board yes) (dnp no) (fields_autoplaced)
-    (property "Reference" "U2" (at 91.44 74.93 0)
+    (property "Reference" "U5" (at 91.44 74.93 0)
       (effects (font (size 1.27 1.27)) (justify left))
     )
@@
       (project "meshium_duo"
         (path "/2783b917-8d7b-4d69-a31c-61fb9333015c/4650415e-d772-4f66-8f38-5713f833944e"
-          (reference "U2") (unit 1)
+          (reference "U5") (unit 1)
         )
       )
@@
   (symbol (lib_id "power:GND") (at 91.44 62.23 90) (unit 1)
     (in_bom yes) (on_board yes) (dnp no) (fields_autoplaced)
-    (property "Reference" "#PWR04" (at 97.79 62.23 0)
+    (property "Reference" "#PWR051" (at 97.79 62.23 0)
       (effects (font (size 1.27 1.27)) hide)
     )
@@
       (project "meshium_duo"
         (path "/2783b917-8d7b-4d69-a31c-61fb9333015c/4650415e-d772-4f66-8f38-5713f833944e"
-          (reference "#PWR04") (unit 1)
+          (reference "#PWR051") (unit 1)
         )
       )
@@
   (symbol (lib_id "Device:C_Small") (at 213.36 106.68 0) (unit 1)
     (in_bom yes) (on_board yes) (dnp no) (fields_autoplaced)
-    (property "Reference" "C2" (at 215.9 105.4163 0)
+    (property "Reference" "C32" (at 215.9 105.4163 0)
       (effects (font (size 1.27 1.27)) (justify left))
     )
@@
       (project "meshium_duo"
         (path "/2783b917-8d7b-4d69-a31c-61fb9333015c/4650415e-d772-4f66-8f38-5713f833944e"
-          (reference "C2") (unit 1)
-        )
-      )
+          (reference "C32") (unit 1)
+        )
+      )
