File: HARDWARE/meshium_duo.kicad_sch (KiCad schematic)
At the start: 0 parts

Commit message: schematic capture
Other:
- sheet Ethernet ports: added ETH_REF_CLK, ETH_RST, ETH_RXD0, ETH_RXD1, ETH_RX_EN, ETH_SPI_MISO, ETH_SPI_MOSI, ETH_SPI_NSS, ETH_SPI_SCK, ETH_TXD0, ETH_TXD1, ETH_TX_EN; removed ETH_RMII, ETH_SPI
- sheet MCU ports: added ETH_REF_CLK, ETH_RST, ETH_RXD0, ETH_RXD1, ETH_RX_EN, ETH_SPI_MISO, ETH_SPI_MOSI, ETH_SPI_NSS, ETH_SPI_SCK, ETH_TXD0, ETH_TXD1, ETH_TX_EN, FMC_A[0..12], FMC_BA0, FMC_BA1, FMC_D[0..16], FMC_NBL0, FMC_NBL1, FMC_SDCKE0, FMC_SDCLK, FMC_SDNCAS, FMC_SDNE0, FMC_SDNRAS, FMC_SDNWE, QSPI_BK1_CLK, QSPI_BK1_IO[0..3], QSPI_BK1_NCS; removed ETH_RMII, ETH_SPI, FMS_SDRAM, QSPI
- sheet Memory ports: added FMC_A[0..12], FMC_BA0, FMC_BA1, FMC_D[0..16], FMC_NBL0, FMC_NBL1, FMC_SDCKE0, FMC_SDCLK, FMC_SDNCAS, FMC_SDNE0, FMC_SDNRAS, FMC_SDNWE, QSPI_BK1_CLK, QSPI_BK1_IO[0..3], QSPI_BK1_NCS; removed FMC_SDRAM, QSPI

Commit message: schematic capture
Other:
- sheet MCU ports: added MCO, NRST, STLINK_RX, STLINK_TX, SWO, TCK, TMS; removed none
- sheet ST-Link ports: added MCO, NRST, PWR_EN, STLINK_RX, STLINK_TX, SWO, TCK, TMS; removed none
Changed lines of the file:
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@@
+    (stroke (width 0) (type default))
+  )
+  (wire (pts (xy 127 119.38) (xy 171.45 119.38))
     (stroke (width 0) (type default))
   )
@@
     (stroke (width 0) (type default))
   )
+  (wire (pts (xy 127 132.08) (xy 171.45 132.08))
+    (stroke (width 0) (type default))
+  )
   (wire (pts (xy 215.9 67.31) (xy 260.35 67.31))
     (stroke (width 0) (type default))
@@
     (stroke (width 0) (type default))
   )
+  (wire (pts (xy 127 140.97) (xy 171.45 140.97))
+    (stroke (width 0) (type default))
+  )
   (wire (pts (xy 127 105.41) (xy 171.45 105.41))
     (stroke (width 0) (type default))
@@
     (stroke (width 0) (type default))
   )
+  (wire (pts (xy 127 124.46) (xy 171.45 124.46))
+    (stroke (width 0) (type default))
+  )
   (wire (pts (xy 215.9 85.09) (xy 260.35 85.09))
     (stroke (width 0) (type default))
@@
     (stroke (width 0) (type default))
   )
+  (wire (pts (xy 127 134.62) (xy 171.45 134.62))
+    (stroke (width 0) (type default))
+  )
   (wire (pts (xy 215.9 80.01) (xy 260.35 80.01))
     (stroke (width 0) (type default))
@@
     (stroke (width 0) (type default))
   )
+  (wire (pts (xy 127 127) (xy 171.45 127))
+    (stroke (width 0) (type default))
+  )
   (wire (pts (xy 127 74.93) (xy 171.45 74.93))
     (stroke (width 0) (type default))
@@
   )
   (wire (pts (xy 215.9 90.17) (xy 260.35 90.17))
+    (stroke (width 0) (type default))
+  )
+  (wire (pts (xy 127 121.92) (xy 171.45 121.92))
     (stroke (width 0) (type default))
   )
@@
     )
   )
-  (sheet (at 135.89 165.1) (size 43.18 33.02) (fields_autoplaced)
+  (sheet (at 99.06 116.84) (size 27.94 33.02) (fields_autoplaced)
     (stroke (width 0.1524) (type solid))
     (fill (color 255 255 194 1.0000))
-    (property "Sheetname" "ST-Link" (at 135.89 164.3884 0)
+    (property "Sheetname" "ST-Link" (at 99.06 116.1284 0)
       (effects (font (size 1.27 1.27)) (justify left bottom))
     )
-    (property "Sheetfile" "st-link.kicad_sch" (at 135.89 198.7046 0)
+    (property "Sheetfile" "st-link.kicad_sch" (at 99.06 150.4446 0)
       (effects (font (size 1.27 1.27)) (justify left top))
+    )
+    (pin "PWR_EN" output (at 127 146.05 0)
+      (effects (font (size 1.27 1.27)) (justify right))
+    )
+    (pin "MCO" output (at 127 140.97 0)
+      (effects (font (size 1.27 1.27)) (justify right))
+    )
+    (pin "TMS" bidirectional (at 127 124.46 0)
+      (effects (font (size 1.27 1.27)) (justify right))
+    )
+    (pin "TCK" output (at 127 121.92 0)
+      (effects (font (size 1.27 1.27)) (justify right))
+    )
+    (pin "STLINK_RX" input (at 127 132.08 0)
+      (effects (font (size 1.27 1.27)) (justify right))
+    )
+    (pin "STLINK_TX" output (at 127 134.62 0)
+      (effects (font (size 1.27 1.27)) (justify right))
+    )
+    (pin "SWO" output (at 127 127 0)
+      (effects (font (size 1.27 1.27)) (justify right))
+    )
+    (pin "NRST" output (at 127 119.38 0)
+      (effects (font (size 1.27 1.27)) (justify right))
     )
     (instances
@@
     )
   )
-  (sheet (at 171.45 63.5) (size 44.45 54.61) (fields_autoplaced)
+  (sheet (at 171.45 63.5) (size 44.45 86.36) (fields_autoplaced)
     (stroke (width 0.1524) (type solid))
     (fill (color 255 255 194 1.0000))
@@
       (effects (font (size 1.27 1.27)) (justify left bottom))
     )
-    (property "Sheetfile" "MCU.kicad_sch" (at 171.45 118.6946 0)
+    (property "Sheetfile" "MCU.kicad_sch" (at 171.45 150.4446 0)
       (effects (font (size 1.27 1.27)) (justify left top))
     )
@@
       (effects (font (size 1.27 1.27)) (justify right))
     )
+    (pin "TMS" bidirectional (at 171.45 124.46 180)
+      (effects (font (size 1.27 1.27)) (justify left))
+    )
+    (pin "NRST" input (at 171.45 119.38 180)
+      (effects (font (size 1.27 1.27)) (justify left))
+    )
+    (pin "TCK" input (at 171.45 121.92 180)
+      (effects (font (size 1.27 1.27)) (justify left))
+    )
+    (pin "STLINK_RX" output (at 171.45 132.08 180)
+      (effects (font (size 1.27 1.27)) (justify left))
+    )
+    (pin "SWO" output (at 171.45 127 180)
+      (effects (font (size 1.27 1.27)) (justify left))
+    )
+    (pin "STLINK_TX" input (at 171.45 134.62 180)
+      (effects (font (size 1.27 1.27)) (justify left))
+    )
+    (pin "MCO" input (at 171.45 140.97 180)
+      (effects (font (size 1.27 1.27)) (justify left))
+    )
     (instances

Commit message: schematic capture
Parts:
- added C30, C32: 1u, Capacitor_SMD:C_0603_1608Metric, symbol Device:C_Small
- added C31, C33, C34: 0.1u, Capacitor_SMD:C_0603_1608Metric, symbol Device:C_Small
- added D7: LED_Small, symbol Device:LED_Small
- added J7: Conn_01x02_Pin, Connector_PinHeader_2.54mm:PinHeader_1x02_P2.54mm_Vertical, symbol Connector:Conn_01x02_Pin
- added J8: Conn_02x03_Odd_Even, symbol Connector_Generic:Conn_02x03_Odd_Even
- added JP10 (x2): Jumper_2_Bridged, Jumper:SolderJumper-2_P1.3mm_Open_TrianglePad1.0x1.5mm, symbol Jumper:Jumper_2_Bridged
- added JP3: Jumper_2_Open, Jumper:SolderJumper-2_P1.3mm_Open_TrianglePad1.0x1.5mm, symbol Jumper:Jumper_2_Open
- added R34: 1K, Resistor_SMD:R_0603_1608Metric, symbol Device:R_Small
Connections:
- new net: D7.2 (A), R34.2
- new net: C32.1, C33.1, JP10.1 (A)
- new net: C32.2, C33.2
- new net: C34.1, J8.4 (Pin_4), JP3.2 (B)
- new net +3V3: J7.2 (Pin_2), JP10.1 (A), JP10.2 (B), JP10.2 (B)
- new net +5V: J8.1 (Pin_1), J8.3 (Pin_3), J8.5 (Pin_5), R34.1
- new net +5V0: J8.2 (Pin_2), J8.6 (Pin_6), JP3.1 (A)
- new net GND: C34.2, D7.1 (K)
- new net VDD: J7.1 (Pin_1)
Other:
- added sheet USB (USB.kicad_sch)

Commit message: schematic capture
Parts:
- added C35: 4.7u, Capacitor_Tantalum_SMD:CP_EIA-6032-28_Kemet-C, symbol Device:C_Polarized_Small
- added D8: LED_Small, LED_SMD:LED_0603_1608Metric, symbol Device:LED_Small
- added R35: 1K, Resistor_SMD:R_0603_1608Metric, symbol Device:R_Small
- added R36: 10K, Resistor_SMD:R_0603_1608Metric, symbol Device:R_Small
- added U10: TPS2051B, Package_TO_SOT_SMD:SOT-23-5, symbol meshium_duo:TPS2051B
- D7: footprint (none) -> LED_SMD:LED_0603_1608Metric
Connections:
- net +5V0: now also C35.1, R35.1, R36.1, U10.5 (IN)
- net GND: now also C35.2, U10.2 (GND)
- net ST-Link/PWR_EN: now also R36.2, U10.4 (~{EN})
- net at C34.1, J8.4 (Pin_4), JP3.2 (B): now also U10.1 (OUT)
- new net: D8.1 (K), U10.3 (~{OC})
- new net: D8.2 (A), R35.2
Other:
- added sheet Connectors (Connectors.kicad_sch)
- sheet MCU ports: added BOOT0, PA[0..15], PB[0..15], PC[0..15], PD[0..15], PE[0..15], PG[0..15], USB_DM, USB_DP, USB_GPIO_IN, USB_GPIO_OUT, USB_ID, USB_VBUS; removed none
- sheet USB ports: added USB_DM, USB_DP, USB_ID, USB_OVERCURRENT, USB_POWER_SWITCH_ON, USB_VBUS, USB_VBUS_DET; removed none
- moved on the sheet: C30, C31, C32, C33, C34, D7, J7, J8, JP10, JP3, R34

Commit message: schematic capture
Parts:
- added J18, J19: Conn_01x02_Pin, Connector_PinHeader_2.54mm:PinHeader_1x02_P2.54mm_Vertical, symbol Connector:Conn_01x02_Pin
- J8: footprint (none) -> Connector_PinHeader_2.54mm:PinHeader_2x03_P2.54mm_Vertical
Connections:
- net GND: now also J18.1 (Pin_1), J18.2 (Pin_2), J19.1 (Pin_1), J19.2 (Pin_2)
Changed lines of the file:
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@@
 (kicad_sch (version 20230121) (generator eeschema)
   (paper "A3")
+  (junction (at 252.73 252.73) (diameter 0) (color 0 0 0 0)
+  )
   (junction (at 167.64 208.28) (diameter 0) (color 0 0 0 0)
   )
@@
   (junction (at 198.12 208.28) (diameter 0) (color 0 0 0 0)
   )
+  (junction (at 260.35 252.73) (diameter 0) (color 0 0 0 0)
+  )
   (junction (at 241.3 208.28) (diameter 0) (color 0 0 0 0)
   )
@@
   (junction (at 323.85 209.55) (diameter 0) (color 0 0 0 0)
   )
+  (junction (at 250.19 252.73) (diameter 0) (color 0 0 0 0)
+  )
   (junction (at 158.75 208.28) (diameter 0) (color 0 0 0 0)
   )
@@
     (stroke (width 0) (type default))
   )
+  (wire (pts (xy 250.19 252.73) (xy 250.19 251.46))
+    (stroke (width 0) (type default))
+  )
+  (wire (pts (xy 252.73 252.73) (xy 260.35 252.73))
+    (stroke (width 0) (type default))
+  )
   (wire (pts (xy 215.9 127) (xy 260.35 127))
     (stroke (width 0) (type default))
@@
     (stroke (width 0) (type default))
   )
+  (wire (pts (xy 260.35 252.73) (xy 262.89 252.73))
+    (stroke (width 0) (type default))
+  )
   (wire (pts (xy 331.47 209.55) (xy 337.82 209.55))
     (stroke (width 0) (type default))
@@
     (stroke (width 0) (type default))
   )
+  (wire (pts (xy 252.73 251.46) (xy 252.73 252.73))
+    (stroke (width 0) (type default))
+  )
   (wire (pts (xy 236.22 205.74) (xy 233.68 205.74))
     (stroke (width 0) (type default))
@@
     (stroke (width 0) (type default))
   )
+  (wire (pts (xy 252.73 252.73) (xy 250.19 252.73))
+    (stroke (width 0) (type default))
+  )
   (wire (pts (xy 127 81.28) (xy 171.45 81.28))
     (stroke (width 0) (type default))
@@
     (stroke (width 0) (type default))
   )
+  (wire (pts (xy 250.19 252.73) (xy 250.19 254))
+    (stroke (width 0) (type default))
+  )
   (wire (pts (xy 323.85 204.47) (xy 323.85 209.55))
     (stroke (width 0) (type default))
@@
     (stroke (width 0) (type default))
   )
+  (wire (pts (xy 262.89 252.73) (xy 262.89 251.46))
+    (stroke (width 0) (type default))
+  )
   (wire (pts (xy 158.75 208.28) (xy 158.75 212.09))
     (stroke (width 0) (type default))
@@
   )
   (bus (pts (xy 127 97.79) (xy 171.45 97.79))
+    (stroke (width 0) (type default))
+  )
+  (wire (pts (xy 260.35 251.46) (xy 260.35 252.73))
     (stroke (width 0) (type default))
   )
@@
     )
   )
+  (symbol (lib_id "Connector:Conn_01x02_Pin") (at 262.89 246.38 270) (unit 1)
+    (in_bom yes) (on_board yes) (dnp no) (fields_autoplaced)
+    (property "Reference" "J19" (at 264.16 247.015 90)
+      (effects (font (size 1.27 1.27)) (justify left))
+    )
+    (property "Value" "Conn_01x02_Pin" (at 265.43 247.015 0)
+      (effects (font (size 1.27 1.27)) hide)
+    )
+    (property "Footprint" "Connector_PinHeader_2.54mm:PinHeader_1x02_P2.54mm_Vertical" (at 262.89 246.38 0)
+      (effects (font (size 1.27 1.27)) hide)
+    )
+    (property "Datasheet" "~" (at 262.89 246.38 0)
+      (effects (font (size 1.27 1.27)) hide)
+    )
+    (pin "1")
+    (pin "2")
+    (instances
+      (project "meshium_duo"
+        (path "/2783b917-8d7b-4d69-a31c-61fb9333015c/4c1314f5-8ce3-41c8-9fa4-b5bc01ef554b"
+          (reference "J19") (unit 1)
+        )
+        (path "/2783b917-8d7b-4d69-a31c-61fb9333015c"
+          (reference "J19") (unit 1)
+        )
+      )
+    )
+  )
   (symbol (lib_id "Device:C_Small") (at 264.16 210.82 0) (unit 1)
     (in_bom yes) (on_board yes) (dnp no) (fields_autoplaced)
@@
     )
   )
+  (symbol (lib_id "power:GND") (at 250.19 254 0) (unit 1)
+    (in_bom yes) (on_board yes) (dnp no) (fields_autoplaced)
+    (property "Reference" "#PWR0109" (at 250.19 260.35 0)
+      (effects (font (size 1.27 1.27)) hide)
+    )
+    (property "Value" "GND" (at 250.19 259.08 0)
+      (effects (font (size 1.27 1.27)))
+    )
+    (property "Footprint" "" (at 250.19 254 0)
+      (effects (font (size 1.27 1.27)) hide)
+    )
+    (property "Datasheet" "" (at 250.19 254 0)
+      (effects (font (size 1.27 1.27)) hide)
+    )
+    (pin "1")
+    (instances
+      (project "meshium_duo"
+        (path "/2783b917-8d7b-4d69-a31c-61fb9333015c"
+          (reference "#PWR0109") (unit 1)
+        )
+      )
+    )
+  )
   (symbol (lib_id "power:GND") (at 241.3 224.79 0) (unit 1)
     (in_bom yes) (on_board yes) (dnp no) (fields_autoplaced)
@@
     )
   )
+  (symbol (lib_id "Connector:Conn_01x02_Pin") (at 252.73 246.38 270) (unit 1)
+    (in_bom yes) (on_board yes) (dnp no) (fields_autoplaced)
+    (property "Reference" "J18" (at 254 247.015 90)
+      (effects (font (size 1.27 1.27)) (justify left))
+    )
+    (property "Value" "Conn_01x02_Pin" (at 255.27 247.015 0)
+      (effects (font (size 1.27 1.27)) hide)
+    )
+    (property "Footprint" "Connector_PinHeader_2.54mm:PinHeader_1x02_P2.54mm_Vertical" (at 252.73 246.38 0)
+      (effects (font (size 1.27 1.27)) hide)
+    )
+    (property "Datasheet" "~" (at 252.73 246.38 0)
+      (effects (font (size 1.27 1.27)) hide)
+    )
+    (pin "1")
+    (pin "2")
+    (instances
+      (project "meshium_duo"
+        (path "/2783b917-8d7b-4d69-a31c-61fb9333015c/4c1314f5-8ce3-41c8-9fa4-b5bc01ef554b"
+          (reference "J18") (unit 1)
+        )
+        (path "/2783b917-8d7b-4d69-a31c-61fb9333015c"
+          (reference "J18") (unit 1)
+        )
+      )
+    )
+  )
   (symbol (lib_id "Connector_Generic:Conn_02x03_Odd_Even") (at 228.6 208.28 180) (unit 1)
     (in_bom yes) (on_board yes) (dnp no) (fields_autoplaced)
@@
       (effects (font (size 1.27 1.27)) hide)
     )
-    (property "Footprint" "" (at 228.6 208.28 0)
-      (effects (font (size 1.27 1.27)) hide)
-    )
+    (property "Footprint" "Connector_PinHeader_2.54mm:PinHeader_2x03_P2.54mm_Vertical" (at 228.6 208.28 0)
+      (effects (font (size 1.27 1.27)) hide)
+    )

Commit message: schematic capture
Parts:
- added L1: SDR0604-2R2ML, symbol Device:L_Small
- added U11: ST1S06PUR, symbol meshium_duo:ST1S06PUR
Changed lines of the file:
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@@
+    )
+  )
+  (symbol (lib_id "meshium_duo:ST1S06PUR") (at 312.42 172.72 0) (unit 1)
+    (in_bom yes) (on_board yes) (dnp no) (fields_autoplaced)
+    (property "Reference" "U11" (at 312.42 163.83 0)
+      (effects (font (size 1.27 1.27)))
+    )
+    (property "Value" "ST1S06PUR" (at 312.42 166.37 0)
+      (effects (font (size 1.27 1.27)))
+    )
+    (property "Footprint" "" (at 315.595 181.61 0)
+      (effects (font (size 1.27 1.27) italic) (justify left) hide)
+    )
+    (property "Datasheet" "" (at 313.69 161.29 0)
+      (effects (font (size 1.27 1.27)) hide)
+    )
+    (pin "1")
+    (pin "2")
+    (pin "3")
+    (pin "4")
+    (pin "5")
+    (pin "6")
+    (pin "7")
+    (instances
+      (project "meshium_duo"
+        (path "/2783b917-8d7b-4d69-a31c-61fb9333015c"
+          (reference "U11") (unit 1)
+        )
+      )
     )
   )
@@
         )
       )
+    )
+  )
+  (symbol (lib_id "Device:L_Small") (at 331.47 170.18 90) (unit 1)
+    (in_bom yes) (on_board yes) (dnp no) (fields_autoplaced)
+    (property "Reference" "L1" (at 331.47 165.1 90)
+      (effects (font (size 1.27 1.27)))
+    )
+    (property "Value" "SDR0604-2R2ML" (at 331.47 167.64 90)
+      (effects (font (size 1.27 1.27)))
+    )
+    (property "Footprint" "" (at 331.47 170.18 0)
+      (effects (font (size 1.27 1.27)) hide)
+    )
+    (property "Datasheet" "~" (at 331.47 170.18 0)
+      (effects (font (size 1.27 1.27)) hide)
+    )
+    (pin "1")
+    (pin "2")
+    (instances
+      (project "meshium_duo"
+        (path "/2783b917-8d7b-4d69-a31c-61fb9333015c"
+          (reference "L1") (unit 1)
+        )
+      )

Commit message: schematic capture
Parts:
- removed C32: 1u, Capacitor_SMD:C_0603_1608Metric, symbol Device:C_Small
- removed C33: 0.1u, Capacitor_SMD:C_0603_1608Metric, symbol Device:C_Small
- removed J18, J19: Conn_01x02_Pin, Connector_PinHeader_2.54mm:PinHeader_1x02_P2.54mm_Vertical, symbol Connector:Conn_01x02_Pin
- added C2: 4.7u, Capacitor_SMD:C_0603_1608Metric, symbol Device:C_Small
- added C3: 0.1u, Capacitor_SMD:C_0603_1608Metric, symbol Device:C_Small
- added C5, C8: 22u, Capacitor_SMD:C_0805_2012Metric, symbol Device:C_Small
- added L1: SDR0604-2R2ML, Footpint:L_Bourns-SRN0604, symbol Device:L_Small
- added R?: 15K, Resistor_SMD:R_0603_1608Metric, symbol Device:R_Small
- added R?: 100K, Resistor_SMD:R_0603_1608Metric, symbol Device:R_Small
- added R?: 47K, Resistor_SMD:R_0603_1608Metric, symbol Device:R_Small
- added R?: 19K, Resistor_SMD:R_0603_1608Metric, symbol Device:R_Small
- added U1: ST1S10PUR, Package_DFN_QFN:DFN-8-1EP_4x4mm_P0.8mm_EP2.5x3.6mm, symbol Regulator_Switching:ST1S10PUR
- C6: renamed from C30; value 1u -> 4.7u
- L2: renamed from L1; footprint (none) -> Footpint:L_Bourns-SRN0604
- U3: renamed from U11; footprint (none) -> Package_DFN_QFN:DFN-6-1EP_3x3mm_P0.95mm_EP1.7x2.6mm
- renumbered C35 to C1, C34 to C4, C31 to C7, D8 to D1, D7 to D2, J8 to J1, J7 to J?, JP3 to JP?, JP10 to JP?, R36 to R1, R35 to R2, R34 to R5, U10 to U2
Connections:
- net +5V: now also C6.1, C7.1, U3.4 (VINSW), U3.5 (VINA), U3.6 (INH)
- net +5V0: now also C5.1, L1.2, R?.2
- net GND: now also C6.2, C7.2, U3.2 (GND), U3.7 (PADGND), C2.2, C3.2, C5.2, C8.2, R?.1, R?.1, U1.4 (AGND), U1.5 (SYNC), U1.8 (PGND), U1.9 (PADGND)
- net at JP?.1 (A): now also L2.2, C8.1, R?.2
- net at U3.1 (FB): now also R?.1, R?.2
- net at U3.3 (SW): now also L2.1
- new net: L1.1, U1.7 (SW)
- new net: R?.1, R?.2, U1.3 (FB)
- new net VIN: C2.1, C3.1, U1.1 (VINA), U1.2 (INH), U1.6 (VINSW)
Other:
- moved on the sheet: C1, C4, C6, C7, D1, D2, J1, J?, JP?, L2, R1, R2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
