File: HARDWARE/meshium_duo.kicad_sch (KiCad schematic)
At the start: 27 parts, among them J1 Conn_02x03_Odd_Even, U1 ST1S10PUR, U2 TPS2051B, U3 ST1S06PUR

Commit message: tracerouting
Connections:
- net +3V3: no longer JP?.2 (B)
- net +5V0 renamed U5V
- net U5V: no longer C5.1, J1.2 (Pin_2), J1.6 (Pin_6), L1.2, R?.2
- new net +3V3_PER: JP?.2 (B)
- new net E5V: J1.2 (Pin_2)
- new net VIN_5V: C5.1, J1.6 (Pin_6), L1.2, R?.2
Changed lines of the file:
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@@
+    )
+  )
+  (symbol (lib_name "+3V3_PER_1") (lib_id "meshium_duo:+3V3_PER") (at 359.41 219.71 270) (unit 1)
+    (in_bom yes) (on_board yes) (dnp no) (fields_autoplaced)
+    (property "Reference" "#PWR0154" (at 355.6 219.71 0)
+      (effects (font (size 1.27 1.27)) hide)
+    )
+    (property "Value" "+3V3_PER" (at 363.22 219.71 90)
+      (effects (font (size 1.27 1.27)) (justify left))
+    )
+    (property "Footprint" "" (at 359.41 219.71 0)
+      (effects (font (size 1.27 1.27)) hide)
+    )
+    (property "Datasheet" "" (at 359.41 219.71 0)
+      (effects (font (size 1.27 1.27)) hide)
+    )
+    (pin "1")
+    (instances
+      (project "meshium_duo"
+        (path "/2783b917-8d7b-4d69-a31c-61fb9333015c"
+          (reference "#PWR0154") (unit 1)
+        )
+      )
     )
   )
@@
     )
   )
-  (symbol (lib_id "meshium_duo:+3V3_PER") (at 359.41 219.71 270) (unit 1)
-    (in_bom yes) (on_board yes) (dnp no) (fields_autoplaced)
-    (property "Reference" "#PWR015" (at 355.6 219.71 0)
-      (effects (font (size 1.27 1.27)) hide)
-    )
-    (property "Value" "+3V3_PER" (at 363.22 219.71 90)
-      (effects (font (size 1.27 1.27)) (justify left))
-    )
-    (property "Footprint" "" (at 359.41 219.71 0)
-      (effects (font (size 1.27 1.27)) hide)
-    )
-    (property "Datasheet" "" (at 359.41 219.71 0)
-      (effects (font (size 1.27 1.27)) hide)
-    )
-    (pin "1")
-    (instances
-      (project "meshium_duo"
-        (path "/2783b917-8d7b-4d69-a31c-61fb9333015c"
-          (reference "#PWR015") (unit 1)
-        )
-      )
-    )
-  )
   (symbol (lib_id "Device:R_Small") (at 248.92 217.17 0) (unit 1)
     (in_bom yes) (on_board yes) (dnp no) (fields_autoplaced)
@@
     )
   )
-  (symbol (lib_id "meshium_duo:VIN_5V") (at 226.06 179.07 0) (unit 1)
-    (in_bom yes) (on_board yes) (dnp no) (fields_autoplaced)
-    (property "Reference" "#PWR08" (at 226.06 182.88 0)
-      (effects (font (size 1.27 1.27)) hide)
-    )
-    (property "Value" "VIN_5V" (at 226.06 173.99 0)
-      (effects (font (size 1.27 1.27)))
-    )
-    (property "Footprint" "" (at 226.06 179.07 0)
-      (effects (font (size 1.27 1.27)) hide)
-    )
-    (property "Datasheet" "" (at 226.06 179.07 0)
-      (effects (font (size 1.27 1.27)) hide)
-    )
-    (pin "1")
-    (instances
-      (project "meshium_duo"
-        (path "/2783b917-8d7b-4d69-a31c-61fb9333015c"
-          (reference "#PWR08") (unit 1)
-        )
-      )
-    )
-  )
   (symbol (lib_id "Device:C_Small") (at 265.43 217.17 0) (unit 1)
     (in_bom yes) (on_board yes) (dnp no) (fields_autoplaced)
@@
     )
   )
+  (symbol (lib_name "U5V_1") (lib_id "meshium_duo:U5V") (at 158.75 210.82 0) (unit 1)
+    (in_bom yes) (on_board yes) (dnp no) (fields_autoplaced)
+    (property "Reference" "#PWR0151" (at 158.75 214.63 0)
+      (effects (font (size 1.27 1.27)) hide)
+    )
+    (property "Value" "U5V" (at 158.75 205.74 0)
+      (effects (font (size 1.27 1.27)))
+    )
+    (property "Footprint" "" (at 158.75 210.82 0)
+      (effects (font (size 1.27 1.27)) hide)
+    )
+    (property "Datasheet" "" (at 158.75 210.82 0)
+      (effects (font (size 1.27 1.27)) hide)
+    )
+    (pin "1")
+    (instances
+      (project "meshium_duo"
+        (path "/2783b917-8d7b-4d69-a31c-61fb9333015c"
+          (reference "#PWR0151") (unit 1)
+        )
+      )
+    )
+  )
   (symbol (lib_id "Device:C_Small") (at 162.56 194.31 0) (unit 1)
     (in_bom yes) (on_board yes) (dnp no) (fields_autoplaced)
@@
     )
   )
-  (symbol (lib_id "meshium_duo:E5V") (at 226.06 214.63 90) (unit 1)
-    (in_bom yes) (on_board yes) (dnp no) (fields_autoplaced)
-    (property "Reference" "#PWR09" (at 229.87 214.63 0)
-      (effects (font (size 1.27 1.27)) hide)
-    )
-    (property "Value" "E5V" (at 222.25 214.63 90)
-      (effects (font (size 1.27 1.27)) (justify left))
-    )
-    (property "Footprint" "" (at 226.06 214.63 0)
-      (effects (font (size 1.27 1.27)) hide)
-    )
-    (property "Datasheet" "" (at 226.06 214.63 0)
-      (effects (font (size 1.27 1.27)) hide)
-    )
-    (pin "1")
-    (instances
-      (project "meshium_duo"
-        (path "/2783b917-8d7b-4d69-a31c-61fb9333015c"
-          (reference "#PWR09") (unit 1)
-        )
-      )
-    )
-  )
-  (symbol (lib_id "meshium_duo:U5V") (at 158.75 210.82 0) (unit 1)
-    (in_bom yes) (on_board yes) (dnp no) (fields_autoplaced)
-    (property "Reference" "#PWR04" (at 158.75 214.63 0)
-      (effects (font (size 1.27 1.27)) hide)
-    )
-    (property "Value" "U5V" (at 158.75 205.74 0)
-      (effects (font (size 1.27 1.27)))
-    )
-    (property "Footprint" "" (at 158.75 210.82 0)
-      (effects (font (size 1.27 1.27)) hide)
-    )
-    (property "Datasheet" "" (at 158.75 210.82 0)
-      (effects (font (size 1.27 1.27)) hide)
-    )
-    (pin "1")
-    (instances
-      (project "meshium_duo"
-        (path "/2783b917-8d7b-4d69-a31c-61fb9333015c"
-          (reference "#PWR04") (unit 1)
-        )
-      )
-    )
-  )
   (symbol (lib_id "power:+3V3") (at 345.44 207.01 0) (unit 1)
     (in_bom yes) (on_board yes) (dnp no) (fields_autoplaced)
@@
         (path "/2783b917-8d7b-4d69-a31c-61fb9333015c"
           (reference "#PWR013") (unit 1)
-        )
-      )
-    )
-  )
-  (symbol (lib_id "meshium_duo:VIN") (at 149.86 182.88 90) (unit 1)
-    (in_bom yes) (on_board yes) (dnp no) (fields_autoplaced)
-    (property "Reference" "#PWR01" (at 153.67 182.88 0)
-      (effects (font (size 1.27 1.27)) hide)
-    )
-    (property "Value" "VIN" (at 146.05 182.88 90)
-      (effects (font (size 1.27 1.27)) (justify left))
-    )
-    (property "Footprint" "" (at 149.86 182.88 0)
-      (effects (font (size 1.27 1.27)) hide)
-    )
-    (property "Datasheet" "" (at 149.86 182.88 0)
-      (effects (font (size 1.27 1.27)) hide)
-    )
-    (pin "1")
-    (instances
-      (project "meshium_duo"
-        (path "/2783b917-8d7b-4d69-a31c-61fb9333015c"
-          (reference "#PWR01") (unit 1)
         )
       )
@@
         (path "/2783b917-8d7b-4d69-a31c-61fb9333015c"
           (reference "C5") (unit 1)
+        )
+      )
+    )
+  )
+  (symbol (lib_name "E5V_1") (lib_id "meshium_duo:E5V") (at 226.06 214.63 90) (unit 1)
+    (in_bom yes) (on_board yes) (dnp no) (fields_autoplaced)
+    (property "Reference" "#PWR0153" (at 229.87 214.63 0)
+      (effects (font (size 1.27 1.27)) hide)
+    )
+    (property "Value" "E5V" (at 222.25 214.63 90)
+      (effects (font (size 1.27 1.27)) (justify left))
+    )
+    (property "Footprint" "" (at 226.06 214.63 0)
+      (effects (font (size 1.27 1.27)) hide)
+    )
+    (property "Datasheet" "" (at 226.06 214.63 0)
+      (effects (font (size 1.27 1.27)) hide)
+    )
+    (pin "1")
+    (instances
+      (project "meshium_duo"
+        (path "/2783b917-8d7b-4d69-a31c-61fb9333015c"
+          (reference "#PWR0153") (unit 1)
         )
       )
@@
         (path "/2783b917-8d7b-4d69-a31c-61fb9333015c"
           (reference "R2") (unit 1)
+        )
+      )
+    )
+  )
+  (symbol (lib_id "meshium_duo:VIN") (at 149.86 182.88 90) (unit 1)
+    (in_bom yes) (on_board yes) (dnp no) (fields_autoplaced)
+    (property "Reference" "#PWR0150" (at 153.67 182.88 0)
+      (effects (font (size 1.27 1.27)) hide)
+    )
+    (property "Value" "VIN" (at 146.05 182.88 90)
+      (effects (font (size 1.27 1.27)) (justify left))
+    )
+    (property "Footprint" "" (at 149.86 182.88 0)
+      (effects (font (size 1.27 1.27)) hide)
+    )
+    (property "Datasheet" "" (at 149.86 182.88 0)
+      (effects (font (size 1.27 1.27)) hide)
+    )
+    (pin "1")
+    (instances
+      (project "meshium_duo"
+        (path "/2783b917-8d7b-4d69-a31c-61fb9333015c"
+          (reference "#PWR0150") (unit 1)
         )
       )
@@
         )
       )
+    )
+  )
+  (symbol (lib_name "VIN_5V_1") (lib_id "meshium_duo:VIN_5V") (at 226.06 179.07 0) (unit 1)
+    (in_bom yes) (on_board yes) (dnp no) (fields_autoplaced)
+    (property "Reference" "#PWR0152" (at 226.06 182.88 0)
+      (effects (font (size 1.27 1.27)) hide)
+    )
+    (property "Value" "VIN_5V" (at 226.06 173.99 0)
+      (effects (font (size 1.27 1.27)))
+    )
+    (property "Footprint" "" (at 226.06 179.07 0)
+      (effects (font (size 1.27 1.27)) hide)
+    )
+    (property "Datasheet" "" (at 226.06 179.07 0)
+      (effects (font (size 1.27 1.27)) hide)
+    )
+    (pin "1")
+    (instances
+      (project "meshium_duo"
+        (path "/2783b917-8d7b-4d69-a31c-61fb9333015c"
+          (reference "#PWR0152") (unit 1)
+        )
+      )

Commit message: tracerouting
Parts:
- gave numbers to parts that had none: 8
Changed lines of the file:
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@@
   (symbol (lib_id "Device:R_Small") (at 312.42 223.52 0) (mirror x) (unit 1)
     (in_bom yes) (on_board yes) (dnp no)
-    (property "Reference" "R?" (at 317.5 222.25 0)
+    (property "Reference" "R6" (at 317.5 222.25 0)
       (effects (font (size 1.27 1.27)) (justify right))
     )
@@
     (instances
       (project "meshium_duo"
-        (path "/2783b917-8d7b-4d69-a31c-61fb9333015c/4c1314f5-8ce3-41c8-9fa4-b5bc01ef554b"
-          (reference "R?") (unit 1)
-        )
-        (path "/2783b917-8d7b-4d69-a31c-61fb9333015c/191f4f98-48ae-4893-bf0a-75f1c9b9512d"
-          (reference "R?") (unit 1)
-        )
         (path "/2783b917-8d7b-4d69-a31c-61fb9333015c"
           (reference "R6") (unit 1)
@@
   (symbol (lib_id "Jumper:Jumper_2_Open") (at 190.5 212.09 0) (unit 1)
     (in_bom yes) (on_board yes) (dnp no) (fields_autoplaced)
-    (property "Reference" "JP?" (at 190.5 208.28 0)
+    (property "Reference" "JP1" (at 190.5 208.28 0)
       (effects (font (size 1.27 1.27)))
     )
@@
     (instances
       (project "meshium_duo"
-        (path "/2783b917-8d7b-4d69-a31c-61fb9333015c/4c1314f5-8ce3-41c8-9fa4-b5bc01ef554b"
-          (reference "JP?") (unit 1)
-        )
         (path "/2783b917-8d7b-4d69-a31c-61fb9333015c"
           (reference "JP1") (unit 1)
@@
   (symbol (lib_id "Device:R_Small") (at 208.28 187.96 90) (mirror x) (unit 1)
     (in_bom yes) (on_board yes) (dnp no)
-    (property "Reference" "R?" (at 208.28 185.42 90)
+    (property "Reference" "R4" (at 208.28 185.42 90)
       (effects (font (size 1.27 1.27)))
     )
@@
     (instances
       (project "meshium_duo"
-        (path "/2783b917-8d7b-4d69-a31c-61fb9333015c/4c1314f5-8ce3-41c8-9fa4-b5bc01ef554b"
-          (reference "R?") (unit 1)
-        )
-        (path "/2783b917-8d7b-4d69-a31c-61fb9333015c/191f4f98-48ae-4893-bf0a-75f1c9b9512d"
-          (reference "R?") (unit 1)
-        )
         (path "/2783b917-8d7b-4d69-a31c-61fb9333015c"
           (reference "R4") (unit 1)
@@
   (symbol (lib_id "Device:R_Small") (at 318.77 219.71 90) (mirror x) (unit 1)
     (in_bom yes) (on_board yes) (dnp no) (fields_autoplaced)
-    (property "Reference" "R?" (at 318.77 214.63 90)
+    (property "Reference" "R7" (at 318.77 214.63 90)
       (effects (font (size 1.27 1.27)))
     )
@@
     (instances
       (project "meshium_duo"
-        (path "/2783b917-8d7b-4d69-a31c-61fb9333015c/4c1314f5-8ce3-41c8-9fa4-b5bc01ef554b"
-          (reference "R?") (unit 1)
-        )
-        (path "/2783b917-8d7b-4d69-a31c-61fb9333015c/191f4f98-48ae-4893-bf0a-75f1c9b9512d"
-          (reference "R?") (unit 1)
-        )
         (path "/2783b917-8d7b-4d69-a31c-61fb9333015c"
           (reference "R7") (unit 1)
@@
   (symbol (lib_id "Device:R_Small") (at 201.93 191.77 0) (mirror x) (unit 1)
     (in_bom yes) (on_board yes) (dnp no)
-    (property "Reference" "R?" (at 200.66 190.5 0)
+    (property "Reference" "R3" (at 200.66 190.5 0)
       (effects (font (size 1.27 1.27)) (justify right))
     )
@@
     (instances
       (project "meshium_duo"
-        (path "/2783b917-8d7b-4d69-a31c-61fb9333015c/4c1314f5-8ce3-41c8-9fa4-b5bc01ef554b"
-          (reference "R?") (unit 1)
-        )
-        (path "/2783b917-8d7b-4d69-a31c-61fb9333015c/191f4f98-48ae-4893-bf0a-75f1c9b9512d"
-          (reference "R?") (unit 1)
-        )
         (path "/2783b917-8d7b-4d69-a31c-61fb9333015c"
           (reference "R3") (unit 1)
@@
   (symbol (lib_id "Jumper:Jumper_2_Bridged") (at 337.82 212.09 0) (unit 1)
     (in_bom yes) (on_board yes) (dnp no) (fields_autoplaced)
-    (property "Reference" "JP?" (at 337.82 209.55 0)
+    (property "Reference" "JP2" (at 337.82 209.55 0)
       (effects (font (size 1.27 1.27)))
     )
@@
     (instances
       (project "meshium_duo"
-        (path "/2783b917-8d7b-4d69-a31c-61fb9333015c/4c1314f5-8ce3-41c8-9fa4-b5bc01ef554b"
-          (reference "JP?") (unit 1)
-        )
         (path "/2783b917-8d7b-4d69-a31c-61fb9333015c"
           (reference "JP2") (unit 1)
@@
   (symbol (lib_id "Jumper:Jumper_2_Bridged") (at 351.79 219.71 0) (unit 1)
     (in_bom yes) (on_board yes) (dnp no) (fields_autoplaced)
-    (property "Reference" "JP?" (at 351.79 217.17 0)
+    (property "Reference" "JP3" (at 351.79 217.17 0)
       (effects (font (size 1.27 1.27)))
     )
@@
     (instances
       (project "meshium_duo"
-        (path "/2783b917-8d7b-4d69-a31c-61fb9333015c/4c1314f5-8ce3-41c8-9fa4-b5bc01ef554b"
-          (reference "JP?") (unit 1)
-        )
         (path "/2783b917-8d7b-4d69-a31c-61fb9333015c"
           (reference "JP3") (unit 1)
@@
   (symbol (lib_id "Connector:Conn_01x02_Pin") (at 353.06 207.01 270) (unit 1)
     (in_bom yes) (on_board yes) (dnp no) (fields_autoplaced)
-    (property "Reference" "J?" (at 354.33 207.645 90)
+    (property "Reference" "J2" (at 354.33 207.645 90)
       (effects (font (size 1.27 1.27)) (justify left))
     )
@@
     (instances
       (project "meshium_duo"
-        (path "/2783b917-8d7b-4d69-a31c-61fb9333015c/4c1314f5-8ce3-41c8-9fa4-b5bc01ef554b"
-          (reference "J?") (unit 1)
-        )
         (path "/2783b917-8d7b-4d69-a31c-61fb9333015c"
           (reference "J2") (unit 1)
