File: HARDWARE/MCU.kicad_sch (KiCad schematic)
At the start: 1 part, among them U1 STM32F767ZITx

Commit message: pcb creation
Changed lines of the file:
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@@
-    (stroke (width 0) (type default))
-  )
-  (wire (pts (xy 109.22 93.98) (xy 123.19 93.98))
     (stroke (width 0) (type default))
   )
@@
     (effects (font (size 1.27 1.27)) (justify right bottom))
   )
-  (label "FMC_D0" (at 123.19 93.98 180) (fields_autoplaced)
-    (effects (font (size 1.27 1.27)) (justify right bottom))
-  )
   (label "FMC_D15" (at 157.48 210.82 0) (fields_autoplaced)
     (effects (font (size 1.27 1.27)) (justify left bottom))
@@
     (effects (font (size 1.27 1.27)) (justify left bottom))
   )
+  (global_label "FMC_D0" (shape input) (at 157.48 220.98 180) (fields_autoplaced)
+    (effects (font (size 1.27 1.27)) (justify right))
+    (property "Intersheetrefs" "${INTERSHEET_REFS}" (at 147.2377 220.98 0)
+      (effects (font (size 1.27 1.27)) (justify right) hide)
+    )
+  )
   (hierarchical_label "ETH_SPI" (shape bidirectional) (at 46.99 127 180) (fields_autoplaced)

Commit message: schematic capture
Parts:
- renumbered U1 to U?
Connections:
- net SDMMC1_CK: no longer names the net of U?.113 (PC12)
- net SDMMC1_CMD: no longer names the net of U?.116 (PD2)
- net SDMMC1_D0: no longer names the net of U?.98 (PC8)
- net SDMMC1_D1: no longer names the net of U?.99 (PC9)
- net SDMMC1_D2: no longer names the net of U?.111 (PC10)
- net SDMMC1_D3: no longer names the net of U?.112 (PC11)

Commit message: schematic capture
Parts:
- added JP10: Jumper_2_Bridged, symbol Jumper:Jumper_2_Bridged
Connections:
- net ETH_SPI1_MISO is gone; now on net ETH_SPI_MISO: U?.42 (PA6)
- net ETH_SPI1_MOSI is gone; now on net ETH_SPI_MOSI: U?.123 (PD7)
- net ETH_SPI1_NSS is gone; now on net ETH_SPI_NSS: U?.40 (PA4)
- net ETH_SPI1_SCK is gone; now on net ETH_SPI_SCK: U?.41 (PA5)
- net QSPI_BK1_IO2: now also U?.19 (PF7)
- net RCC_OSC_IN: now also JP10.1 (A)
- net TMS: now reaches U?.105 (PA13)
- net TCK: now reaches U?.109 (PA14)
- net SWO: now reaches U?.133 (PB3)
- net NRST: now reaches U?.25 (NRST)
- new net MCO: JP10.2 (B)

Commit message: schematic capture
Changed lines of the file:
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@@
+    (stroke (width 0) (type default))
+  )
+  (wire (pts (xy 149.86 83.82) (xy 175.26 83.82))
     (stroke (width 0) (type default))
   )
@@
     (stroke (width 0) (type default))
   )
+  (wire (pts (xy 149.86 81.28) (xy 175.26 81.28))
+    (stroke (width 0) (type default))
+  )
   (wire (pts (xy 50.8 60.96) (xy 67.31 60.96))
     (stroke (width 0) (type default))
@@
     (stroke (width 0) (type default))
   )
+  (wire (pts (xy 149.86 76.2) (xy 175.26 76.2))
+    (stroke (width 0) (type default))
+  )
   (wire (pts (xy 157.48 58.42) (xy 175.26 58.42))
     (stroke (width 0) (type default))
@@
     (stroke (width 0) (type default))
   )
+  (wire (pts (xy 149.86 93.98) (xy 175.26 93.98))
+    (stroke (width 0) (type default))
+  )
   (wire (pts (xy 368.3 170.18) (xy 382.27 170.18))
     (stroke (width 0) (type default))
@@
     (stroke (width 0) (type default))
   )
+  (wire (pts (xy 149.86 86.36) (xy 175.26 86.36))
+    (stroke (width 0) (type default))
+  )
   (wire (pts (xy 157.48 66.04) (xy 175.26 66.04))
     (stroke (width 0) (type default))
@@
     (stroke (width 0) (type default))
   )
+  (wire (pts (xy 149.86 60.96) (xy 175.26 60.96))
+    (stroke (width 0) (type default))
+  )
   (wire (pts (xy 236.22 76.2) (xy 254 76.2))
     (stroke (width 0) (type default))
@@
     (stroke (width 0) (type default))
   )
+  (wire (pts (xy 149.86 63.5) (xy 175.26 63.5))
+    (stroke (width 0) (type default))
+  )
   (bus (pts (xy 368.3 205.74) (xy 368.3 203.2))
     (stroke (width 0) (type default))
   )
+  (wire (pts (xy 149.86 55.88) (xy 175.26 55.88))
+    (stroke (width 0) (type default))
+  )
   (wire (pts (xy 157.48 203.2) (xy 175.26 203.2))
     (stroke (width 0) (type default))
@@
     (stroke (width 0) (type default))
   )
+  (wire (pts (xy 149.86 78.74) (xy 175.26 78.74))
+    (stroke (width 0) (type default))
+  )

Commit message: schematic capture
Parts:
- added J7: Conn_01x02_Pin, Connector_PinHeader_2.54mm:PinHeader_1x02_P2.54mm_Vertical, symbol Connector:Conn_01x02_Pin
- added JP10 (x7): Jumper_2_Bridged, Jumper:SolderJumper-2_P1.3mm_Open_TrianglePad1.0x1.5mm, symbol Jumper:Jumper_2_Bridged
- added JP9 (x2): Jumper_2_Open, Jumper:SolderJumper-2_P1.3mm_Open_TrianglePad1.0x1.5mm, symbol Jumper:Jumper_2_Open
- added R12: 10K, Resistor_SMD:R_0603_1608Metric, symbol Device:R_Small
- JP10: footprint (none) -> Jumper:SolderJumper-2_P1.3mm_Open_TrianglePad1.0x1.5mm
Connections:
- net STLINK_RX: now also JP10.1 (A)
- net STLINK_TX: now also JP10.1 (A)
- net SWO: now also JP10.1 (A); no longer U?.133 (PB3)
- net TCK: now also JP10.1 (A); no longer U?.109 (PA14)
- net TMS: now also JP10.1 (A); no longer U?.105 (PA13)
- net PA8: now reaches U?.100 (PA8)
- net PA9: now reaches U?.101 (PA9)
- net PA9: now also JP9.2 (B)
- net PA10: now reaches U?.102 (PA10)
- net PA10: now also JP9.2 (B)
- net PA11: now reaches U?.103 (PA11)
- net PA11: now also JP10.2 (B)
- net PA12: now reaches U?.104 (PA12)
- net PA12: now also JP10.2 (B)
- net PA15: now reaches U?.110 (PA15)
- net PC10: now reaches U?.111 (PC10)
- net PC11: now reaches U?.112 (PC11)
- net PC12: now reaches U?.113 (PC12)
- net PD2: now reaches U?.116 (PD2)
- net PD3: now reaches U?.117 (PD3)
- net PD4: now reaches U?.118 (PD4)
- net PD5: now reaches U?.119 (PD5)
- net PD6: now reaches U?.122 (PD6)
- net PG9: now reaches U?.124 (PG9)
- net PG10: now reaches U?.125 (PG10)
- net PG11: now reaches U?.126 (PG11)
- net PG12: now reaches U?.127 (PG12)
- net PG13: now reaches U?.128 (PG13)
- net PG14: now reaches U?.129 (PG14)
- net PB4: now reaches U?.134 (PB4)
- net PB5: now reaches U?.135 (PB5)
- net PB6: now reaches U?.136 (PB6)
- net PB7: now reaches U?.137 (PB7)
- net PB8: now reaches U?.139 (PB8)
- net PB9: now reaches U?.140 (PB9)
- net PE3: now reaches U?.2 (PE3)
- net PC1: now reaches U?.27 (PC1)
- net PE4: now reaches U?.3 (PE4)
- net PA0: now reaches U?.34 (PA0)
- net PA2: now reaches U?.36 (PA2)
- net PA3: now reaches U?.37 (PA3)
- net PE5: now reaches U?.4 (PE5)
- net PB0: now reaches U?.46 (PB0)
- net PB1: now reaches U?.47 (PB1)
- net PB2: now reaches U?.48 (PB2)
- net PE6: now reaches U?.5 (PE6)
- net PC13: now reaches U?.7 (PC13)
- net PB14: now reaches U?.75 (PB14)
- net PB15: now reaches U?.76 (PB15)
- net PC14: now reaches U?.8 (PC14)
- net PD11: now reaches U?.80 (PD11)
- net PD12: now reaches U?.81 (PD12)
- net PD13: now reaches U?.82 (PD13)
- net PG3: now reaches U?.88 (PG3)
- net PC15: now reaches U?.9 (PC15)
- net USB_GPIO_OUT: now reaches U?.91 (PG6)
- net PG7: now reaches U?.92 (PG7)
- net PG7: now also J7.2 (Pin_2)
- net PC6: now reaches U?.96 (PC6)
- net PC7: now reaches U?.97 (PC7)
- net PC8: now reaches U?.98 (PC8)
- net PC9: now reaches U?.99 (PC9)
- new net: JP9.1 (A), R12.2
- new net PA13: JP10.2 (B), U?.105 (PA13)
- new net PA14: JP10.2 (B), U?.109 (PA14)
- new net PB3: JP10.2 (B), U?.133 (PB3)
- new net USB_DM: JP10.1 (A)
- new net USB_DP: JP10.1 (A)
- new net USB_GPIO_IN: J7.1 (Pin_1)
- new net USB_ID: JP9.1 (A)
- new net USB_VBUS: R12.1
Other:
- moved on the sheet: JP10, U?

Commit message: schematic capture
Parts:
- added C11 (x14), C16: 0.1u, Capacitor_SMD:C_0603_1608Metric, symbol Device:C_Small
- added C11: 4.7u, Capacitor_SMD:C_0603_1608Metric, symbol Device:C_Small
- added C16, C17: 10p, Capacitor_SMD:C_0603_1608Metric, symbol Device:C_Small
- added C16, C17: 2p, Capacitor_SMD:C_0603_1608Metric, symbol Device:C_Small
- added C36, C38: 2.2u, Capacitor_SMD:C_0805_2012Metric, symbol Device:C_Small
- added D8 (x2): LED_Small, LED_SMD:LED_0603_1608Metric, symbol Device:LED_Small
- added FB1: FerriteBead_Small, Capacitor_SMD:C_0603_1608Metric, symbol Device:FerriteBead_Small
- added JP10 (x8): Jumper_2_Bridged, Jumper:SolderJumper-2_P1.3mm_Open_TrianglePad1.0x1.5mm, symbol Jumper:Jumper_2_Bridged
- added JP9 (x4): Jumper_2_Open, Jumper:SolderJumper-2_P1.3mm_Open_TrianglePad1.0x1.5mm, symbol Jumper:Jumper_2_Open
- added R12: 10K, Resistor_SMD:R_0603_1608Metric, symbol Device:R_Small
- added R35: 220K, Resistor_SMD:R_0603_1608Metric, symbol Device:R_Small
- added R35 (x2): 1K, Resistor_SMD:R_0603_1608Metric, symbol Device:R_Small
- added R35: 680, Resistor_SMD:R_0603_1608Metric, symbol Device:R_Small
- added SW1, SW2: SW_Push_Dual, symbol Switch:SW_Push_Dual
- added Y2: 25 MHz, Crystal:Crystal_SMD_3225-4Pin_3.2x2.5mm, symbol Device:Crystal_Small
- added Y2: 32.768 kHz, Crystal:Crystal_SMD_3215-2Pin_3.2x1.5mm, symbol Device:Crystal_Small
Connections:
- net BOOT0: now also U?.138 (BOOT0), JP10.1 (A), JP10.2 (B), R12.1
- net GND: now also C11.1, C11.1, C11.1, C11.1, C11.1, C11.1, C11.1, C11.1, C11.1, C11.1, C11.1, C11.1, C11.1, C11.1, C11.1, C16.1, C16.1, C16.1, C17.1, C17.1, C36.2, C38.2, D8.1 (K), D8.1 (K), JP10.1 (A), R12.2, R35.1, SW2.2, SW2.4; no longer U?.31 (VSSA)
- net NRST: now also C16.2, JP10.1 (A), JP10.2 (B), SW2.1, SW2.3
- net PB7: now also JP10.2 (B), JP10.2 (B)
- net PC13: now also JP10.2 (B)
- net PC14: now also JP9.1 (A)
- net PC15: now also JP9.1 (A)
- net at U?.106 (VCAP_2): now also C36.1
- net VDD: now reaches U?.108 (VDD)
- net VDD: now also U?.121 (VDDSDMMC), U?.131 (VDD), U?.143 (PDR_ON), U?.144 (VDD), U?.17 (VDD), U?.30 (VDD), U?.39 (VDD), U?.52 (VDD), U?.62 (VDD), U?.72 (VDD), U?.84 (VDD), U?.95 (VDDUSB), C11.2, C11.2, C11.2, C11.2, C11.2, C11.2, C11.2, C11.2, C11.2, C11.2, C11.2, C11.2, C11.2, FB1.1, JP10.1 (A), SW1.2, SW1.4
- net VDDA: now reaches U?.32 (VREF+)
- net VDDA: now also U?.33 (VDDA), C11.2, JP10.1 (A)
- net VBAT: now reaches U?.6 (VBAT)
- net VBAT: now also C11.2, JP10.2 (B)
- net at U?.71 (VCAP_1): now also C38.1
- net RCC_OSC_IN renamed PH0
- net PH0: now also JP9.1 (A)
- net RCC_OSC_OUT renamed PH1
- net PH1: now also JP9.1 (A)
- new net: FB1.2, JP10.2 (B)
- new net: C16.2, JP9.2 (B), Y2.1 (x2)
- new net: C17.2, JP9.2 (B), Y2.3 (x2)
- new net: JP10.1 (A), R35.1 (x3)
- new net: D8.2 (A), R35.2 (x2)
- new net: R35.2, R35.2, SW1.1, SW1.3
- new net GNDA: JP10.2 (B), U?.31 (VSSA)

Commit message: schematic capture
Parts:
- renumbered C36 to C22, C38 to C23, C11 to C?, C17 to C?, C16 to C?, D8 to D?, FB1 to FB?, J7 to J?, JP10 to JP?, JP9 to JP?, R12 to R?, R35 to R?, Y2 to Y?
Other:
- moved on the sheet: C?, D?, J?, JP?, R?, SW1, SW2
