File: HARDWARE/MCU.kicad_sch (KiCad schematic)
At the start: 59 parts, among them SW1 SW_Push_Dual, SW2 SW_Push_Dual

Commit message: tracerouting
Parts:
- removed Y?: 25 MHz, Crystal:Crystal_SMD_3225-4Pin_3.2x2.5mm, symbol Device:Crystal_Small
- added Y1: 25MHz, Crystal:Crystal_SMD_3225-4Pin_3.2x2.5mm, symbol Device:Crystal_GND24_Small
Connections:
- net GND: now also Y1.2, Y1.4
- net at C?.2, JP?.2 (B): now also Y1.3
- net at C?.2, JP?.2 (B): now also Y1.1
Changed lines of the file:
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@@
   (junction (at 203.2 255.27) (diameter 0) (color 0 0 0 0)
   )
+  (junction (at 367.03 41.91) (diameter 0) (color 0 0 0 0)
+  )
   (junction (at 177.8 265.43) (diameter 0) (color 0 0 0 0)
   )
@@
     (stroke (width 0) (type default))
   )
+  (wire (pts (xy 365.76 41.91) (xy 367.03 41.91))
+    (stroke (width 0) (type default))
+  )
   (wire (pts (xy 242.57 106.68) (xy 267.97 106.68))
     (stroke (width 0) (type default))
   )
+  (wire (pts (xy 359.41 41.91) (xy 359.41 38.1))
+    (stroke (width 0) (type default))
+  )
   (wire (pts (xy 85.09 140.97) (xy 96.52 140.97))
     (stroke (width 0) (type default))
@@
     (stroke (width 0) (type default))
   )
+  (wire (pts (xy 359.41 38.1) (xy 367.03 38.1))
+    (stroke (width 0) (type default))
+  )
   (wire (pts (xy 369.57 95.25) (xy 372.11 95.25))
     (stroke (width 0) (type default))
@@
     (stroke (width 0) (type default))
   )
+  (wire (pts (xy 367.03 41.91) (xy 373.38 41.91))
+    (stroke (width 0) (type default))
+  )
   (wire (pts (xy 50.8 222.25) (xy 96.52 222.25))
     (stroke (width 0) (type default))
@@
     (stroke (width 0) (type default))
   )
+  (wire (pts (xy 367.03 38.1) (xy 367.03 41.91))
+    (stroke (width 0) (type default))
+  )
   (bus (pts (xy 153.67 215.9) (xy 153.67 213.36))
     (stroke (width 0) (type default))
@@
     (stroke (width 0) (type default))
   )
+  (wire (pts (xy 360.68 41.91) (xy 359.41 41.91))
+    (stroke (width 0) (type default))
+  )
   (wire (pts (xy 163.83 185.42) (xy 181.61 185.42))
     (stroke (width 0) (type default))
@@
     )
   )
-  (symbol (lib_id "Device:Crystal_Small") (at 363.22 41.91 270) (unit 1)
-    (in_bom yes) (on_board yes) (dnp no)
-    (property "Reference" "Y?" (at 359.41 40.64 90)
-      (effects (font (size 1.27 1.27)))
-    )
-    (property "Value" "25 MHz" (at 358.14 43.18 90)
-      (effects (font (size 1.27 1.27)))
-    )
-    (property "Footprint" "Crystal:Crystal_SMD_3225-4Pin_3.2x2.5mm" (at 363.22 41.91 0)
-      (effects (font (size 1.27 1.27)) hide)
-    )
-    (property "Datasheet" "~" (at 363.22 41.91 0)
-      (effects (font (size 1.27 1.27)) hide)
-    )
-    (pin "1")
-    (pin "3")
-    (instances
-      (project "meshium_duo"
-        (path "/2783b917-8d7b-4d69-a31c-61fb9333015c/4c1314f5-8ce3-41c8-9fa4-b5bc01ef554b"
-          (reference "Y?") (unit 1)
-        )
-        (path "/2783b917-8d7b-4d69-a31c-61fb9333015c/b5f76ac1-5f31-46a3-a641-c3c4fe73e10b"
-          (reference "Y1") (unit 1)
-        )
-      )
-    )
-  )
   (symbol (lib_id "Jumper:Jumper_2_Open") (at 353.06 64.77 0) (unit 1)
     (in_bom yes) (on_board yes) (dnp no)
@@
         )
       )
+    )
+  )
+  (symbol (lib_id "Device:Crystal_GND24_Small") (at 363.22 41.91 90) (unit 1)
+    (in_bom yes) (on_board yes) (dnp no)
+    (property "Reference" "Y1" (at 356.87 41.91 90)
+      (effects (font (size 1.27 1.27)))
+    )
+    (property "Value" "25MHz" (at 358.14 44.45 90)
+      (effects (font (size 1 1)))
+    )
+    (property "Footprint" "Crystal:Crystal_SMD_3225-4Pin_3.2x2.5mm" (at 363.22 41.91 0)
+      (effects (font (size 1.27 1.27)) hide)
+    )
+    (property "Datasheet" "~" (at 363.22 41.91 0)
+      (effects (font (size 1.27 1.27)) hide)
+    )
+    (pin "2")
+    (pin "1")
+    (pin "3")
+    (pin "4")
+    (instances
+      (project "meshium_duo"
+        (path "/2783b917-8d7b-4d69-a31c-61fb9333015c/b5f76ac1-5f31-46a3-a641-c3c4fe73e10b"
+          (reference "Y1") (unit 1)
+        )
+      )

Commit message: tracerouting
Parts:
- gave numbers to parts that had none: 54
Connections:
- net VCAP1: now reaches C23.1, U4.71 (VCAP_1)
- net VCAP2: now reaches C22.1, U4.106 (VCAP_2)
