File: HARDWARE/meshium_duo.kicad_pcb (KiCad board)
At the start: 2 copper layers, 25 parts, among them J1 RJ45_Wuerth_7499151120, Q1 BC848, U1 STM32F767ZITx, U2 MX25L3233FZN, U3 MT48LC16M16A2P, U4 KSZ8463FRL, U5 STM32F103CBTx, U6 LD3985M33R_SOT23

Commit message: schematic capture
Parts:
- removed J1: RJ45_Wuerth_7499151120, Connector_RJ:RJ45_Wuerth_7499151120_Horizontal
- U2: value MX25L3233FZN -> MX25L25635F; footprint Package_SON:WSON-8-1EP_6x5mm_P1.27mm_EP3.4x4mm -> Package_SON:WSON-8-1EP_8x6mm_P1.27mm_EP3.4x4.3mm
- moved U3 54.7 mm to (62.5, 82.6)
- moved U2 50.9 mm to (77.6, 78.7)
- renumbered C13 to C18, C14 to C19, C15 to C20, C16 to C21, C17 to C22, R2 to R1, R1 to R2, R6 to R3, R7 to R4, R3 to R5, R5 to R6, R4 to R7
Connections:
- net FMC_D0 renamed /MCU/FMC_D0
- U1 pad 111: /MCU/SDMMC1_D2 -> unconnected-(U1-PC10-Pad111)
- U1 pad 112: /MCU/SDMMC1_D3 -> unconnected-(U1-PC11-Pad112)
- U1 pad 113: /MCU/SDMMC1_CK -> unconnected-(U1-PC12-Pad113)
- U1 pad 116: /MCU/SDMMC1_CMD -> unconnected-(U1-PD2-Pad116)
- U1 pad 35: /MCU/ETH_REF_CLK -> /Ethernet/ETH_REF_CLK
- U1 pad 43: /MCU/ETH_RX_EN -> /Ethernet/ETH_RX_EN
- U1 pad 44: /MCU/ETH_RXD0 -> /Ethernet/ETH_RXD0
- U1 pad 45: /MCU/ETH_RXD1 -> /Ethernet/ETH_RXD1
- U1 pad 70: /MCU/ETH_TX_EN -> /Ethernet/ETH_TX_EN
- U1 pad 73: /MCU/ETH_TXD0 -> /Ethernet/ETH_TXD0
- U1 pad 74: /MCU/ETH_TXD1 -> /Ethernet/ETH_TXD1
- U1 pad 98: /MCU/SDMMC1_D0 -> unconnected-(U1-PC8-Pad98)
- U1 pad 99: /MCU/SDMMC1_D1 -> unconnected-(U1-PC9-Pad99)
- U2 pad 1: /Memory/QSPI_BK1_NCS -> /MCU/QSPI_BK1_NCS
- U2 pad 2: /Memory/QSPI_BK1_IO1 -> /MCU/QSPI_BK1_IO1
- U2 pad 3: /Memory/QSPI_BK1_IO2 -> /MCU/QSPI_BK1_IO2
- U2 pad 5: /Memory/QSPI_BK1_IO0 -> /MCU/QSPI_BK1_IO0
- U2 pad 6: /Memory/QSPI_BK1_CLK -> /MCU/QSPI_BK1_CLK
- U2 pad 7: /Memory/QSPI_BK1_IO3 -> /MCU/QSPI_BK1_IO3
- U2 pad 9: GND -> (no net)
- U3 pad 10: /Memory/FMC_D5 -> /MCU/FMC_D5
- U3 pad 11: /Memory/FMC_D6 -> /MCU/FMC_D6
- U3 pad 13: /Memory/FMC_D7 -> /MCU/FMC_D7
- U3 pad 15: /Memory/FMC_NBL0 -> /MCU/FMC_NBL0
- U3 pad 16: /Memory/FMC_SDNWE -> /MCU/FMC_SDNWE
- U3 pad 17: /Memory/FMC_SDNCAS -> /MCU/FMC_SDNCAS
- U3 pad 18: /Memory/FMC_SDNRAS -> /MCU/FMC_SDNRAS
- U3 pad 19: /Memory/FMC_SDNE0 -> /MCU/FMC_SDNE0
- U3 pad 20: /Memory/FMC_BA0 -> /MCU/FMC_BA0
- U3 pad 21: /Memory/FMC_BA1 -> /MCU/FMC_BA1
- U3 pad 22: /Memory/FMC_A10 -> /MCU/FMC_A10
- U3 pad 23: /Memory/FMC_A0 -> /MCU/FMC_A0
- U3 pad 24: /Memory/FMC_A1 -> /MCU/FMC_A1
- U3 pad 25: /Memory/FMC_A2 -> /MCU/FMC_A2
- U3 pad 26: /Memory/FMC_A3 -> /MCU/FMC_A3
- U3 pad 29: /Memory/FMC_A4 -> /MCU/FMC_A4
- U3 pad 30: /Memory/FMC_A5 -> /MCU/FMC_A5
- U3 pad 31: /Memory/FMC_A6 -> /MCU/FMC_A6
- U3 pad 32: /Memory/FMC_A7 -> /MCU/FMC_A7
- U3 pad 33: /Memory/FMC_A8 -> /MCU/FMC_A8
- U3 pad 34: /Memory/FMC_A9 -> /MCU/FMC_A9
- U3 pad 35: /Memory/FMC_A11 -> /MCU/FMC_A11
- U3 pad 36: /Memory/FMC_A12 -> /MCU/FMC_A12
- U3 pad 37: /Memory/FMC_SDCKE0 -> /MCU/FMC_SDCKE0
- U3 pad 38: /Memory/FMC_SDCLK -> /MCU/FMC_SDCLK
- U3 pad 39: /Memory/FMC_NBL1 -> /MCU/FMC_NBL1
- U3 pad 4: /Memory/FMC_D1 -> /MCU/FMC_D1
- U3 pad 42: /Memory/FMC_D8 -> /MCU/FMC_D8
- U3 pad 44: /Memory/FMC_D9 -> /MCU/FMC_D9
- U3 pad 45: /Memory/FMC_D10 -> /MCU/FMC_D10
- U3 pad 47: /Memory/FMC_D11 -> /MCU/FMC_D11
- U3 pad 48: /Memory/FMC_D12 -> /MCU/FMC_D12
- U3 pad 5: /Memory/FMC_D2 -> /MCU/FMC_D2
- U3 pad 50: /Memory/FMC_D13 -> /MCU/FMC_D13
- U3 pad 51: /Memory/FMC_D14 -> /MCU/FMC_D14
- U3 pad 53: /Memory/FMC_D15 -> /MCU/FMC_D15
- U3 pad 7: /Memory/FMC_D3 -> /MCU/FMC_D3
- U3 pad 8: /Memory/FMC_D4 -> /MCU/FMC_D4

Commit message: schematic capture
Parts:
- moved U4 28.5 mm to (124.0, 82.0)
- moved U2 2.33 mm to (76.0, 77.0), turned to 90 degrees
- moved U1 0.87 mm to (95.0, 82.0)
- moved U3 0.81 mm to (63.0, 82.0)
Connections:
- U1 pad 123: /MCU/ETH_SPI1_MOSI -> /Ethernet/ETH_SPI_MOSI
- U1 pad 19: unconnected-(U1-PF7-Pad19) -> /MCU/QSPI_BK1_IO2
- U1 pad 40: /MCU/ETH_SPI1_NSS -> /Ethernet/ETH_SPI_NSS
- U1 pad 41: /MCU/ETH_SPI1_SCK -> /Ethernet/ETH_SPI_SCK
- U1 pad 42: /MCU/ETH_SPI1_MISO -> /Ethernet/ETH_SPI_MISO
Routing:
- net /MCU/FMC_BA1: track 0.00 -> 73.1 mm, vias 0 -> 2
- net /MCU/FMC_BA0: track 0.00 -> 72.6 mm, vias 0 -> 2
- net /MCU/FMC_D1: track 0.00 -> 56.5 mm, vias 0 -> 2
- net /MCU/FMC_D0: track 0.00 -> 56.4 mm, vias 0 -> 2
- net /MCU/FMC_D14: track 0.00 -> 54.2 mm, vias 0 -> 2
- net /MCU/FMC_D4: track 0.00 -> 54.2 mm, vias 0 -> 2
- net /MCU/FMC_D5: track 0.00 -> 54.2 mm, vias 0 -> 2
- net /MCU/FMC_D6: track 0.00 -> 54.0 mm, vias 0 -> 2
- net /Ethernet/ETH_REF_CLK: track 0.00 -> 53.3 mm, vias 0 -> 2
- net /MCU/FMC_D7: track 0.00 -> 52.8 mm, vias 0 -> 2
- net /MCU/FMC_D2: track 0.00 -> 50.0 mm, vias 0 -> 2
- net /MCU/FMC_D3: track 0.00 -> 49.3 mm, vias 0 -> 2
- net /MCU/FMC_A3: track 0.00 -> 49.1 mm, vias 0 -> 2
- net /MCU/FMC_SDNCAS: track 0.00 -> 47.8 mm, vias 0 -> 2
- net /MCU/FMC_D12: track 0.00 -> 47.6 mm, vias 0 -> 2
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Other:
- copper layers 2 -> 4

Commit message: schematic capture
Parts:
- added C16: 10p, Capacitor_SMD:C_0603_1608Metric, F.Cu at (91.6, 102.2)
- added C17: 10p, Capacitor_SMD:C_0603_1608Metric, F.Cu at (95.3, 102.2)
- added C23: 0.1u, Capacitor_SMD:C_0603_1608Metric, F.Cu at (86.5, 95.2)
- added C24: 0.1u, Capacitor_SMD:C_0603_1608Metric, F.Cu at (101.2, 93.8)
- added C25: 0.1u, Capacitor_SMD:C_0603_1608Metric, F.Cu at (101.2, 88.3)
- added C26: 0.1u, Capacitor_SMD:C_0603_1608Metric, F.Cu at (91.2, 83.5)
- added C27: 0.1u, Capacitor_SMD:C_0603_1608Metric, F.Cu at (86.5, 92.3)
- added C28: 10p, Capacitor_SMD:C_0603_1608Metric, F.Cu at (96.2, 83.5)
- added C29: 0.1u, Capacitor_SMD:C_0603_1608Metric, F.Cu at (89.7, 72.8)
- added D4: LED_Dual_AAKK, Footpint:LED_Kingbright_KPBD-3224, F.Cu at (85.2, 64.7)
- added D5: BAT60A, Diode_SMD:D_SOD-323, F.Cu at (86.5, 86.2)
- added D6: BAT60A, Diode_SMD:D_SOD-323, F.Cu at (84.4, 115.5)
- added J3: USB_B_Micro, Footpint:USB_Micro-B_CUZD188-CB1Z, F.Cu at (80.0, 80.0)
- added J4: Conn_01x04_Pin, Connector_PinHeader_2.54mm:PinHeader_1x04_P2.54mm_Vertical, F.Cu at (83.1, 110.5)
- added J5: Conn_01x02_Pin, Connector_PinHeader_2.54mm:PinHeader_1x02_P2.54mm_Vertical, F.Cu at (103.4, 110.5)
- added J6: Conn_01x06_Pin, Connector_PinHeader_2.54mm:PinHeader_1x06_P2.54mm_Vertical, F.Cu at (88.4, 119.2)
- added J7: Conn_01x02_Pin, Connector_PinHeader_2.54mm:PinHeader_1x02_P2.54mm_Vertical, F.Cu at (81.3, 91.0)
- added JP1: SolderJumper_3_Open, Jumper:SolderJumper-3_P2.0mm_Open_TrianglePad1.0x1.5mm_NumberLabels, F.Cu at (66.7, 93.7)
- added JP10: Jumper_2_Bridged, Jumper:SolderJumper-2_P1.3mm_Open_TrianglePad1.0x1.5mm, B.Cu at (62.6, 103.0)
- added JP11: Jumper_2_Bridged, Jumper:SolderJumper-2_P1.3mm_Open_TrianglePad1.0x1.5mm, B.Cu at (62.6, 106.5)
- added JP12: Jumper_2_Bridged, Jumper:SolderJumper-2_P1.3mm_Open_TrianglePad1.0x1.5mm, B.Cu at (62.6, 110.0)
- added JP2: Jumper_2_Bridged, Jumper:SolderJumper-2_P1.3mm_Open_TrianglePad1.0x1.5mm, B.Cu at (71.3, 103.0)
- added JP3: Jumper_2_Open, Jumper:SolderJumper-2_P1.3mm_Open_TrianglePad1.0x1.5mm, B.Cu at (71.3, 106.5)
- added JP4: Jumper_2_Bridged, Jumper:SolderJumper-2_P1.3mm_Open_TrianglePad1.0x1.5mm, B.Cu at (71.3, 110.0)
- added JP5: Jumper_2_Bridged, Jumper:SolderJumper-2_P1.3mm_Open_TrianglePad1.0x1.5mm, B.Cu at (71.3, 113.6)
- added JP6: Jumper_2_Bridged, Jumper:SolderJumper-2_P1.3mm_Open_TrianglePad1.0x1.5mm, B.Cu at (67.0, 103.0)
- added JP7: Jumper_2_Open, Jumper:SolderJumper-2_P1.3mm_Open_TrianglePad1.0x1.5mm, B.Cu at (67.0, 106.5)
- added JP8: Jumper_2_Open, Jumper:SolderJumper-2_P1.3mm_Open_TrianglePad1.0x1.5mm, B.Cu at (67.0, 110.0)
- added JP9: Jumper_2_Open, Jumper:SolderJumper-2_P1.3mm_Open_TrianglePad1.0x1.5mm, B.Cu at (67.0, 113.6)
- added R10: 100K, Resistor_SMD:R_0603_1608Metric, F.Cu at (86.2, 83.6)
- added R11: 1.5K, Resistor_SMD:R_0603_1608Metric, F.Cu at (86.2, 82.1)
- added R12: 10K, Resistor_SMD:R_0603_1608Metric, F.Cu at (89.7, 68.3)
- added R13: 36K, Resistor_SMD:R_0603_1608Metric, F.Cu at (89.7, 69.8)
- added R14: 100, Resistor_SMD:R_0603_1608Metric, F.Cu at (89.7, 71.3)
- added R15: 100, Resistor_SMD:R_0603_1608Metric, F.Cu at (89.7, 64.0)
- added R16: 100, Resistor_SMD:R_0603_1608Metric, F.Cu at (89.7, 65.5)
- added R17: 10K, Resistor_SMD:R_0603_1608Metric, F.Cu at (86.5, 96.7)
- added R18: 10K, Resistor_SMD:R_0603_1608Metric, F.Cu at (86.5, 98.2)
- added R19: 10K, Resistor_SMD:R_0603_1608Metric, F.Cu at (86.5, 93.8)
- added R20: 4K7, Resistor_SMD:R_0603_1608Metric, F.Cu at (98.9, 97.5)
- added R21: 4K7, Resistor_SMD:R_0603_1608Metric, F.Cu at (98.9, 98.9)
- added R22: 100, Resistor_SMD:R_0603_1608Metric, F.Cu at (101.2, 86.8)
- added R23: 4K7, Resistor_SMD:R_0603_1608Metric, F.Cu at (86.5, 87.8)
- added R24: 4K7, Resistor_SMD:R_0603_1608Metric, F.Cu at (86.5, 89.3)
- added R25: 100K, Resistor_SMD:R_0603_1608Metric, F.Cu at (66.3, 88.5)
- added R26: 100K, Resistor_SMD:R_0603_1608Metric, F.Cu at (66.3, 91.0)
- added R27: 22, Resistor_SMD:R_0603_1608Metric, F.Cu at (90.9, 115.5)
- added R28: 22, Resistor_SMD:R_0603_1608Metric, F.Cu at (96.0, 115.5)
- added R29: 22, Resistor_SMD:R_0603_1608Metric, F.Cu at (98.6, 115.5)
- added R30: 22, Resistor_SMD:R_0603_1608Metric, F.Cu at (101.1, 115.5)
- added R31: 10K, Resistor_SMD:R_0603_1608Metric, F.Cu at (88.4, 115.5)
- added R32: 100, Resistor_SMD:R_0603_1608Metric, F.Cu at (86.2, 115.5)
- added R33: 100, Resistor_SMD:R_0603_1608Metric, F.Cu at (94.8, 83.5)
- added U7: USBLC6-2SC6, Package_TO_SOT_SMD:SOT-23-6, F.Cu at (86.2, 79.7)
- added Y2: 8 MHz, Crystal:Crystal_SMD_5032-2Pin_5.0x3.2mm, F.Cu at (93.5, 98.8)
- C18, C19, C20, C21, C22: footprint Resistor_SMD:R_0603_1608Metric -> Capacitor_SMD:C_0603_1608Metric
- moved R1 82.0 mm to (231.1, 68.6)
- moved R2 82.0 mm to (231.1, 66.6)
- moved R3 82.0 mm to (234.0, 70.6)
- moved R4 82.0 mm to (236.9, 66.6)
- moved R5 82.0 mm to (231.1, 70.6)
- moved R6 82.0 mm to (234.0, 68.6)
- moved R7 82.0 mm to (234.0, 66.6)
- moved R8 82.0 mm to (236.9, 68.6)
- moved R9 82.0 mm to (236.9, 70.6)
- moved U1 82.0 mm to (177.0, 82.0)
- moved U2 82.0 mm to (158.0, 77.0)
- moved U3 82.0 mm to (145.0, 82.0)
- moved U4 82.0 mm to (206.0, 82.0)
- moved U5 51.9 mm to (94.0, 91.0), turned to 90 degrees
- moved D1 48.0 mm to (96.4, 78.7), turned to -90 degrees
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Connections:
- C21 pad 1: Net-(U6-VOUT) -> +3V3
- C22 pad 1: Net-(U6-VOUT) -> +3V3
- D1 pad 2: unconnected-(D1-A-Pad2) -> +5V0
- D2 pad 2: unconnected-(D2-A-Pad2) -> +5V0
- D3 pad 2: unconnected-(D3-A-Pad2) -> +5V0
- U1 pad 105: unconnected-(U1-PA13-Pad105) -> /MCU/TMS
- U1 pad 109: unconnected-(U1-PA14-Pad109) -> /MCU/TCK
- U1 pad 133: unconnected-(U1-PB3-Pad133) -> /MCU/SWO
- U1 pad 25: unconnected-(U1-NRST-Pad25) -> /MCU/NRST
- U5 pad 1: unconnected-(U5-VBAT-Pad1) -> +3V3
- U5 pad 2: /ST-Link/BI0 -> Net-(U5-PC13)
- U5 pad 24: unconnected-(U5-VDD-Pad24) -> +3V3
- U5 pad 29: /ST-Link/MCO -> /MCU/MCO
- U5 pad 3: /ST-Link/BI1 -> Net-(U5-PC14)
- U5 pad 36: unconnected-(U5-VDD-Pad36) -> +3V3
- U5 pad 44: unconnected-(U5-BOOT0-Pad44) -> Net-(JP1-C)
- U5 pad 48: unconnected-(U5-VDD-Pad48) -> +3V3
- U5 pad 7: /ST-Link/STM_RST -> Net-(U5-NRST)
- U5 pad 9: unconnected-(U5-VDDA-Pad9) -> +3V3
- U6 pad 5: Net-(U6-VOUT) -> +3V3
Routing:
- net Net-(U5-PD0): track 0.00 -> 6.94 mm
- net Net-(U5-PD1): track 0.00 -> 6.91 mm
- net Net-(D4-A1): track 0.00 -> 5.87 mm
- net /ST-Link/STLINK_USB_DM: track 0.00 -> 5.76 mm
- net /ST-Link/STLINK_USB_DP: track 0.00 -> 5.74 mm
- net Net-(J3-ID): track 0.00 -> 5.60 mm
- net /ST-Link/AIN1: track 0.00 -> 5.48 mm
- net Net-(Q1-B): track 0.00 -> 4.96 mm
- net /ST-Link/T_SWDIO_IN: track 0.00 -> 3.42 mm
- net Net-(D4-K2): track 0.00 -> 2.06 mm
- net GND: track 0.00 -> 1.11 mm, vias 0 -> 1

Commit message: schematic capture
Parts:
- added C1: 0.1u, Capacitor_SMD:C_0603_1608Metric, F.Cu at (51.9, 61.9)
- added C10: 0.1u, Capacitor_SMD:C_0603_1608Metric, F.Cu at (34.6, 8.92)
- added C11: 0.1u, Capacitor_SMD:C_0603_1608Metric, F.Cu at (34.6, 11.4)
- added C12: 0.1u, Capacitor_SMD:C_0603_1608Metric, F.Cu at (34.6, 13.9)
- added C13: 0.1u, Capacitor_SMD:C_0603_1608Metric, F.Cu at (38.6, 6.41)
- added C14: 0.1u, Capacitor_SMD:C_0603_1608Metric, F.Cu at (38.6, 8.92)
- added C15: 0.1u, Capacitor_SMD:C_0603_1608Metric, F.Cu at (38.6, 11.4)
- added C2: 1u, Capacitor_SMD:C_0603_1608Metric, F.Cu at (51.9, 64.4)
- added C3: 0.1u, Capacitor_SMD:C_0603_1608Metric, F.Cu at (51.9, 66.9)
- added C30: 1u, Capacitor_SMD:C_0603_1608Metric, F.Cu at (30.6, 18.4)
- added C31: 0.1u, Capacitor_SMD:C_0603_1608Metric, F.Cu at (30.6, 21.0)
- added C32: 1u, Capacitor_SMD:C_0603_1608Metric, F.Cu at (30.6, 23.5)
- added C33: 0.1u, Capacitor_SMD:C_0603_1608Metric, F.Cu at (30.6, 26.0)
- added C34: 0.1u, Capacitor_SMD:C_0603_1608Metric, F.Cu at (30.6, 28.5)
- added C35: 4.7u, Capacitor_Tantalum_SMD:CP_EIA-6032-28_Kemet-C, F.Cu at (41.3, 36.5)
- added C37: 4.7u, Capacitor_Tantalum_SMD:CP_EIA-6032-28_Kemet-C, F.Cu at (42.1, 59.0)
- added C4: 0.1u, Capacitor_SMD:C_0603_1608Metric, F.Cu at (51.9, 69.4)
- added C5: 18p, Capacitor_SMD:C_0603_1608Metric, F.Cu at (30.6, 6.41)
- added C6: 18p, Capacitor_SMD:C_0603_1608Metric, F.Cu at (30.6, 8.92)
- added C7: 0.1u, Capacitor_SMD:C_0603_1608Metric, F.Cu at (30.6, 11.4)
- added C8: 0.1u, Capacitor_SMD:C_0603_1608Metric, F.Cu at (30.6, 13.9)
- added C9: 0.1u, Capacitor_SMD:C_0603_1608Metric, F.Cu at (34.6, 6.41)
- added D10: LED_Small, LED_SMD:LED_0603_1608Metric, F.Cu at (39.8, 52.8)
- added D11: LED_Small, LED_SMD:LED_0603_1608Metric, F.Cu at (39.8, 55.4)
- added D7: LED_Small, LED_SMD:LED_0603_1608Metric, F.Cu at (46.2, 18.5)
- added D8: LED_Small, LED_SMD:LED_0603_1608Metric, F.Cu at (46.2, 21.1)
- added D9: ESDA6V1BC6, Package_TO_SOT_SMD:SOT-23-6, F.Cu at (35.2, 53.7)
- added FB1: FerriteBead_Small, Capacitor_SMD:C_0603_1608Metric, F.Cu at (38.6, 13.9)
- added J1: KLS12-TL051, Footpint:KLS12-TL051, F.Cu at (224.9, 104.2)
- added J10: USB_B_Micro, Footpint:USB_Micro-B_CUZD188-CB1Z, F.Cu at (42.4, 44.7)
- added J11: Conn_01x02_Pin, Connector_PinHeader_2.54mm:PinHeader_1x02_P2.54mm_Vertical, F.Cu at (60.9, 43.2)
- added J12: Conn_02x08_Odd_Even, Connector_PinHeader_2.54mm:PinHeader_2x08_P2.54mm_Vertical, F.Cu at (125.6, 118.3)
- added J13: Conn_02x10_Odd_Even, Connector_PinHeader_2.54mm:PinHeader_2x10_P2.54mm_Vertical, F.Cu at (120.3, 68.8)
- added J14: Conn_02x15_Odd_Even, Connector_PinHeader_2.54mm:PinHeader_2x15_P2.54mm_Vertical, F.Cu at (157.8, 118.0)
- added J15: Conn_02x17_Odd_Even, Connector_PinHeader_2.54mm:PinHeader_2x16_P2.54mm_Vertical, F.Cu at (152.3, 68.7)
- added J16: Conn_02x37_Odd_Even, Connector_PinHeader_2.54mm:PinHeader_2x37_P2.54mm_Vertical, F.Cu at (115.5, 130.3)
- added J17: Conn_02x37_Odd_Even, Connector_PinHeader_2.54mm:PinHeader_2x37_P2.54mm_Vertical, F.Cu at (116.5, 53.3)
- added J18: Conn_01x02_Pin, Connector_PinHeader_2.54mm:PinHeader_1x02_P2.54mm_Vertical, F.Cu at (44.0, 29.2)
- added J19: Conn_01x02_Pin, Connector_PinHeader_2.54mm:PinHeader_1x02_P2.54mm_Vertical, F.Cu at (48.6, 29.2)
- added J2: KLS12-TL051, Footpint:KLS12-TL051, F.Cu at (224.7, 85.1)
- added J8: Conn_02x03_Odd_Even, Connector_PinHeader_2.54mm:PinHeader_2x03_P2.54mm_Vertical, F.Cu at (39.3, 19.5)
- added J9: Conn_01x02_Pin, Connector_PinHeader_2.54mm:PinHeader_1x02_P2.54mm_Vertical, F.Cu at (39.3, 29.2)
- added JP13: Jumper_2_Bridged, Jumper:SolderJumper-2_P1.3mm_Open_TrianglePad1.0x1.5mm, F.Cu at (52.1, 42.6)
- added JP14: Jumper_2_Bridged, Jumper:SolderJumper-2_P1.3mm_Open_TrianglePad1.0x1.5mm, F.Cu at (34.8, 19.0)
- added JP15: Jumper_2_Bridged, Jumper:SolderJumper-2_P1.3mm_Open_TrianglePad1.0x1.5mm, F.Cu at (34.8, 22.5)
- added JP16: Jumper_2_Open, Jumper:SolderJumper-2_P1.3mm_Open_TrianglePad1.0x1.5mm, F.Cu at (34.8, 26.1)
- added JP17: Jumper_2_Bridged, Jumper:SolderJumper-2_P1.3mm_Open_TrianglePad1.0x1.5mm, F.Cu at (34.8, 42.6)
- added JP18: Jumper_2_Bridged, Jumper:SolderJumper-2_P1.3mm_Open_TrianglePad1.0x1.5mm, F.Cu at (52.1, 46.2)
- added JP19: Jumper_2_Bridged, Jumper:SolderJumper-2_P1.3mm_Open_TrianglePad1.0x1.5mm, F.Cu at (34.8, 46.2)
- added JP20: Jumper_2_Bridged, Jumper:SolderJumper-2_P1.3mm_Open_TrianglePad1.0x1.5mm, F.Cu at (34.8, 49.7)
- added JP21: Jumper_2_Bridged, Jumper:SolderJumper-2_P1.3mm_Open_TrianglePad1.0x1.5mm, F.Cu at (52.1, 49.7)
- added JP22: Jumper_2_Bridged, Jumper:SolderJumper-2_P1.3mm_Open_TrianglePad1.0x1.5mm, F.Cu at (52.1, 53.3)
- added JP23: Jumper_2_Bridged, Jumper:SolderJumper-2_P1.3mm_Open_TrianglePad1.0x1.5mm, F.Cu at (24.4, 57.3)
- added JP24: Jumper_2_Open, Jumper:SolderJumper-2_P1.3mm_Open_TrianglePad1.0x1.5mm, F.Cu at (24.4, 60.9)
- added JP25: Jumper_2_Open, Jumper:SolderJumper-2_P1.3mm_Open_TrianglePad1.0x1.5mm, F.Cu at (24.4, 64.4)
- added JP26: Jumper_2_Open, Jumper:SolderJumper-2_P1.3mm_Open_TrianglePad1.0x1.5mm, F.Cu at (52.1, 56.8)
- added JP27: Jumper_2_Bridged, Jumper:SolderJumper-2_P1.3mm_Open_TrianglePad1.0x1.5mm, F.Cu at (56.4, 42.6)
- added JP28: Jumper_2_Bridged, Jumper:SolderJumper-2_P1.3mm_Open_TrianglePad1.0x1.5mm, F.Cu at (56.4, 46.2)
- added JP29: Jumper_2_Bridged, Jumper:SolderJumper-2_P1.3mm_Open_TrianglePad1.0x1.5mm, F.Cu at (24.4, 68.0)
- added JP30: Jumper_2_Bridged, Jumper:SolderJumper-2_P1.3mm_Open_TrianglePad1.0x1.5mm, F.Cu at (56.4, 49.7)
- added JP31: Jumper_2_Bridged, Jumper:SolderJumper-2_P1.3mm_Open_TrianglePad1.0x1.5mm, F.Cu at (56.4, 53.3)
- added JP32: Jumper_2_Open, Jumper:SolderJumper-2_P1.3mm_Open_TrianglePad1.0x1.5mm, F.Cu at (24.4, 71.5)
- added JP33: Jumper_2_Open, Jumper:SolderJumper-2_P1.3mm_Open_TrianglePad1.0x1.5mm, F.Cu at (56.4, 56.8)
- added Q2: BC848, Package_TO_SOT_SMD:SOT-23, F.Cu at (44.3, 53.7)
- added R34: 1K, Resistor_SMD:R_0603_1608Metric, F.Cu at (30.6, 31.0)
- added R35: 1K, Resistor_SMD:R_0603_1608Metric, F.Cu at (30.6, 33.5)
- added R36: 10K, Resistor_SMD:R_0603_1608Metric, F.Cu at (30.6, 36.0)
- added R37: 10K, Resistor_SMD:R_0603_1608Metric, F.Cu at (30.6, 42.1)
- added R38: 10K, Resistor_SMD:R_0603_1608Metric, F.Cu at (60.6, 49.3)
- added R44: 620, Resistor_SMD:R_0603_1608Metric, F.Cu at (30.6, 44.6)
- added R45: 47K, Resistor_SMD:R_0603_1608Metric, F.Cu at (30.6, 47.1)
- added R46: 430K, Resistor_SMD:R_0603_1608Metric, F.Cu at (30.6, 49.6)
- added R47: 620K, Resistor_SMD:R_0603_1608Metric, F.Cu at (30.6, 52.1)
- added R48: 47K, Resistor_SMD:R_0603_1608Metric, F.Cu at (30.6, 54.6)
- added R49: 330, Resistor_SMD:R_0603_1608Metric, F.Cu at (30.6, 57.2)
- added R50: 47K, Resistor_SMD:R_0603_1608Metric, F.Cu at (30.6, 59.7)
- added U10: TPS2051B, Package_TO_SOT_SMD:SOT-23-5, F.Cu at (48.1, 36.3)
- added U12: TPS2051B, Package_TO_SOT_SMD:SOT-23-5, F.Cu at (35.2, 58.2)
- added U8: USBLC6-4SC6, Package_TO_SOT_SMD:SOT-23-6, F.Cu at (43.2, 7.38)
- added U9: USBLC6-4SC6, Package_TO_SOT_SMD:SOT-23-6, F.Cu at (43.2, 11.8)
- added Y1: 25Mhz, Crystal:Crystal_SMD_3225-4Pin_3.2x2.5mm, F.Cu at (48.4, 7.38)
- R1, R2, R3, R4, R5, R6, R7, R8, R9: footprint Resistor_SMD:R_0402_1005Metric -> Resistor_SMD:R_0603_1608Metric
- moved U1 19.7 mm to (159.1, 90.3)
- moved U2 19.7 mm to (140.1, 85.3)
- moved U3 19.7 mm to (127.1, 90.3)
- moved U4 19.7 mm to (188.1, 90.3)
- moved R1 15.8 mm to (244.2, 59.8)
- moved R2 15.8 mm to (244.2, 57.8)
- moved R4 15.8 mm to (250.0, 57.8)
- moved R6 15.8 mm to (247.1, 59.8)
- moved R7 15.8 mm to (247.1, 57.8)
- moved R8 15.8 mm to (250.0, 59.8)
- moved R3 15.8 mm to (247.1, 61.8)
- moved R5 15.8 mm to (244.2, 61.8)
- moved R9 15.8 mm to (250.0, 61.8)
Connections:
- net /MCU/NRST renamed /Connectors/NRST
- net /ST-Link/STLNK_RX renamed /MCU/USART3_TX
- net /ST-Link/STLNK_TX renamed /MCU/USART3_RX
- U1 pad 100: unconnected-(U1-PA8-Pad100) -> /Connectors/PA8
- U1 pad 101: unconnected-(U1-PA9-Pad101) -> /Connectors/PA9
- U1 pad 102: unconnected-(U1-PA10-Pad102) -> /Connectors/PA10
- U1 pad 103: unconnected-(U1-PA11-Pad103) -> /Connectors/PA11
- U1 pad 104: unconnected-(U1-PA12-Pad104) -> /Connectors/PA12
- U1 pad 105: /MCU/TMS -> /Connectors/PA13
- U1 pad 109: /MCU/TCK -> /Connectors/PA14
- U1 pad 110: unconnected-(U1-PA15-Pad110) -> /Connectors/PA15
- U1 pad 111: unconnected-(U1-PC10-Pad111) -> /Connectors/PC10
- U1 pad 112: unconnected-(U1-PC11-Pad112) -> /Connectors/PC11
- U1 pad 113: unconnected-(U1-PC12-Pad113) -> /Connectors/PC12
- U1 pad 116: unconnected-(U1-PD2-Pad116) -> /Connectors/PD2
- U1 pad 117: unconnected-(U1-PD3-Pad117) -> /Connectors/PD3
- U1 pad 118: unconnected-(U1-PD4-Pad118) -> /Connectors/PD4
- U1 pad 119: unconnected-(U1-PD5-Pad119) -> /Connectors/PD5
- U1 pad 122: unconnected-(U1-PD6-Pad122) -> /Connectors/PD6
- U1 pad 124: unconnected-(U1-PG9-Pad124) -> /Connectors/PG9
- U1 pad 125: unconnected-(U1-PG10-Pad125) -> /Connectors/PG10
- U1 pad 126: unconnected-(U1-PG11-Pad126) -> /Connectors/PG11
- U1 pad 127: unconnected-(U1-PG12-Pad127) -> /Connectors/PG12
- U1 pad 128: unconnected-(U1-PG13-Pad128) -> /Connectors/PG13
- U1 pad 129: unconnected-(U1-PG14-Pad129) -> /Connectors/PG14
- U1 pad 133: /MCU/SWO -> /Connectors/PB3
- U1 pad 134: unconnected-(U1-PB4-Pad134) -> /Connectors/PB4
- U1 pad 135: unconnected-(U1-PB5-Pad135) -> /Connectors/PB5
- U1 pad 136: unconnected-(U1-PB6-Pad136) -> /Connectors/PB6
- U1 pad 137: unconnected-(U1-PB7-Pad137) -> /Connectors/PB7
- U1 pad 139: unconnected-(U1-PB8-Pad139) -> /Connectors/PB8
- U1 pad 140: unconnected-(U1-PB9-Pad140) -> /Connectors/PB9
- U1 pad 2: unconnected-(U1-PE3-Pad2) -> /Connectors/PE3
- U1 pad 27: unconnected-(U1-PC1-Pad27) -> /Connectors/PC1
- U1 pad 3: unconnected-(U1-PE4-Pad3) -> /Connectors/PE4
- U1 pad 34: unconnected-(U1-PA0-Pad34) -> /Connectors/PA0
- U1 pad 36: unconnected-(U1-PA2-Pad36) -> /Connectors/PA2
- U1 pad 37: unconnected-(U1-PA3-Pad37) -> /Connectors/PA3
- U1 pad 4: unconnected-(U1-PE5-Pad4) -> /Connectors/PE5
- U1 pad 46: unconnected-(U1-PB0-Pad46) -> /Connectors/PB0
- U1 pad 47: unconnected-(U1-PB1-Pad47) -> /Connectors/PB1
- U1 pad 48: unconnected-(U1-PB2-Pad48) -> /Connectors/PB2
- U1 pad 5: unconnected-(U1-PE6-Pad5) -> /Connectors/PE6
- U1 pad 7: unconnected-(U1-PC13-Pad7) -> /Connectors/PC13
- U1 pad 75: unconnected-(U1-PB14-Pad75) -> /Connectors/PB14
- U1 pad 76: unconnected-(U1-PB15-Pad76) -> /Connectors/PB15
- U1 pad 8: unconnected-(U1-PC14-Pad8) -> /Connectors/PC14
- U1 pad 80: unconnected-(U1-PD11-Pad80) -> /Connectors/PD11
- U1 pad 81: unconnected-(U1-PD12-Pad81) -> /Connectors/PD12
- U1 pad 82: unconnected-(U1-PD13-Pad82) -> /Connectors/PD13
- U1 pad 88: unconnected-(U1-PG3-Pad88) -> /Connectors/PG3
- U1 pad 9: unconnected-(U1-PC15-Pad9) -> /Connectors/PC15
- U1 pad 91: unconnected-(U1-PG6-Pad91) -> /Connectors/PG6
- U1 pad 92: unconnected-(U1-PG7-Pad92) -> /Connectors/PG7
- U1 pad 96: unconnected-(U1-PC6-Pad96) -> /Connectors/PC6
- U1 pad 97: unconnected-(U1-PC7-Pad97) -> /Connectors/PC7
- U1 pad 98: unconnected-(U1-PC8-Pad98) -> /Connectors/PC8
- U1 pad 99: unconnected-(U1-PC9-Pad99) -> /Connectors/PC9

Commit message: schematic capture
Parts:
- moved J16 70.9 mm to (129.5, 60.9)
- moved J17 69.8 mm to (129.5, 121.8)
- moved J12 14.7 mm to (139.7, 114.2)
- moved U1 10.9 mm to (170.0, 90.0)
- moved U2 10.9 mm to (151.0, 85.0)
- moved U3 10.9 mm to (138.0, 90.0)
- moved U4 10.9 mm to (199.0, 90.0)
- moved J13 10.2 mm to (130.5, 68.5)
- moved J14 6.08 mm to (162.5, 114.2)
- moved J15 5.13 mm to (157.5, 68.5)
