File: HARDWARE/meshium_duo.kicad_pcb (KiCad board)
At the start: 4 copper layers, 160 parts, among them J1 KLS12-TL051, J10 USB_B_Micro, J11 Conn_01x02_Pin, J12 Conn_02x08_Odd_Even, J13 Conn_02x10_Odd_Even, J14 Conn_02x15_Odd_Even, J15 Conn_02x17_Odd_Even, J16 Conn_02x37_Odd_Even, J17 Conn_02x37_Odd_Even, J18 Conn_01x02_Pin, J19 Conn_01x02_Pin, J2 KLS12-TL051, J3 USB_B_Micro, J4 Conn_01x04_Pin, J5 Conn_01x02_Pin, J6 Conn_01x06_Pin, J7 Conn_01x02_Pin, J8 Conn_02x03_Odd_Even, J9 Conn_01x02_Pin, Q1 BC848, Q2 BC848, U1 STM32F767ZITx, U10 TPS2051B, U12 TPS2051B, U2 MX25L25635F, U3 MT48LC16M16A2P, U4 KSZ8463FRL, U5 STM32F103CBTx, U6 LD3985M33R_SOT23, U7 USBLC6-2SC6, U8 USBLC6-4SC6, U9 USBLC6-4SC6, Y1 25Mhz, Y2 8 MHz

Commit message: schematic capture
Parts:
- removed the C32 at (30.6, 23.5)
- removed the C33 at (30.6, 26.0)
- removed the J18 at (44.0, 29.2)
- removed the J19 at (48.6, 29.2)
- added C10: 0.1u, Capacitor_SMD:C_0603_1608Metric, F.Cu at (77.4, 36.1)
- added C11: 0.1u, Capacitor_SMD:C_0603_1608Metric, F.Cu at (77.4, 38.6)
- added C12: 0.1u, Capacitor_SMD:C_0603_1608Metric, F.Cu at (77.4, 41.1)
- added C13: 0.1u, Capacitor_SMD:C_0603_1608Metric, F.Cu at (77.4, 43.6)
- added C14: 0.1u, Capacitor_SMD:C_0603_1608Metric, F.Cu at (77.4, 46.2)
- added C15: 0.1u, Capacitor_SMD:C_0603_1608Metric, F.Cu at (77.4, 48.7)
- added C16: 0.1u, Capacitor_SMD:C_0603_1608Metric, F.Cu at (81.4, 33.6)
- added C17: 0.1u, Capacitor_SMD:C_0603_1608Metric, F.Cu at (81.4, 36.1)
- added C18: 0.1u, Capacitor_SMD:C_0603_1608Metric, F.Cu at (81.4, 38.6)
- added C19: 0.1u, Capacitor_SMD:C_0603_1608Metric, F.Cu at (81.4, 41.1)
- added C2: 4.7u, Capacitor_SMD:C_0603_1608Metric, F.Cu at (146.0, 32.7)
- added C20: 0.1u, Capacitor_SMD:C_0603_1608Metric, F.Cu at (81.4, 43.6)
- added C21: 4.7u, Capacitor_SMD:C_0603_1608Metric, F.Cu at (81.4, 46.2)
- added C22: 2.2u, Capacitor_SMD:C_0805_2012Metric, F.Cu at (93.7, 41.7)
- added C23: 2.2u, Capacitor_SMD:C_0805_2012Metric, F.Cu at (93.7, 44.7)
- added C24: 0.1u, Capacitor_SMD:C_0603_1608Metric, F.Cu at (81.4, 48.7)
- added C25: 0.1u, Capacitor_SMD:C_0603_1608Metric, F.Cu at (85.4, 33.6)
- added C26: 0.1u, Capacitor_SMD:C_0603_1608Metric, F.Cu at (85.4, 36.1)
- added C27: 10p, Capacitor_SMD:C_0603_1608Metric, F.Cu at (85.4, 38.6)
- added C28: 10p, Capacitor_SMD:C_0603_1608Metric, F.Cu at (85.4, 41.1)
- added C29: 2p, Capacitor_SMD:C_0603_1608Metric, F.Cu at (85.4, 43.6)
- added C3: 0.1u, Capacitor_SMD:C_0603_1608Metric, F.Cu at (146.0, 31.2)
- added C30: 2p, Capacitor_SMD:C_0603_1608Metric, F.Cu at (85.4, 46.2)
- added C5: 22u, Capacitor_SMD:C_0805_2012Metric, F.Cu at (149.0, 27.2)
- added C8: 22u, Capacitor_SMD:C_0805_2012Metric, F.Cu at (134.9, 40.0)
- added C9: 0.1u, Capacitor_SMD:C_0603_1608Metric, F.Cu at (77.4, 33.6)
- added D3: LED_Small, LED_SMD:LED_0603_1608Metric, F.Cu at (94.8, 23.0)
- added D4: LED_Small, LED_SMD:LED_0603_1608Metric, F.Cu at (94.8, 25.6)
- added FB1: FerriteBead_Small, Capacitor_SMD:C_0603_1608Metric, F.Cu at (85.4, 48.7)
- added J13: Conn_01x02_Pin, Connector_PinHeader_2.54mm:PinHeader_1x02_P2.54mm_Vertical, F.Cu at (101.2, 42.5)
- added J16: Conn_01x02_Pin, Connector_PinHeader_2.54mm:PinHeader_1x02_P2.54mm_Vertical, F.Cu at (105.8, 42.5)
- added JP15: Jumper_2_Bridged, Jumper:SolderJumper-2_P1.3mm_Open_TrianglePad1.0x1.5mm, F.Cu at (77.6, 30.6)
- added JP16: Jumper_2_Bridged, Jumper:SolderJumper-2_P1.3mm_Open_TrianglePad1.0x1.5mm, F.Cu at (81.9, 23.5)
- added JP17: Jumper_2_Bridged, Jumper:SolderJumper-2_P1.3mm_Open_TrianglePad1.0x1.5mm, F.Cu at (81.9, 27.0)
- added JP19: Jumper_2_Bridged, Jumper:SolderJumper-2_P1.3mm_Open_TrianglePad1.0x1.5mm, F.Cu at (81.9, 30.6)
- added JP20: Jumper_2_Bridged, Jumper:SolderJumper-2_P1.3mm_Open_TrianglePad1.0x1.5mm, F.Cu at (86.3, 23.5)
- added JP21: Jumper_2_Bridged, Jumper:SolderJumper-2_P1.3mm_Open_TrianglePad1.0x1.5mm, F.Cu at (86.3, 27.0)
- added JP22: Jumper_2_Open, Jumper:SolderJumper-2_P1.3mm_Open_TrianglePad1.0x1.5mm, F.Cu at (86.3, 30.6)
- added JP23: Jumper_2_Open, Jumper:SolderJumper-2_P1.3mm_Open_TrianglePad1.0x1.5mm, F.Cu at (90.6, 23.5)
- added JP24: Jumper_2_Open, Jumper:SolderJumper-2_P1.3mm_Open_TrianglePad1.0x1.5mm, F.Cu at (90.6, 27.0)
- added JP25: Jumper_2_Open, Jumper:SolderJumper-2_P1.3mm_Open_TrianglePad1.0x1.5mm, F.Cu at (90.6, 30.6)
- added JP41: Jumper_2_Open, Jumper:SolderJumper-2_P1.3mm_Open_TrianglePad1.0x1.5mm, F.Cu at (110.3, 42.0)
- added JP42: Jumper_2_Open, Jumper:SolderJumper-2_P1.3mm_Open_TrianglePad1.0x1.5mm, F.Cu at (110.3, 45.5)
- added JP7: Jumper_2_Bridged, Jumper:SolderJumper-2_P1.3mm_Open_TrianglePad1.0x1.5mm, F.Cu at (77.6, 23.5)
- added JP8: Jumper_2_Bridged, Jumper:SolderJumper-2_P1.3mm_Open_TrianglePad1.0x1.5mm, F.Cu at (77.6, 27.0)
- added L1: SDR0604-2R2ML, Footpint:L_Bourns-SRN0604, F.Cu at (147.1, 21.1)
- added L2: SDR0604-2R2ML, Footpint:L_Bourns-SRN0604, F.Cu at (132.9, 34.2)
- added R10: 680, Resistor_SMD:R_0603_1608Metric, F.Cu at (89.4, 36.1)
- added R11: 1K, Resistor_SMD:R_0603_1608Metric, F.Cu at (89.4, 38.6)
- added R12: 1K, Resistor_SMD:R_0603_1608Metric, F.Cu at (89.4, 41.1)
- added R13: 220K, Resistor_SMD:R_0603_1608Metric, F.Cu at (89.4, 43.6)
- added R3: 19K, Resistor_SMD:R_0603_1608Metric, F.Cu at (149.9, 29.7)
- added R4: 100K, Resistor_SMD:R_0603_1608Metric, F.Cu at (150.9, 27.2)
- added R6: 15K, Resistor_SMD:R_0603_1608Metric, F.Cu at (137.8, 41.0)
- added R7: 47K, Resistor_SMD:R_0603_1608Metric, F.Cu at (137.8, 39.0)
- added R9: 10K, Resistor_SMD:R_0603_1608Metric, F.Cu at (89.4, 33.6)
- added U1: ST1S10PUR, Package_DFN_QFN:DFN-8-1EP_4x4mm_P0.8mm_EP2.5x3.6mm, F.Cu at (145.6, 27.5)
- added U3: ST1S06PUR, Package_DFN_QFN:DFN-6-1EP_3x3mm_P0.95mm_EP1.7x2.6mm, F.Cu at (131.9, 40.0)
- added Y1: 25 MHz, Crystal:Crystal_SMD_3225-4Pin_3.2x2.5mm, F.Cu at (94.1, 34.6)
- added Y2: 32.768 kHz, Crystal:Crystal_SMD_3215-2Pin_3.2x1.5mm, F.Cu at (94.0, 38.5)
- C6: renamed from C30; value 1u -> 4.7u
- Y4: renamed from Y2; footprint Crystal:Crystal_SMD_5032-2Pin_5.0x3.2mm -> Crystal:Crystal_SMD_3225-4Pin_3.2x2.5mm
- moved J11 197.0 mm to (228.3, 110.0), turned to 90 degrees
- moved C6 101.0 mm to (129.3, 40.0), turned to 90 degrees
- moved C7 99.0 mm to (127.8, 40.0), turned to 90 degrees
- moved J5 10.1 mm to (225.0, 75.0)
- moved J4 9.19 mm to (225.0, 95.0)
- renumbered C35 to C1, C1 to C31, C2 to C32, C3 to C33, C4 to C34, C5 to C35, C6 to C36, C7 to C37, C8 to C38, C9 to C39, C34 to C4, C10 to C40, C11 to C41, C12 to C42, C13 to C43, C14 to C44, C15 to C45, C23 to C46, C24 to C47, C28 to C48, C25 to C49, C26 to C50, C29 to C51, C27 to C52, C17 to C53, C16 to C54, C18 to C55, C19 to C56, C20 to C57, C21 to C58, C22 to C59, C37 to C60, C31 to C7, D8 to D1, D3 to D10, D10 to D11, D9 to D12, D11 to D13, D7 to D2, D4 to D6, D6 to D7, D1 to D8, D2 to D9, FB1 to FB2, J8 to J1, J4 to J10, J10 to J11, J17 to J12, J12 to J14, J14 to J15, J13 to J17, J15 to J18, J16 to J19, J9 to J2, J11 to J3, J1 to J4, J2 to J5, J3 to J6, J5 to J7, J7 to J8, J6 to J9, JP16 to JP1, JP30 to JP10, JP33 to JP11, JP26 to JP12, JP28 to JP13, JP27 to JP14, JP13 to JP18, JP14 to JP2, JP12 to JP26, JP1 to JP27, JP2 to JP28, JP4 to JP29, JP15 to JP3, JP5 to JP30, JP6 to JP31, JP10 to JP32, JP11 to JP33, JP3 to JP34, JP7 to JP35, JP8 to JP36, JP9 to JP37, JP19 to JP38, JP17 to JP39, JP22 to JP4, JP20 to JP40, JP29 to JP43, JP32 to JP44, JP23 to JP45, JP24 to JP46, JP25 to JP47, JP18 to JP5, JP21 to JP6, JP31 to JP9, R36 to R1, R1 to R14, R2 to R15, R5 to R16, R3 to R17, R4 to R18, R6 to R19, R35 to R2, R7 to R20, R8 to R21, R9 to R22, R20 to R23, R21 to R24, R10 to R25, R33 to R26, R11 to R27, R12 to R28, R13 to R29, R19 to R30, R14 to R31, R22 to R32, R17 to R33, R18 to R34, R23 to R35, R24 to R36, R15 to R37, R16 to R38, R26 to R39, R25 to R40, R31 to R41, R27 to R42, R28 to R43, R29 to R44, R30 to R45, R32 to R46, R45 to R47, R44 to R48, R37 to R49, R34 to R5, R46 to R50, R47 to R51, R48 to R52, R50 to R53, R49 to R54, R38 to R8, U7 to U10, U5 to U11, U6 to U12, U12 to U13, U10 to U2, U1 to U4, U2 to U5, U3 to U6, U4 to U7, Y1 to Y3
Connections:
- net /MCU/RCC_OSC_IN renamed /MCU/PH0
- C53 pad 2: Net-(U5-PD1) -> Net-(U11-PD1)
- C6 pad 1: unconnected-(C30-Pad1) -> +5V
- C6 pad 2: unconnected-(C30-Pad2) -> GND
- C7 pad 1: unconnected-(C31-Pad1) -> +5V
- C7 pad 2: unconnected-(C31-Pad2) -> GND
- J12 pad 29: unconnected-(J17-Pin_29-Pad29) -> Net-(J12-Pin_29)
- J12 pad 31: unconnected-(J17-Pin_31-Pad31) -> Net-(J12-Pin_31)
- J4 pad 1: Net-(J1-TD+) -> Net-(J4-TD+)
- J4 pad 2: Net-(J1-TD-) -> Net-(J4-TD-)
- J4 pad 7: Net-(J1-RD+) -> Net-(J4-RD+)
- J4 pad 8: Net-(J1-RD-) -> Net-(J4-RD-)
- J5 pad 1: Net-(J2-TD+) -> Net-(J5-TD+)
- J5 pad 2: Net-(J2-TD-) -> Net-(J5-TD-)
- J5 pad 7: Net-(J2-RD+) -> Net-(J5-RD+)
- J5 pad 8: Net-(J2-RD-) -> Net-(J5-RD-)
- JP39 pad 1: /MCU/PG6 -> /Connectors/PG6
- U11 pad 6: Net-(U5-PD1) -> Net-(U11-PD1)
- U4 pad 106: unconnected-(U1-VCAP_2-Pad106) -> Net-(U4-VCAP_2)
- U4 pad 108: unconnected-(U1-VDD-Pad108) -> VDD
- U4 pad 121: unconnected-(U1-VDDSDMMC-Pad121) -> VDD
- U4 pad 131: unconnected-(U1-VDD-Pad131) -> VDD
- U4 pad 138: unconnected-(U1-BOOT0-Pad138) -> /Connectors/BOOT0
- U4 pad 143: unconnected-(U1-PDR_ON-Pad143) -> VDD
- U4 pad 144: unconnected-(U1-VDD-Pad144) -> VDD
- U4 pad 17: unconnected-(U1-VDD-Pad17) -> VDD
- U4 pad 24: /MCU/RCC_OSC_OUT -> /MCU/PH1
- U4 pad 30: unconnected-(U1-VDD-Pad30) -> VDD
- U4 pad 31: GND -> GNDA
- U4 pad 32: unconnected-(U1-VREF+-Pad32) -> VDDA
- U4 pad 33: unconnected-(U1-VDDA-Pad33) -> VDDA
- U4 pad 39: unconnected-(U1-VDD-Pad39) -> VDD
- U4 pad 52: unconnected-(U1-VDD-Pad52) -> VDD
- U4 pad 6: unconnected-(U1-VBAT-Pad6) -> VBAT
- U4 pad 62: unconnected-(U1-VDD-Pad62) -> VDD
- U4 pad 71: unconnected-(U1-VCAP_1-Pad71) -> Net-(U4-VCAP_1)
- U4 pad 72: unconnected-(U1-VDD-Pad72) -> VDD
- U4 pad 84: unconnected-(U1-VDD-Pad84) -> VDD
- U4 pad 95: unconnected-(U1-VDDUSB-Pad95) -> VDD
- U7 pad 1: Net-(J1-TD+) -> Net-(J4-TD+)
- U7 pad 10: Net-(J2-TD+) -> Net-(J5-TD+)
- U7 pad 11: Net-(J2-TD-) -> Net-(J5-TD-)
- U7 pad 13: Net-(J2-RD+) -> Net-(J5-RD+)
- U7 pad 14: Net-(J2-RD-) -> Net-(J5-RD-)
- U7 pad 2: Net-(J1-TD-) -> Net-(J4-TD-)
- U7 pad 4: Net-(J1-RD+) -> Net-(J4-RD+)
- U7 pad 5: Net-(J1-RD-) -> Net-(J4-RD-)
- U8 pad 1: unconnected-(U8-I/O1-Pad1) -> Net-(J4-RD-)
- U8 pad 2: unconnected-(U8-GND-Pad2) -> GND
- U8 pad 3: unconnected-(U8-I/O2-Pad3) -> Net-(J4-RD+)
- U8 pad 4: unconnected-(U8-I/O3-Pad4) -> Net-(J4-TD+)
- U8 pad 5: unconnected-(U8-VBUS-Pad5) -> +3V3
- U8 pad 6: unconnected-(U8-I/O4-Pad6) -> Net-(J4-TD-)
- U9 pad 1: unconnected-(U9-I/O1-Pad1) -> Net-(J5-RD+)
- U9 pad 2: unconnected-(U9-GND-Pad2) -> GND
- U9 pad 3: unconnected-(U9-I/O2-Pad3) -> Net-(J5-RD-)
- U9 pad 4: unconnected-(U9-I/O3-Pad4) -> Net-(J5-TD+)
- U9 pad 5: unconnected-(U9-VBUS-Pad5) -> +3V3
- U9 pad 6: unconnected-(U9-I/O4-Pad6) -> Net-(J5-TD-)
- Y4 pad 2: Net-(U5-PD1) -> (no net)
Routing:
- net Net-(U3-FB): track 0.00 -> 11.1 mm, vias 0 -> 2
- net +5V: track 0.00 -> 9.14 mm
- net Net-(JP2-A): track 0.00 -> 6.98 mm
- net Net-(U5-PD1): track 6.91 -> 0.00 mm
- net Net-(U11-PD1): track 0.00 -> 6.91 mm
- net Net-(U3-SW): track 0.00 -> 4.51 mm
- net /Ethernet/ETH_TXD1: track 29.4 -> 27.8 mm
- net /Ethernet/ETH_RXD0: track 43.9 -> 42.3 mm
- net /Ethernet/ETH_RXD1: track 45.6 -> 44.1 mm
- net /Ethernet/ETH_TXD0: track 32.6 -> 31.0 mm
- net /Ethernet/ETH_RX_EN: track 44.2 -> 42.6 mm
- net /MCU/FMC_A12: track 42.8 -> 44.3 mm
- net /Ethernet/ETH_SPI_MISO: track 36.4 -> 35.2 mm
- net /Ethernet/ETH_SPI_SCK: track 37.6 -> 36.4 mm
- net /Ethernet/ETH_SPI_NSS: track 38.9 -> 37.8 mm
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
Commit message: tracerouting
Parts:
- JP1, JP10, JP16, JP4, JP43, JP44, JP45, JP46, JP47, JP5, JP6, JP7, JP8, JP9: moved to B.Cu
- moved R52 219.6 mm to (238.6, 125.3), turned to 180 degrees
- moved R53 217.4 mm to (238.5, 123.5), turned to 180 degrees
- moved R54 214.3 mm to (234.9, 121.9), turned to 180 degrees
- moved D12 210.5 mm to (237.9, 110.4), turned to 90 degrees
- moved D13 203.9 mm to (232.0, 123.6), turned to 90 degrees
- moved Q2 203.2 mm to (234.8, 124.4), turned to 180 degrees
- moved R47 200.0 mm to (222.0, 105.2)
- moved R49 198.3 mm to (217.6, 108.1), turned to 180 degrees
- moved C42 198.1 mm to (212.0, 102.1)
- moved R48 196.5 mm to (217.6, 105.1), turned to 180 degrees
- moved C44 196.1 mm to (212.0, 100.5)
- moved R50 193.3 mm to (214.2, 110.3), turned to 180 degrees
- moved R51 193.0 mm to (214.2, 111.8)
- moved U13 192.9 mm to (221.6, 107.7), turned to 180 degrees
- moved C39 191.8 mm to (207.6, 89.2)
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Connections:
- JP39 pad 1: /Connectors/PG6 -> /MCU/PG6
