File: HARDWARE/meshium_duo.kicad_pcb (KiCad board)
At the start: 4 copper layers, 216 parts, among them J1 Conn_02x03_Odd_Even, J10 Conn_01x04_Pin, J11 USB_B_Micro, J12 Conn_02x37_Odd_Even, J13 Conn_01x02_Pin, J14 Conn_02x08_Odd_Even, J15 Conn_02x15_Odd_Even, J16 Conn_01x02_Pin, J17 Conn_02x10_Odd_Even, J18 Conn_02x17_Odd_Even, J19 Conn_02x37_Odd_Even, J2 Conn_01x02_Pin, J3 Conn_01x02_Pin, J4 KLS12-TL051, J5 KLS12-TL051, J6 USB_B_Micro, J7 Conn_01x02_Pin, J8 Conn_01x02_Pin, J9 Conn_01x06_Pin, Q1 BC848, Q2 BC848, U1 ST1S10PUR, U10 USBLC6-2SC6, U11 STM32F103CBTx, U12 LD3985M33R_SOT23, U13 TPS2051B, U2 TPS2051B, U3 ST1S06PUR, U4 STM32F767ZITx, U5 MX25L25635F, U6 MT48LC16M16A2P, U7 KSZ8463FRL, U8 USBLC6-4SC6, U9 USBLC6-4SC6, Y1 25 MHz, Y2 32.768 kHz, Y3 25Mhz, Y4 8 MHz

Commit message: tracerouting
Parts:
- removed J4, J5: KLS12-TL051, Footpint:KLS12-TL051
- Y1: value 25 MHz -> 25MHz
- Y3: value 25Mhz -> 25MHz
- moved Y3 122.9 mm to (87.4, 36.8), turned to 0 degrees
- moved Y1 89.0 mm to (87.4, 43.2), turned to 0 degrees
- moved C1 21.7 mm to (106.6, 60.2)
- moved C4 21.7 mm to (104.3, 62.8)
- moved D1 21.7 mm to (104.3, 67.7)
- moved JP1 21.7 mm to (103.7, 61.0)
- moved R1 21.7 mm to (107.7, 65.2)
- moved R2 21.7 mm to (107.3, 67.7)
- moved U2 21.7 mm to (104.8, 65.2)
Connections:
- C1 pad 1: +5V0 -> U5V
- C46 pad 1: +3V3 -> +3V3_ST_LINK
- C47 pad 1: +3V3 -> +3V3_ST_LINK
- C49 pad 1: +3V3 -> +3V3_ST_LINK
- C5 pad 1: +5V0 -> VIN_5V
- C50 pad 1: +3V3 -> +3V3_ST_LINK
- C51 pad 1: +5V0 -> U5V
- C58 pad 1: +3V3 -> +3V3_ST_LINK
- C59 pad 1: +3V3 -> +3V3_ST_LINK
- D10 pad 2: +5V0 -> U5V
- D6 pad 2: +3V3 -> +3V3_ST_LINK
- D8 pad 2: +5V0 -> VIN_5V
- D9 pad 2: +5V0 -> E5V
- J1 pad 2: +5V0 -> E5V
- J1 pad 6: +5V0 -> VIN_5V
- J12 pad 6: +5V0 -> E5V
- J6 pad 1: +5V0 -> U5V
- J8 pad 2: +3V3 -> +3V3_ST_LINK
- JP1 pad 1: +5V0 -> U5V
- JP3 pad 2: +3V3 -> +3V3_PER
- JP34 pad 2: +3V3 -> +3V3_ST_LINK
- JP39 pad 1: /MCU/PG6 -> /Connectors/PG6
- JP44 pad 1: +3V3 -> +3V3_PER
- L1 pad 2: +5V0 -> VIN_5V
- Q1 pad 3: +3V3 -> +3V3_ST_LINK
- R1 pad 1: +5V0 -> U5V
- R2 pad 1: +5V0 -> U5V
- R23 pad 2: +3V3 -> +3V3_PER
- R28 pad 1: +5V0 -> U5V
- R30 pad 2: +3V3 -> +3V3_ST_LINK
- R39 pad 2: +3V3 -> +3V3_ST_LINK
- R4 pad 2: +5V0 -> VIN_5V
- R47 pad 1: +3V3 -> +3V3_PER
- R48 pad 1: +3V3 -> +3V3_PER
- R54 pad 1: +3V3 -> +3V3_PER
- U10 pad 5: +5V0 -> U5V
- U11 pad 1: +3V3 -> +3V3_ST_LINK
- U11 pad 24: +3V3 -> +3V3_ST_LINK
- U11 pad 36: +3V3 -> +3V3_ST_LINK
- U11 pad 48: +3V3 -> +3V3_ST_LINK
- U11 pad 9: +3V3 -> +3V3_ST_LINK
- U12 pad 5: +3V3 -> +3V3_ST_LINK
- U2 pad 5: +5V0 -> U5V
- U7 pad 1: Net-(J4-TD+) -> /Ethernet/RXM1
- U7 pad 10: Net-(J5-TD+) -> /Ethernet/RXM2
- U7 pad 11: Net-(J5-TD-) -> /Ethernet/RXP2
- U7 pad 13: Net-(J5-RD+) -> /Ethernet/TXM2
- U7 pad 14: Net-(J5-RD-) -> /Ethernet/TXP2
- U7 pad 2: Net-(J4-TD-) -> /Ethernet/RXP1
- U7 pad 4: Net-(J4-RD+) -> /Ethernet/TXM1
- U7 pad 5: Net-(J4-RD-) -> /Ethernet/TXP1
- U8 pad 1: Net-(J4-RD-) -> /Ethernet/RXM1
- U8 pad 3: Net-(J4-RD+) -> /Ethernet/RXP1
- U8 pad 4: Net-(J4-TD+) -> /Ethernet/TXM1
- U8 pad 6: Net-(J4-TD-) -> /Ethernet/TXP1
- U9 pad 1: Net-(J5-RD+) -> /Ethernet/RXM2
- U9 pad 3: Net-(J5-RD-) -> /Ethernet/RXP2
- U9 pad 4: Net-(J5-TD+) -> /Ethernet/TXM2
- U9 pad 6: Net-(J5-TD-) -> /Ethernet/TXP2
- Y1 pad 1: Net-(JP22-B) -> Net-(JP23-B)
- Y1 pad 2: (no net) -> GND
- Y1 pad 3: Net-(JP23-B) -> Net-(JP22-B)
- Y1 pad 4: (no net) -> GND
- Y3 pad 1: Net-(U7-XI) -> Net-(U7-XO)
- Y3 pad 2: Net-(U7-XO) -> GND
- Y3 pad 3: (no net) -> Net-(U7-XI)
- Y3 pad 4: (no net) -> GND

Commit message: tracerouting
Parts:
- JP15, JP2, JP22, JP23, JP3: moved to B.Cu
- moved Y1 88.7 mm to (151.7, 104.3), turned to -90 degrees
- moved L1 80.6 mm to (120.6, 97.2)
- moved R3 80.6 mm to (123.4, 105.8)
- moved R4 80.6 mm to (124.4, 103.3)
- moved C2 80.6 mm to (119.5, 108.8)
- moved C3 80.6 mm to (119.5, 107.3)
- moved C5 80.6 mm to (122.5, 103.3)
- moved U1 80.6 mm to (119.1, 103.6)
- moved L2 49.8 mm to (120.8, 82.5)
- moved JP2 45.4 mm to (125.1, 78.4)
- moved R7 43.1 mm to (120.2, 78.3), turned to 0 degrees
- moved U3 40.2 mm to (116.8, 77.3), turned to 90 degrees
- moved R6 39.5 mm to (120.2, 76.4), turned to 180 degrees
- moved C8 39.3 mm to (122.7, 77.4), turned to 90 degrees
- moved JP3 39.2 mm to (126.6, 75.8)
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Routing:
- net /Connectors/PA14: track 0.00 -> 85.4 mm, vias 0 -> 1
- net /Connectors/PG12: track 0.00 -> 75.5 mm, vias 0 -> 1
- net /Connectors/PG10: track 0.00 -> 73.0 mm, vias 0 -> 1
- net /Connectors/PG13: track 0.00 -> 69.8 mm, vias 0 -> 1
- net /Connectors/PG11: track 0.00 -> 68.2 mm, vias 0 -> 1
- net /Connectors/PC10: track 0.00 -> 67.7 mm, vias 0 -> 1
- net /Connectors/PC11: track 0.00 -> 63.7 mm, vias 0 -> 1
- net /Connectors/PC12: track 0.00 -> 59.4 mm, vias 0 -> 1
- net /Connectors/PC15: track 0.00 -> 47.7 mm, vias 0 -> 2
- net /Connectors/PD2: track 0.00 -> 46.4 mm, vias 0 -> 1
- net /Connectors/PA15: track 0.00 -> 46.1 mm, vias 0 -> 1
- net /Connectors/PB8: track 0.00 -> 45.6 mm
- net /MCU/FMC_NBL0: track 0.00 -> 42.5 mm, vias 0 -> 2
- net /Connectors/PA2: track 0.00 -> 40.9 mm, vias 0 -> 1
- net /Connectors/PB9: track 0.00 -> 40.1 mm
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Other:
- copper layers 4 -> 6

Commit message: tracerouting
Routing:
- net /Connectors/PA14: track 85.4 -> 7.78 mm
- net /Connectors/PG12: track 75.5 -> 4.03 mm
- net /Connectors/PG10: track 73.0 -> 2.06 mm
- net /Connectors/PG13: track 69.8 -> 4.00 mm
- net /Connectors/PG11: track 68.2 -> 3.03 mm
- net /Connectors/PC8: track 12.7 -> 65.4 mm
- net /Connectors/PC9: track 13.0 -> 64.6 mm
- net /Connectors/PC10: track 67.7 -> 31.1 mm
- net /Connectors/PC11: track 63.7 -> 28.0 mm
- net /Connectors/PG14: track 15.6 -> 50.7 mm
- net /Connectors/PB15: track 7.48 -> 39.9 mm
- net /Connectors/PG3: track 7.88 -> 38.8 mm
- net /Connectors/PC12: track 59.4 -> 31.2 mm
- net /Connectors/PE6: track 0.00 -> 27.6 mm
- net /Connectors/PB5: track 19.9 -> 47.4 mm
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