File: HARDWARE/st-link.kicad_sch (KiCad schematic)
At the start: 23 parts, among them J2 USB_B_Micro, Q1 BC848, U5 STM32F103CBTx, U6 LD3985M33R_SOT23, Y2 8 MHz

Commit message: schematic capture
Parts:
- renumbered C12 to C16, C11 to C17, C13 to C18, C14 to C19, C15 to C20, C16 to C21, C17 to C22, J2 to J3
Changed lines of the file:
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@@
   (symbol (lib_id "power:GND") (at 194.31 45.72 180) (unit 1)
     (in_bom yes) (on_board yes) (dnp no) (fields_autoplaced)
-    (property "Reference" "#PWR026" (at 194.31 39.37 0)
+    (property "Reference" "#PWR032" (at 194.31 39.37 0)
       (effects (font (size 1.27 1.27)) hide)
     )
@@
       (project "meshium_duo"
         (path "/2783b917-8d7b-4d69-a31c-61fb9333015c/4c1314f5-8ce3-41c8-9fa4-b5bc01ef554b"
-          (reference "#PWR026") (unit 1)
+          (reference "#PWR032") (unit 1)
         )
       )
@@
   (symbol (lib_id "Connector:USB_B_Micro") (at 41.91 147.32 0) (unit 1)
     (in_bom yes) (on_board yes) (dnp no) (fields_autoplaced)
-    (property "Reference" "J2" (at 41.91 134.62 0)
+    (property "Reference" "J3" (at 41.91 134.62 0)
       (effects (font (size 1.27 1.27)))
     )
@@
       (project "meshium_duo"
         (path "/2783b917-8d7b-4d69-a31c-61fb9333015c/4c1314f5-8ce3-41c8-9fa4-b5bc01ef554b"
-          (reference "J2") (unit 1)
+          (reference "J3") (unit 1)
         )
       )
@@
   (symbol (lib_id "power:GND") (at 144.78 127 0) (unit 1)
     (in_bom yes) (on_board yes) (dnp no) (fields_autoplaced)
-    (property "Reference" "#PWR029" (at 144.78 133.35 0)
+    (property "Reference" "#PWR030" (at 144.78 133.35 0)
       (effects (font (size 1.27 1.27)) hide)
     )
@@
       (project "meshium_duo"
         (path "/2783b917-8d7b-4d69-a31c-61fb9333015c/4c1314f5-8ce3-41c8-9fa4-b5bc01ef554b"
-          (reference "#PWR029") (unit 1)
+          (reference "#PWR030") (unit 1)
         )
       )
@@
   (symbol (lib_id "power:+5V") (at 52.07 138.43 0) (unit 1)
     (in_bom yes) (on_board yes) (dnp no) (fields_autoplaced)
-    (property "Reference" "#PWR027" (at 52.07 142.24 0)
+    (property "Reference" "#PWR028" (at 52.07 142.24 0)
       (effects (font (size 1.27 1.27)) hide)
     )
@@
       (project "meshium_duo"
         (path "/2783b917-8d7b-4d69-a31c-61fb9333015c/4c1314f5-8ce3-41c8-9fa4-b5bc01ef554b"
-          (reference "#PWR027") (unit 1)
+          (reference "#PWR028") (unit 1)
         )
       )
@@
   (symbol (lib_id "Device:C_Small") (at 200.66 52.07 0) (unit 1)
     (in_bom yes) (on_board yes) (dnp no) (fields_autoplaced)
-    (property "Reference" "C11" (at 203.2 50.8063 0)
+    (property "Reference" "C17" (at 203.2 50.8063 0)
       (effects (font (size 1.27 1.27)) (justify left))
     )
@@
       (project "meshium_duo"
         (path "/2783b917-8d7b-4d69-a31c-61fb9333015c/4c1314f5-8ce3-41c8-9fa4-b5bc01ef554b"
-          (reference "C11") (unit 1)
+          (reference "C17") (unit 1)
         )
       )
@@
   (symbol (lib_id "power:+3V3") (at 88.9 158.75 0) (unit 1)
     (in_bom yes) (on_board yes) (dnp no)
-    (property "Reference" "#PWR030" (at 88.9 162.56 0)
+    (property "Reference" "#PWR029" (at 88.9 162.56 0)
       (effects (font (size 1.27 1.27)) hide)
     )
@@
       (project "meshium_duo"
         (path "/2783b917-8d7b-4d69-a31c-61fb9333015c/4c1314f5-8ce3-41c8-9fa4-b5bc01ef554b"
-          (reference "#PWR030") (unit 1)
+          (reference "#PWR029") (unit 1)
         )
       )
@@
   (symbol (lib_id "Device:C_Small") (at 264.16 156.21 0) (unit 1)
     (in_bom yes) (on_board yes) (dnp no) (fields_autoplaced)
-    (property "Reference" "C17" (at 266.7 154.9463 0)
+    (property "Reference" "C22" (at 266.7 154.9463 0)
       (effects (font (size 1.27 1.27)) (justify left))
     )
@@
       (project "meshium_duo"
         (path "/2783b917-8d7b-4d69-a31c-61fb9333015c/4c1314f5-8ce3-41c8-9fa4-b5bc01ef554b"
-          (reference "C17") (unit 1)
+          (reference "C22") (unit 1)
         )
       )
@@
   (symbol (lib_id "Device:C_Small") (at 227.33 156.21 0) (unit 1)
     (in_bom yes) (on_board yes) (dnp no) (fields_autoplaced)
-    (property "Reference" "C14" (at 229.87 154.9463 0)
+    (property "Reference" "C19" (at 229.87 154.9463 0)
       (effects (font (size 1.27 1.27)) (justify left))
     )
@@
       (project "meshium_duo"
         (path "/2783b917-8d7b-4d69-a31c-61fb9333015c/4c1314f5-8ce3-41c8-9fa4-b5bc01ef554b"
-          (reference "C14") (unit 1)
+          (reference "C19") (unit 1)
         )
       )
@@
   (symbol (lib_id "Device:C_Small") (at 250.19 156.21 0) (unit 1)
     (in_bom yes) (on_board yes) (dnp no) (fields_autoplaced)
-    (property "Reference" "C15" (at 252.73 154.9463 0)
+    (property "Reference" "C20" (at 252.73 154.9463 0)
       (effects (font (size 1.27 1.27)) (justify left))
     )
@@
       (project "meshium_duo"
         (path "/2783b917-8d7b-4d69-a31c-61fb9333015c/4c1314f5-8ce3-41c8-9fa4-b5bc01ef554b"
-          (reference "C15") (unit 1)
+          (reference "C20") (unit 1)
         )
       )
@@
   (symbol (lib_id "Device:C_Small") (at 187.96 52.07 0) (unit 1)
     (in_bom yes) (on_board yes) (dnp no)
-    (property "Reference" "C12" (at 182.88 50.8 0)
+    (property "Reference" "C16" (at 182.88 50.8 0)
       (effects (font (size 1.27 1.27)) (justify left))
     )
@@
       (project "meshium_duo"
         (path "/2783b917-8d7b-4d69-a31c-61fb9333015c/4c1314f5-8ce3-41c8-9fa4-b5bc01ef554b"
-          (reference "C12") (unit 1)
+          (reference "C16") (unit 1)
         )
       )
@@
   (symbol (lib_id "Device:C_Small") (at 217.17 153.67 0) (unit 1)
     (in_bom yes) (on_board yes) (dnp no) (fields_autoplaced)
-    (property "Reference" "C13" (at 219.71 152.4063 0)
+    (property "Reference" "C18" (at 219.71 152.4063 0)
       (effects (font (size 1.27 1.27)) (justify left))
     )
@@
       (project "meshium_duo"
         (path "/2783b917-8d7b-4d69-a31c-61fb9333015c/4c1314f5-8ce3-41c8-9fa4-b5bc01ef554b"
-          (reference "C13") (unit 1)
+          (reference "C18") (unit 1)
         )
       )
@@
   (symbol (lib_id "Device:C_Small") (at 257.81 152.4 0) (unit 1)
     (in_bom yes) (on_board yes) (dnp no) (fields_autoplaced)
-    (property "Reference" "C16" (at 260.35 151.1363 0)
+    (property "Reference" "C21" (at 260.35 151.1363 0)
       (effects (font (size 1.27 1.27)) (justify left))
     )
@@
       (project "meshium_duo"
         (path "/2783b917-8d7b-4d69-a31c-61fb9333015c/4c1314f5-8ce3-41c8-9fa4-b5bc01ef554b"
-          (reference "C16") (unit 1)
+          (reference "C21") (unit 1)
         )
       )
@@
   (symbol (lib_id "power:GND") (at 264.16 100.33 90) (unit 1)
     (in_bom yes) (on_board yes) (dnp no) (fields_autoplaced)
-    (property "Reference" "#PWR032" (at 270.51 100.33 0)
+    (property "Reference" "#PWR034" (at 270.51 100.33 0)
       (effects (font (size 1.27 1.27)) hide)
     )
@@
       (project "meshium_duo"
         (path "/2783b917-8d7b-4d69-a31c-61fb9333015c/4c1314f5-8ce3-41c8-9fa4-b5bc01ef554b"
-          (reference "#PWR032") (unit 1)
+          (reference "#PWR034") (unit 1)
         )
       )
@@
   (symbol (lib_id "power:GND") (at 39.37 160.02 0) (unit 1)
     (in_bom yes) (on_board yes) (dnp no) (fields_autoplaced)
-    (property "Reference" "#PWR028" (at 39.37 166.37 0)
+    (property "Reference" "#PWR027" (at 39.37 166.37 0)
       (effects (font (size 1.27 1.27)) hide)
     )
@@
       (project "meshium_duo"
         (path "/2783b917-8d7b-4d69-a31c-61fb9333015c/4c1314f5-8ce3-41c8-9fa4-b5bc01ef554b"
-          (reference "#PWR028") (unit 1)
+          (reference "#PWR027") (unit 1)
         )
       )
@@
   (symbol (lib_id "power:GND") (at 217.17 162.56 0) (unit 1)
     (in_bom yes) (on_board yes) (dnp no) (fields_autoplaced)
-    (property "Reference" "#PWR031" (at 217.17 168.91 0)
+    (property "Reference" "#PWR033" (at 217.17 168.91 0)
       (effects (font (size 1.27 1.27)) hide)
     )
@@
       (project "meshium_duo"
         (path "/2783b917-8d7b-4d69-a31c-61fb9333015c/4c1314f5-8ce3-41c8-9fa4-b5bc01ef554b"
-          (reference "#PWR031") (unit 1)
+          (reference "#PWR033") (unit 1)
         )
       )
@@
   (symbol (lib_id "power:GND") (at 167.64 83.82 90) (unit 1)
     (in_bom yes) (on_board yes) (dnp no) (fields_autoplaced)
-    (property "Reference" "#PWR025" (at 173.99 83.82 0)
+    (property "Reference" "#PWR031" (at 173.99 83.82 0)
       (effects (font (size 1.27 1.27)) hide)
     )
@@
       (project "meshium_duo"
         (path "/2783b917-8d7b-4d69-a31c-61fb9333015c/4c1314f5-8ce3-41c8-9fa4-b5bc01ef554b"
-          (reference "#PWR025") (unit 1)
-        )
-      )
+          (reference "#PWR031") (unit 1)
+        )
+      )

Commit message: schematic capture
Parts:
- added C23, C24, C25, C26, C27: 0.1u, Resistor_SMD:R_0603_1608Metric, symbol Device:C_Small
- added C28: 10p, symbol Device:C_Small
- added D5, D6: BAT60A, Diode_SMD:D_SOD-323, symbol Diode:BAT60A
- added J4: Conn_01x04_Pin, symbol Connector:Conn_01x04_Pin
- added J5, J7: Conn_01x02_Pin, symbol Connector:Conn_01x02_Pin
- added J6: Conn_01x06_Pin, symbol Connector:Conn_01x06_Pin
- added JP1: SolderJumper_3_Open, symbol Jumper:SolderJumper_3_Open
- added JP10, JP11, JP12, JP2, JP4, JP5, JP6: Jumper_2_Bridged, symbol Jumper:Jumper_2_Bridged
- added JP3, JP7, JP8, JP9: Jumper_2_Open, symbol Jumper:Jumper_2_Open
- added R17, R18, R19, R31: 10K, symbol Device:R_Small
- added R20, R21, R23, R24: 4K7, symbol Device:R_Small
- added R22, R32, R33: 100, symbol Device:R_Small
- added R25, R26: 100K, symbol Device:R_Small
- added R27, R28, R29, R30: 22, symbol Device:R_Small
Connections:
- net +3V3: now also C21.1, C22.1, D4.1 (A1), U5.1 (VBAT), U5.24 (VDD), U5.36 (VDD), U5.48 (VDD), U5.9 (VDDA), U6.5 (VOUT), C23.1, C24.1, C25.1, C26.1, J7.2 (Pin_2), JP3.2 (B), R19.2, R20.2, R26.2
- net +5V: now also D5.2 (A); no longer J3.1 (VBUS)
- net AIN1: now also R20.1, R21.2, R32.1
- net GND: now also R13.2, C23.2, C24.2, C25.2, C26.2, C27.2, C28.1, J6.3 (Pin_3), JP8.2 (B), R17.1, R18.1, R21.1, R24.1, R25.1, R31.2
- net MCO: now also JP12.1 (A), R33.2
- net PWR_EXT: now also J7.1 (Pin_1), R23.1, R24.2
- net STM_JTCK: now also JP7.2 (B)
- net STM_JTMS: now also JP9.2 (B)
- net T_JTCK: now also JP2.1 (A), R27.1
- net T_JTMS: now also JP5.1 (A), R22.1, R28.1
- net T_NRST: now also JP10.1 (A), R29.1
- net T_SWDIO_IN: now also R22.2
- net T_SWO: now also JP11.1 (A), R30.1
- net +5V0: now reaches D2.2 (A)
- net +5V0: now also D1.2 (A), D3.2 (A), J3.1 (VBUS), R12.1
- net at U5.44 (BOOT0): now also JP1.2 (C)
- net BI0: no longer names the net of U5.2 (PC13)
- net BI0: now also R18.2
- net BI1: no longer names the net of U5.3 (PC14)
- net BI1: now also R17.2
- net STLNK_RX renamed STLINK_RX
- net STLINK_RX: now also J5.2 (Pin_2)
- net STLNK_TX renamed STLINK_TX
- net STLINK_TX: now also J5.1 (Pin_1)
- net STM_RST: no longer names the net of U5.7 (NRST)
- net STM_RST: now also C27.1, R19.1
- new net: D6.1 (K), R32.2
- new net: J4.1 (Pin_1), JP2.2 (B), JP3.1 (A)
- new net: J6.6 (Pin_6), R30.2
- new net: C28.2, JP12.2 (B), R33.1
- new net: J6.5 (Pin_5), R29.2
- new net: D6.2 (A), J6.1 (Pin_1)
- new net: JP1.1 (A), R26.1
- new net: J4.2 (Pin_2), JP4.2 (B), JP7.1 (A)
- new net: D5.1 (K), R23.2
- new net: J6.2 (Pin_2), R27.2
- new net: J6.4 (Pin_4), R28.2
- new net: J4.3 (Pin_3), JP5.2 (B), JP8.1 (A)
- new net: JP1.3 (B), R25.2
- new net: J4.4 (Pin_4), JP6.2 (B), JP9.1 (A)
- new net NRST: JP10.2 (B)
- new net SWO: JP11.2 (B)
- new net TCK: JP6.1 (A)
- new net TMS: JP4.1 (A)
Other:
- note removed: "STLINK"
- moved on the sheet: C18, C19, C20, C21, C22, D1, D2, D3, D4, J3, Q1, R10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

Commit message: schematic capture
Parts:
- added C29: 0.1u, Capacitor_SMD:C_0603_1608Metric, symbol Device:C_Small
- added U7: USBLC6-2SC6, Package_TO_SOT_SMD:SOT-23-6, symbol Power_Protection:USBLC6-2SC6
- C16, C17, C28: footprint (none) -> Capacitor_SMD:C_0603_1608Metric
- C18, C19, C20, C21, C22, C23, C24, C25, C26, C27: footprint Resistor_SMD:R_0603_1608Metric -> Capacitor_SMD:C_0603_1608Metric
- D4: footprint (none) -> Footpint:LED_Kingbright_KPBD-3224
- J3: footprint (none) -> Footpint:USB_Micro-B_CUZD188-CB1Z
- J4: footprint (none) -> Connector_PinHeader_2.54mm:PinHeader_1x04_P2.54mm_Vertical
- J5, J7: footprint (none) -> Connector_PinHeader_2.54mm:PinHeader_1x02_P2.54mm_Vertical
- J6: footprint (none) -> Connector_PinHeader_2.54mm:PinHeader_1x06_P2.54mm_Vertical
- JP1: footprint (none) -> Jumper:SolderJumper-3_P2.0mm_Open_TrianglePad1.0x1.5mm_NumberLabels
- JP10, JP11, JP12, JP2, JP3, JP4, JP5, JP6, JP7, JP8, JP9: footprint (none) -> Jumper:SolderJumper-2_P1.3mm_Open_TrianglePad1.0x1.5mm
- R10, R11, R12, R13, R14, R15, R16, R17, R18, R19, R20, R21, R22, R23, R24, R25, R26, R27, R28, R29, R30, R31, R32, R33: footprint (none) -> Resistor_SMD:R_0603_1608Metric
- Y2: footprint (none) -> Crystal:Crystal_SMD_5032-2Pin_5.0x3.2mm
Connections:
- net +3V3: now also D4.2 (A2); no longer D4.1 (A1)
- net +5V0: now also C29.1, U7.5 (VBUS)
- net GND: now also D4.3 (K1), C29.2, U7.2 (GND); no longer D4.4 (K2)
- net STLINK_USB_DM: now also J3.2 (D-), U7.1 (I/O1), U7.6 (I/O1); no longer J3.3 (D+), R11.1
- net STLINK_USB_DP: now also J3.3 (D+), R11.1, U7.3 (I/O2), U7.4 (I/O2); no longer J3.2 (D-)
- net at R16.2: now also D4.1 (A1); no longer D4.2 (A2)
- net at R15.2: now also D4.4 (K2); no longer D4.3 (K1)
- net at D6.2 (A), J6.1 (Pin_1): now also R31.1
Other:
- moved on the sheet: Q1, R11, R12, R13, R14, R15, R16

Commit message: schematic capture
Parts:
- Y2: footprint Crystal:Crystal_SMD_5032-2Pin_5.0x3.2mm -> Crystal:Crystal_SMD_3225-4Pin_3.2x2.5mm
Connections:
- net at C17.2, U5.6 (PD1): now also Y2.3; no longer Y2.2
Changed lines of the file:
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@@
       (effects (font (size 1.27 1.27)))
     )
-    (property "Footprint" "Crystal:Crystal_SMD_5032-2Pin_5.0x3.2mm" (at 147.32 68.58 0)
+    (property "Footprint" "Crystal:Crystal_SMD_3225-4Pin_3.2x2.5mm" (at 147.32 68.58 0)
       (effects (font (size 1.27 1.27)) hide)
     )
@@
     )
     (pin "1")
-    (pin "2")
+    (pin "3")
     (instances
       (project "meshium_duo"

Commit message: schematic capture
Parts:
- renumbered C23 to C46, C24 to C47, C28 to C48, C25 to C49, C26 to C50, C29 to C51, C27 to C52, C17 to C53, C16 to C54, C18 to C55, C19 to C56, C20 to C57, C21 to C58, C22 to C59, D3 to D10, D4 to D6, D6 to D7, D1 to D8, D2 to D9, J4 to J10, J3 to J6, J5 to J7, J7 to J8, J6 to J9, JP12 to JP26, JP1 to JP27, JP2 to JP28, JP4 to JP29, JP5 to JP30, JP6 to JP31, JP10 to JP32, JP11 to JP33, JP3 to JP34, JP7 to JP35, JP8 to JP36, JP9 to JP37, R20 to R23, R21 to R24, R10 to R25, R33 to R26, R11 to R27, R12 to R28, R13 to R29, R19 to R30, R14 to R31, R22 to R32, R17 to R33, R18 to R34, R23 to R35, R24 to R36, R15 to R37, R16 to R38, R26 to R39, R25 to R40, R31 to R41, R27 to R42, R28 to R43, R29 to R44, R30 to R45, R32 to R46, U7 to U10, U5 to U11, U6 to U12, Y2 to Y4

Commit message: tracerouting
Connections:
- net +3V3 renamed +3V3_ST_LINK
- net +3V3_ST_LINK: no longer R23.2
- net +5V0 renamed U5V
- net U5V: no longer D8.2 (A), D9.2 (A)
- new net +3V3_PER: R23.2
- new net E5V: D9.2 (A)
- new net VIN_5V: D8.2 (A)
