File: HARDWARE/Connectors.kicad_sch (KiCad schematic)
At the start: 11 parts, among them J12 Conn_02x08_Odd_Even, J13 Conn_02x10_Odd_Even, J14 Conn_02x15_Odd_Even, J15 Conn_02x17_Odd_Even, J16 Conn_02x36_Odd_Even, J17 Conn_02x36_Odd_Even

Commit message: schematic capture
Parts:
- removed J16, J17: Conn_02x36_Odd_Even, symbol Connector_Generic:Conn_02x36_Odd_Even
- added J16, J17: Conn_02x37_Odd_Even, Connector_PinHeader_2.54mm:PinHeader_2x37_P2.54mm_Vertical, symbol Connector_Generic:Conn_02x37_Odd_Even
- J12: footprint (none) -> Connector_PinHeader_2.54mm:PinHeader_2x08_P2.54mm_Vertical
- J13: footprint (none) -> Connector_PinHeader_2.54mm:PinHeader_2x10_P2.54mm_Vertical
- J14: footprint (none) -> Connector_PinHeader_2.54mm:PinHeader_2x15_P2.54mm_Vertical
- J15: footprint (none) -> Connector_PinHeader_2.54mm:PinHeader_2x16_P2.54mm_Vertical
Connections:
- net +5V0: now also J17.6 (Pin_6)
- net BOOT0: now also J17.7 (Pin_7)
- net GND: now also J16.20 (Pin_20), J16.39 (Pin_39), J16.54 (Pin_54), J16.63 (Pin_63), J16.73 (Pin_73), J16.74 (Pin_74), J16.9 (Pin_9), J17.19 (Pin_19), J17.20 (Pin_20), J17.22 (Pin_22), J17.49 (Pin_49), J17.60 (Pin_60), J17.73 (Pin_73), J17.74 (Pin_74), J17.8 (Pin_8)
- net GNDA: now also J16.32 (Pin_32)
- net IOREF: now also J17.12 (Pin_12)
- net NRST: now also J17.14 (Pin_14)
- net PA0: now also J17.28 (Pin_28)
- net PA10: now also J16.33 (Pin_33)
- net PA11: now also J16.14 (Pin_14)
- net PA12: now also J16.12 (Pin_12)
- net PA13: now also J17.13 (Pin_13)
- net PA14: now also J17.15 (Pin_15)
- net PA15: now also J17.17 (Pin_17)
- net PA2: now also J16.35 (Pin_35)
- net PA3: now also J16.37 (Pin_37)
- net PA8: now also J16.21 (Pin_21)
- net PA9: now also J16.19 (Pin_19)
- net PB0: now also J17.34 (Pin_34)
- net PB1: now also J16.24 (Pin_24)
- net PB14: now also J16.28 (Pin_28)
- net PB15: now also J16.26 (Pin_26)
- net PB2: now also J16.22 (Pin_22)
- net PB3: now also J16.31 (Pin_31)
- net PB4: now also J16.27 (Pin_27)
- net PB5: now also J16.29 (Pin_29)
- net PB6: now also J16.15 (Pin_15)
- net PB7: now also J17.21 (Pin_21)
- net PB8: now also J16.3 (Pin_3)
- net PB9: now also J16.5 (Pin_5)
- net PC1: now also J17.36 (Pin_36)
- net PC10: now also J17.1 (Pin_1)
- net PC11: now also J17.2 (Pin_2)
- net PC12: now also J17.3 (Pin_3)
- net PC13: now also J17.23 (Pin_23)
- net PC14: now also J17.25 (Pin_25)
- net PC15: now also J17.27 (Pin_27)
- net PC6: now also J16.4 (Pin_4)
- net PC7: now also J16.17 (Pin_17)
- net PC8: now also J16.2 (Pin_2)
- net PC9: now also J16.1 (Pin_1)
- net PD11: now also J16.45 (Pin_45)
- net PD12: now also J16.43 (Pin_43)
- net PD13: now also J16.41 (Pin_41)
- net PD2: now also J17.4 (Pin_4)
- net PD3: now also J17.40 (Pin_40)
- net PD4: now also J17.39 (Pin_39)
- net PD5: now also J17.41 (Pin_41)
- net PD6: now also J17.43 (Pin_43)
- net PE3: now also J17.47 (Pin_47)
- net PE4: now also J17.48 (Pin_48)
- net PE5: now also J17.50 (Pin_50)
- net PE6: now also J17.62 (Pin_62)
- net PG10: now also J17.66 (Pin_66)
- net PG11: now also J17.70 (Pin_70)
- net PG12: now also J17.65 (Pin_65)
- net PG13: now also J17.68 (Pin_68)
- net PG14: now also J16.61 (Pin_61)
- net PG3: now also J17.44 (Pin_44)
- net PG6: now also J16.70 (Pin_70)
- net PG7: now also J16.67 (Pin_67)
- net PG9: now also J17.63 (Pin_63)
- net VBAT: now also J17.33 (Pin_33)
- net VDD: now also J17.5 (Pin_5)
- net VDDA: now also J16.7 (Pin_7)

Commit message: schematic capture
Parts:
- added JP9 (x2): Jumper_2_Open, Jumper:SolderJumper-2_P1.3mm_Open_TrianglePad1.0x1.5mm, symbol Jumper:Jumper_2_Open
Connections:
- net at J17.29 (Pin_29): now also JP9.2 (B)
- net at J17.31 (Pin_31): now also JP9.2 (B)
- new net PH0: JP9.1 (A)
- new net PH1: JP9.1 (A)
Changed lines of the file:
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@@
+    (stroke (width 0) (type default))
+  )
+  (wire (pts (xy 17.78 88.9) (xy 27.94 88.9))
     (stroke (width 0) (type default))
   )
@@
     (stroke (width 0) (type default))
   )
+  (wire (pts (xy 38.1 88.9) (xy 41.91 88.9))
+    (stroke (width 0) (type default))
+  )
   (wire (pts (xy 231.14 72.39) (xy 242.57 72.39))
     (stroke (width 0) (type default))
@@
     (stroke (width 0) (type default))
   )
+  (wire (pts (xy 38.1 86.36) (xy 41.91 86.36))
+    (stroke (width 0) (type default))
+  )
   (wire (pts (xy 231.14 133.35) (xy 242.57 133.35))
     (stroke (width 0) (type default))
@@
     (stroke (width 0) (type default))
   )
+  (wire (pts (xy 17.78 86.36) (xy 27.94 86.36))
+    (stroke (width 0) (type default))
+  )
   (wire (pts (xy 39.37 111.76) (xy 41.91 111.76))
     (stroke (width 0) (type default))
@@
     (effects (font (size 1.27 1.27)) (justify left bottom))
   )
+  (label "PH0" (at 17.78 86.36 0) (fields_autoplaced)
+    (effects (font (size 1.27 1.27)) (justify left bottom))
+  )
   (label "PB0" (at 66.04 91.44 180) (fields_autoplaced)
     (effects (font (size 1.27 1.27)) (justify right bottom))
@@
   (label "PB14" (at 266.7 82.55 180) (fields_autoplaced)
     (effects (font (size 1.27 1.27)) (justify right bottom))
+  )
+  (label "PH1" (at 17.78 88.9 0) (fields_autoplaced)
+    (effects (font (size 1.27 1.27)) (justify left bottom))
   )
   (label "PA3" (at 231.14 95.25 0) (fields_autoplaced)
@@
     )
   )
+  (symbol (lib_id "Jumper:Jumper_2_Open") (at 33.02 86.36 0) (unit 1)
+    (in_bom yes) (on_board yes) (dnp no)
+    (property "Reference" "JP9" (at 26.67 85.09 0)
+      (effects (font (size 1.27 1.27)))
+    )
+    (property "Value" "Jumper_2_Open" (at 33.02 82.55 0)
+      (effects (font (size 1.27 1.27)) hide)
+    )
+    (property "Footprint" "Jumper:SolderJumper-2_P1.3mm_Open_TrianglePad1.0x1.5mm" (at 33.02 86.36 0)
+      (effects (font (size 1.27 1.27)) hide)
+    )
+    (property "Datasheet" "~" (at 33.02 86.36 0)
+      (effects (font (size 1.27 1.27)) hide)
+    )
+    (pin "1")
+    (pin "2")
+    (instances
+      (project "meshium_duo"
+        (path "/2783b917-8d7b-4d69-a31c-61fb9333015c/4c1314f5-8ce3-41c8-9fa4-b5bc01ef554b"
+          (reference "JP9") (unit 1)
+        )
+        (path "/2783b917-8d7b-4d69-a31c-61fb9333015c/b6a51085-368c-402e-8235-8439715b747c"
+          (reference "JP46") (unit 1)
+        )
+      )
+    )
+  )
   (symbol (lib_id "power:GND") (at 184.15 134.62 0) (unit 1)
     (in_bom yes) (on_board yes) (dnp no) (fields_autoplaced)
@@
         )
       )
+    )
+  )
+  (symbol (lib_id "Jumper:Jumper_2_Open") (at 33.02 88.9 0) (unit 1)
+    (in_bom yes) (on_board yes) (dnp no)
+    (property "Reference" "JP9" (at 26.67 87.63 0)
+      (effects (font (size 1.27 1.27)))
+    )
+    (property "Value" "Jumper_2_Open" (at 33.02 85.09 0)
+      (effects (font (size 1.27 1.27)) hide)
+    )
+    (property "Footprint" "Jumper:SolderJumper-2_P1.3mm_Open_TrianglePad1.0x1.5mm" (at 33.02 88.9 0)
+      (effects (font (size 1.27 1.27)) hide)
+    )
+    (property "Datasheet" "~" (at 33.02 88.9 0)
+      (effects (font (size 1.27 1.27)) hide)
+    )
+    (pin "1")
+    (pin "2")
+    (instances
+      (project "meshium_duo"
+        (path "/2783b917-8d7b-4d69-a31c-61fb9333015c/4c1314f5-8ce3-41c8-9fa4-b5bc01ef554b"
+          (reference "JP9") (unit 1)
+        )
+        (path "/2783b917-8d7b-4d69-a31c-61fb9333015c/b6a51085-368c-402e-8235-8439715b747c"
+          (reference "JP47") (unit 1)
+        )
+      )

Commit message: schematic capture
Parts:
- added J? (x2): Conn_01x02_Pin, Connector_PinHeader_2.54mm:PinHeader_1x02_P2.54mm_Vertical, symbol Connector:Conn_01x02_Pin
- renumbered J17 to J12, J12 to J14, J14 to J15, J13 to J17, J15 to J18, J16 to J19, JP9 to JP?, JP6 to JP?
Connections:
- net GND: now also J?.1 (Pin_1), J?.1 (Pin_1), J?.2 (Pin_2), J?.2 (Pin_2)

Commit message: tracerouting
Connections:
- net +3V3: no longer JP?.1 (A)
- net +5V0 renamed E5V
- new net +3V3_PER: JP?.1 (A)
Changed lines of the file:
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@@
-    )
-  )
-  (symbol (lib_id "meshium_duo:VIN") (at 104.14 67.31 90) (unit 1)
-    (in_bom yes) (on_board yes) (dnp no) (fields_autoplaced)
-    (property "Reference" "#PWR0132" (at 107.95 67.31 0)
-      (effects (font (size 1.27 1.27)) hide)
-    )
-    (property "Value" "VIN" (at 100.33 67.31 90)
-      (effects (font (size 1.27 1.27)) (justify left))
-    )
-    (property "Footprint" "" (at 104.14 67.31 0)
-      (effects (font (size 1.27 1.27)) hide)
-    )
-    (property "Datasheet" "" (at 104.14 67.31 0)
-      (effects (font (size 1.27 1.27)) hide)
-    )
-    (pin "1")
-    (instances
-      (project "meshium_duo"
-        (path "/2783b917-8d7b-4d69-a31c-61fb9333015c/b6a51085-368c-402e-8235-8439715b747c"
-          (reference "#PWR0132") (unit 1)
-        )
-      )
     )
   )
@@
         (path "/2783b917-8d7b-4d69-a31c-61fb9333015c/b6a51085-368c-402e-8235-8439715b747c"
           (reference "#PWR0135") (unit 1)
+        )
+      )
+    )
+  )
+  (symbol (lib_id "meshium_duo:+3V3_PER") (at 78.74 36.83 90) (unit 1)
+    (in_bom yes) (on_board yes) (dnp no) (fields_autoplaced)
+    (property "Reference" "#PWR091" (at 82.55 36.83 0)
+      (effects (font (size 1.27 1.27)) hide)
+    )
+    (property "Value" "+3V3_PER" (at 74.93 36.83 90)
+      (effects (font (size 1.27 1.27)) (justify left))
+    )
+    (property "Footprint" "" (at 78.74 36.83 0)
+      (effects (font (size 1.27 1.27)) hide)
+    )
+    (property "Datasheet" "" (at 78.74 36.83 0)
+      (effects (font (size 1.27 1.27)) hide)
+    )
+    (pin "1")
+    (instances
+      (project "meshium_duo"
+        (path "/2783b917-8d7b-4d69-a31c-61fb9333015c/b6a51085-368c-402e-8235-8439715b747c"
+          (reference "#PWR091") (unit 1)
         )
       )
@@
     )
   )
-  (symbol (lib_id "meshium_duo:+3V3_PER") (at 78.74 36.83 90) (unit 1)
-    (in_bom yes) (on_board yes) (dnp no) (fields_autoplaced)
-    (property "Reference" "#PWR0130" (at 82.55 36.83 0)
-      (effects (font (size 1.27 1.27)) hide)
-    )
-    (property "Value" "+3V3_PER" (at 74.93 36.83 90)
-      (effects (font (size 1.27 1.27)) (justify left))
-    )
-    (property "Footprint" "" (at 78.74 36.83 0)
-      (effects (font (size 1.27 1.27)) hide)
-    )
-    (property "Datasheet" "" (at 78.74 36.83 0)
-      (effects (font (size 1.27 1.27)) hide)
-    )
-    (pin "1")
-    (instances
-      (project "meshium_duo"
-        (path "/2783b917-8d7b-4d69-a31c-61fb9333015c/b6a51085-368c-402e-8235-8439715b747c"
-          (reference "#PWR0130") (unit 1)
-        )
-      )
-    )
-  )
   (symbol (lib_id "power:VDD") (at 39.37 46.99 0) (unit 1)
     (in_bom yes) (on_board yes) (dnp no) (fields_autoplaced)
@@
         (path "/2783b917-8d7b-4d69-a31c-61fb9333015c/b6a51085-368c-402e-8235-8439715b747c"
           (reference "JP41") (unit 1)
+        )
+      )
+    )
+  )
+  (symbol (lib_id "meshium_duo:VIN") (at 104.14 67.31 90) (unit 1)
+    (in_bom yes) (on_board yes) (dnp no) (fields_autoplaced)
+    (property "Reference" "#PWR089" (at 107.95 67.31 0)
+      (effects (font (size 1.27 1.27)) hide)
+    )
+    (property "Value" "VIN" (at 100.33 67.31 90)
+      (effects (font (size 1.27 1.27)) (justify left))
+    )
+    (property "Footprint" "" (at 104.14 67.31 0)
+      (effects (font (size 1.27 1.27)) hide)
+    )
+    (property "Datasheet" "" (at 104.14 67.31 0)
+      (effects (font (size 1.27 1.27)) hide)
+    )
+    (pin "1")
+    (instances
+      (project "meshium_duo"
+        (path "/2783b917-8d7b-4d69-a31c-61fb9333015c/b6a51085-368c-402e-8235-8439715b747c"
+          (reference "#PWR089") (unit 1)
         )
       )
@@
     )
   )
+  (symbol (lib_name "E5V_1") (lib_id "meshium_duo:E5V") (at 66.04 55.88 270) (unit 1)
+    (in_bom yes) (on_board yes) (dnp no) (fields_autoplaced)
+    (property "Reference" "#PWR087" (at 62.23 55.88 0)
+      (effects (font (size 1.27 1.27)) hide)
+    )
+    (property "Value" "E5V" (at 69.85 55.88 90)
+      (effects (font (size 1.27 1.27)) (justify left))
+    )
+    (property "Footprint" "" (at 66.04 55.88 0)
+      (effects (font (size 1.27 1.27)) hide)
+    )
+    (property "Datasheet" "" (at 66.04 55.88 0)
+      (effects (font (size 1.27 1.27)) hide)
+    )
+    (pin "1")
+    (instances
+      (project "meshium_duo"
+        (path "/2783b917-8d7b-4d69-a31c-61fb9333015c/b6a51085-368c-402e-8235-8439715b747c"
+          (reference "#PWR087") (unit 1)
+        )
+      )
+    )
+  )
   (symbol (lib_id "meshium_duo:IOREF") (at 113.03 45.72 0) (unit 1)
     (in_bom yes) (on_board yes) (dnp no) (fields_autoplaced)
@@
         )
       )
-    )
-  )
-  (symbol (lib_id "meshium_duo:E5V") (at 66.04 55.88 270) (unit 1)
-    (in_bom yes) (on_board yes) (dnp no) (fields_autoplaced)
-    (property "Reference" "#PWR0127" (at 62.23 55.88 0)
-      (effects (font (size 1.27 1.27)) hide)
-    )
-    (property "Value" "E5V" (at 69.85 55.88 90)
-      (effects (font (size 1.27 1.27)) (justify left))
-    )
-    (property "Footprint" "" (at 66.04 55.88 0)
-      (effects (font (size 1.27 1.27)) hide)
-    )
-    (property "Datasheet" "" (at 66.04 55.88 0)
-      (effects (font (size 1.27 1.27)) hide)
-    )
-    (pin "1")
-    (instances
-      (project "meshium_duo"
-        (path "/2783b917-8d7b-4d69-a31c-61fb9333015c/b6a51085-368c-402e-8235-8439715b747c"
-          (reference "#PWR0127") (unit 1)
-        )
-      )

Commit message: tracerouting
Parts:
- gave numbers to parts that had none: 9
Changed lines of the file:
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@@
   (symbol (lib_id "Jumper:Jumper_2_Open") (at 33.02 86.36 0) (unit 1)
     (in_bom yes) (on_board yes) (dnp no)
-    (property "Reference" "JP?" (at 26.67 85.09 0)
+    (property "Reference" "JP41" (at 26.67 85.09 0)
       (effects (font (size 1.27 1.27)))
     )
@@
     (instances
       (project "meshium_duo"
-        (path "/2783b917-8d7b-4d69-a31c-61fb9333015c/4c1314f5-8ce3-41c8-9fa4-b5bc01ef554b"
-          (reference "JP?") (unit 1)
-        )
         (path "/2783b917-8d7b-4d69-a31c-61fb9333015c/b6a51085-368c-402e-8235-8439715b747c"
           (reference "JP41") (unit 1)
@@
   (symbol (lib_id "Connector:Conn_01x02_Pin") (at 128.27 172.72 270) (unit 1)
     (in_bom yes) (on_board yes) (dnp no) (fields_autoplaced)
-    (property "Reference" "J?" (at 129.54 173.355 90)
+    (property "Reference" "J16" (at 129.54 173.355 90)
       (effects (font (size 1.27 1.27)) (justify left))
     )
@@
     (instances
       (project "meshium_duo"
-        (path "/2783b917-8d7b-4d69-a31c-61fb9333015c/4c1314f5-8ce3-41c8-9fa4-b5bc01ef554b"
-          (reference "J?") (unit 1)
-        )
-        (path "/2783b917-8d7b-4d69-a31c-61fb9333015c"
-          (reference "J?") (unit 1)
-        )
         (path "/2783b917-8d7b-4d69-a31c-61fb9333015c/b6a51085-368c-402e-8235-8439715b747c"
           (reference "J16") (unit 1)
@@
   (symbol (lib_id "Jumper:Jumper_2_Bridged") (at 90.17 96.52 0) (unit 1)
     (in_bom yes) (on_board yes) (dnp no)
-    (property "Reference" "JP?" (at 83.82 95.25 0)
+    (property "Reference" "JP45" (at 83.82 95.25 0)
       (effects (font (size 1.27 1.27)))
     )
@@
     (instances
       (project "meshium_duo"
-        (path "/2783b917-8d7b-4d69-a31c-61fb9333015c/4c1314f5-8ce3-41c8-9fa4-b5bc01ef554b"
-          (reference "JP?") (unit 1)
-        )
         (path "/2783b917-8d7b-4d69-a31c-61fb9333015c/b6a51085-368c-402e-8235-8439715b747c"
           (reference "JP45") (unit 1)
@@
   (symbol (lib_id "power:GND") (at 115.57 180.34 0) (unit 1)
     (in_bom yes) (on_board yes) (dnp no) (fields_autoplaced)
-    (property "Reference" "#PWR?" (at 115.57 186.69 0)
+    (property "Reference" "#PWR0138" (at 115.57 186.69 0)
       (effects (font (size 1.27 1.27)) hide)
     )
@@
     (instances
       (project "meshium_duo"
-        (path "/2783b917-8d7b-4d69-a31c-61fb9333015c"
-          (reference "#PWR?") (unit 1)
-        )
         (path "/2783b917-8d7b-4d69-a31c-61fb9333015c/b6a51085-368c-402e-8235-8439715b747c"
           (reference "#PWR0138") (unit 1)
@@
   (symbol (lib_id "Jumper:Jumper_2_Bridged") (at 90.17 33.02 0) (unit 1)
     (in_bom yes) (on_board yes) (dnp no)
-    (property "Reference" "JP?" (at 83.82 31.75 0)
+    (property "Reference" "JP43" (at 83.82 31.75 0)
       (effects (font (size 1.27 1.27)))
     )
@@
     (instances
       (project "meshium_duo"
-        (path "/2783b917-8d7b-4d69-a31c-61fb9333015c/4c1314f5-8ce3-41c8-9fa4-b5bc01ef554b"
-          (reference "JP?") (unit 1)
-        )
         (path "/2783b917-8d7b-4d69-a31c-61fb9333015c/b6a51085-368c-402e-8235-8439715b747c"
           (reference "JP43") (unit 1)
@@
   (symbol (lib_id "Jumper:Jumper_2_Open") (at 33.02 88.9 0) (unit 1)
     (in_bom yes) (on_board yes) (dnp no)
-    (property "Reference" "JP?" (at 26.67 87.63 0)
+    (property "Reference" "JP42" (at 26.67 87.63 0)
       (effects (font (size 1.27 1.27)))
     )
@@
     (instances
       (project "meshium_duo"
-        (path "/2783b917-8d7b-4d69-a31c-61fb9333015c/4c1314f5-8ce3-41c8-9fa4-b5bc01ef554b"
-          (reference "JP?") (unit 1)
-        )
         (path "/2783b917-8d7b-4d69-a31c-61fb9333015c/b6a51085-368c-402e-8235-8439715b747c"
           (reference "JP42") (unit 1)
@@
   (symbol (lib_id "Jumper:Jumper_2_Open") (at 90.17 105.41 0) (unit 1)
     (in_bom yes) (on_board yes) (dnp no)
-    (property "Reference" "JP?" (at 83.82 104.14 0)
+    (property "Reference" "JP47" (at 83.82 104.14 0)
       (effects (font (size 1.27 1.27)))
     )
@@
     (instances
       (project "meshium_duo"
-        (path "/2783b917-8d7b-4d69-a31c-61fb9333015c/4c1314f5-8ce3-41c8-9fa4-b5bc01ef554b"
-          (reference "JP?") (unit 1)
-        )
         (path "/2783b917-8d7b-4d69-a31c-61fb9333015c/b6a51085-368c-402e-8235-8439715b747c"
           (reference "JP47") (unit 1)
@@
   (symbol (lib_id "Connector:Conn_01x02_Pin") (at 118.11 172.72 270) (unit 1)
     (in_bom yes) (on_board yes) (dnp no) (fields_autoplaced)
-    (property "Reference" "J?" (at 119.38 173.355 90)
+    (property "Reference" "J13" (at 119.38 173.355 90)
       (effects (font (size 1.27 1.27)) (justify left))
     )
@@
     (instances
       (project "meshium_duo"
-        (path "/2783b917-8d7b-4d69-a31c-61fb9333015c/4c1314f5-8ce3-41c8-9fa4-b5bc01ef554b"
-          (reference "J?") (unit 1)
-        )
-        (path "/2783b917-8d7b-4d69-a31c-61fb9333015c"
-          (reference "J?") (unit 1)
-        )
         (path "/2783b917-8d7b-4d69-a31c-61fb9333015c/b6a51085-368c-402e-8235-8439715b747c"
           (reference "J13") (unit 1)
@@
   (symbol (lib_id "Jumper:Jumper_2_Open") (at 90.17 36.83 0) (unit 1)
     (in_bom yes) (on_board yes) (dnp no)
-    (property "Reference" "JP?" (at 83.82 35.56 0)
+    (property "Reference" "JP44" (at 83.82 35.56 0)
       (effects (font (size 1.27 1.27)))
     )
@@
     (instances
       (project "meshium_duo"
-        (path "/2783b917-8d7b-4d69-a31c-61fb9333015c/4c1314f5-8ce3-41c8-9fa4-b5bc01ef554b"
-          (reference "JP?") (unit 1)
-        )
         (path "/2783b917-8d7b-4d69-a31c-61fb9333015c/b6a51085-368c-402e-8235-8439715b747c"
           (reference "JP44") (unit 1)
@@
   (symbol (lib_id "Jumper:Jumper_2_Open") (at 90.17 100.33 0) (unit 1)
     (in_bom yes) (on_board yes) (dnp no)
-    (property "Reference" "JP?" (at 83.82 99.06 0)
+    (property "Reference" "JP46" (at 83.82 99.06 0)
       (effects (font (size 1.27 1.27)))
     )
@@
     (instances
       (project "meshium_duo"
-        (path "/2783b917-8d7b-4d69-a31c-61fb9333015c/4c1314f5-8ce3-41c8-9fa4-b5bc01ef554b"
-          (reference "JP?") (unit 1)
-        )
         (path "/2783b917-8d7b-4d69-a31c-61fb9333015c/b6a51085-368c-402e-8235-8439715b747c"
           (reference "JP46") (unit 1)
