File: HARDWARE/USB.kicad_sch (KiCad schematic)
At the start: 1 part

Commit message: schematic capture
Parts:
- added C35: 4.7u, Capacitor_Tantalum_SMD:CP_EIA-6032-28_Kemet-C, symbol Device:C_Polarized_Small
- added D8 (x2): LED_Small, LED_SMD:LED_0603_1608Metric, symbol Device:LED_Small
- added D9: ESDA6V1BC6, Package_TO_SOT_SMD:SOT-23-6, symbol Power_Protection:ESDA6V1BC6
- added J3: USB_B_Micro, Footpint:USB_Micro-B_CUZD188-CB1Z, symbol Connector:USB_B_Micro
- added JP10 (x2): Jumper_2_Bridged, Jumper:SolderJumper-2_P1.3mm_Open_TrianglePad1.0x1.5mm, symbol Jumper:Jumper_2_Bridged
- added Q1: BC848, Package_TO_SOT_SMD:SOT-23, symbol Transistor_BJT:BC848
- added R12: 330, Resistor_SMD:R_0603_1608Metric, symbol Device:R_Small
- added R12: 620, Resistor_SMD:R_0603_1608Metric, symbol Device:R_Small
- added R12 (x3): 47K, Resistor_SMD:R_0603_1608Metric, symbol Device:R_Small
- added R12: 620K, Resistor_SMD:R_0603_1608Metric, symbol Device:R_Small
- added R12: 10K, Resistor_SMD:R_0603_1608Metric, symbol Device:R_Small
- added R12: 430K, Resistor_SMD:R_0603_1608Metric, symbol Device:R_Small
- added U10: TPS2051B, Package_TO_SOT_SMD:SOT-23-5, symbol meshium_duo:TPS2051B
Connections:
- net USB_DM: now also D9.4 (TVS3), J3.2 (D-)
- net USB_DP: now also D9.3 (TVS2), J3.3 (D+)
- net USB_ID: now also D9.6 (TVS4), J3.4 (ID)
- net USB_OVERCURRENT: now also JP10.1 (A)
- net USB_POWER_SWITCH_ON: now also JP10.1 (A)
- net USB_VBUS: now also C35.1, D9.1 (TVS1), J3.1 (VBUS), R12.1, R12.1, U10.1 (OUT)
- net at JP10.2 (B): now also R12.1, U10.4 (~{EN})
- new net: D8.1 (K), Q1.3 (C)
- new net: D8.2 (A), R12.2 (x2)
- new net: Q1.1 (B), R12.1, R12.2
- new net: D8.1 (K), JP10.2 (B), R12.2, U10.3 (~{OC})
- new net: JP10.2 (B), R12.1, R12.2
- new net +3V3: R12.1, R12.1, R12.1
- new net +5V: U10.5 (IN)
- new net GND: C35.2, D9.2 (COM), D9.5 (COM), J3.5 (GND), J3.6 (Shield), Q1.2 (E), R12.2, R12.2, R12.2, U10.2 (GND)
- new net USB_VBUS_DET: JP10.1 (A)
Other:
- moved on the sheet: JP10

Commit message: schematic capture
Parts:
- renumbered C35 to C?, D9 to D12, D8 to D?, J3 to J?, JP10 to JP?, Q1 to Q?, R12 to R?, U10 to U?

Commit message: tracerouting
Connections:
- net +3V3 renamed +3V3_PER
Changed lines of the file:
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@@
-    )
-  )
-  (symbol (lib_id "meshium_duo:+3V3_PER") (at 128.27 55.88 0) (unit 1)
-    (in_bom yes) (on_board yes) (dnp no) (fields_autoplaced)
-    (property "Reference" "#PWR?" (at 128.27 59.69 0)
-      (effects (font (size 1.27 1.27)) hide)
-    )
-    (property "Value" "+3V3_PER" (at 128.27 50.8 0)
-      (effects (font (size 1.27 1.27)))
-    )
-    (property "Footprint" "" (at 128.27 55.88 0)
-      (effects (font (size 1.27 1.27)) hide)
-    )
-    (property "Datasheet" "" (at 128.27 55.88 0)
-      (effects (font (size 1.27 1.27)) hide)
-    )
-    (pin "1")
-    (instances
-      (project "meshium_duo"
-        (path "/2783b917-8d7b-4d69-a31c-61fb9333015c"
-          (reference "#PWR?") (unit 1)
-        )
-        (path "/2783b917-8d7b-4d69-a31c-61fb9333015c/191f4f98-48ae-4893-bf0a-75f1c9b9512d"
-          (reference "#PWR0113") (unit 1)
-        )
-      )
     )
   )
@@
     )
   )
+  (symbol (lib_name "+3V3_PER_1") (lib_id "meshium_duo:+3V3_PER") (at 222.25 101.6 0) (unit 1)
+    (in_bom yes) (on_board yes) (dnp no) (fields_autoplaced)
+    (property "Reference" "#PWR080" (at 222.25 105.41 0)
+      (effects (font (size 1.27 1.27)) hide)
+    )
+    (property "Value" "+3V3_PER" (at 222.25 96.52 0)
+      (effects (font (size 1.27 1.27)))
+    )
+    (property "Footprint" "" (at 222.25 101.6 0)
+      (effects (font (size 1.27 1.27)) hide)
+    )
+    (property "Datasheet" "" (at 222.25 101.6 0)
+      (effects (font (size 1.27 1.27)) hide)
+    )
+    (pin "1")
+    (instances
+      (project "meshium_duo"
+        (path "/2783b917-8d7b-4d69-a31c-61fb9333015c/191f4f98-48ae-4893-bf0a-75f1c9b9512d"
+          (reference "#PWR080") (unit 1)
+        )
+      )
+    )
+  )
   (symbol (lib_id "Transistor_BJT:BC848") (at 219.71 120.65 0) (unit 1)
     (in_bom yes) (on_board yes) (dnp no) (fields_autoplaced)
@@
         (path "/2783b917-8d7b-4d69-a31c-61fb9333015c/191f4f98-48ae-4893-bf0a-75f1c9b9512d"
           (reference "JP40") (unit 1)
-        )
-      )
-    )
-  )
-  (symbol (lib_id "meshium_duo:+3V3_PER") (at 222.25 101.6 0) (unit 1)
-    (in_bom yes) (on_board yes) (dnp no) (fields_autoplaced)
-    (property "Reference" "#PWR?" (at 222.25 105.41 0)
-      (effects (font (size 1.27 1.27)) hide)
-    )
-    (property "Value" "+3V3_PER" (at 222.25 96.52 0)
-      (effects (font (size 1.27 1.27)))
-    )
-    (property "Footprint" "" (at 222.25 101.6 0)
-      (effects (font (size 1.27 1.27)) hide)
-    )
-    (property "Datasheet" "" (at 222.25 101.6 0)
-      (effects (font (size 1.27 1.27)) hide)
-    )
-    (pin "1")
-    (instances
-      (project "meshium_duo"
-        (path "/2783b917-8d7b-4d69-a31c-61fb9333015c"
-          (reference "#PWR?") (unit 1)
-        )
-        (path "/2783b917-8d7b-4d69-a31c-61fb9333015c/191f4f98-48ae-4893-bf0a-75f1c9b9512d"
-          (reference "#PWR0121") (unit 1)
         )
       )
@@
         )
       )
+    )
+  )
+  (symbol (lib_name "+3V3_PER_1") (lib_id "meshium_duo:+3V3_PER") (at 128.27 55.88 0) (unit 1)
+    (in_bom yes) (on_board yes) (dnp no) (fields_autoplaced)
+    (property "Reference" "#PWR078" (at 128.27 59.69 0)
+      (effects (font (size 1.27 1.27)) hide)
+    )
+    (property "Value" "+3V3_PER" (at 128.27 50.8 0)
+      (effects (font (size 1.27 1.27)))
+    )
+    (property "Footprint" "" (at 128.27 55.88 0)
+      (effects (font (size 1.27 1.27)) hide)
+    )
+    (property "Datasheet" "" (at 128.27 55.88 0)
+      (effects (font (size 1.27 1.27)) hide)
+    )
+    (pin "1")
+    (instances
+      (project "meshium_duo"
+        (path "/2783b917-8d7b-4d69-a31c-61fb9333015c/191f4f98-48ae-4893-bf0a-75f1c9b9512d"
+          (reference "#PWR078") (unit 1)
+        )
+      )

Commit message: tracerouting
Parts:
- gave numbers to parts that had none: 17
